File: Rart60xt.kicad_sch (KiCad schematic)
At the start: 8 parts, among them Y1 12MHz

Commit message: Process
Parts:
- added C3: 100nF, symbol Device:C_Small
- added F1: 500mA, symbol Device:Polyfuse_Small
- added J1: USB_C_Receptacle_USB2.0, symbol Connector:USB_C_Receptacle_USB2.0
- added R4: 1k, symbol Device:R_Small
- added R5, R6: 5.1k, symbol Device:R_Small
- added SW1: Boot, symbol Switch:SW_Push
- added U9: W25Q128JVS, Package_SO:SOIC-8_5.23x5.23mm_P1.27mm, symbol Memory_Flash:W25Q128JVS
- added U?: SRV05-4, Package_TO_SOT_SMD:SOT-23-6, symbol Power_Protection:SRV05-4
Connections:
- net +3.3V: now also C3.2, U9.8 (VCC)
- net GND: now also C3.1, J1.A1 (GND), J1.A12 (GND), J1.B1 (GND), J1.B12 (GND), J1.S1 (SHIELD), R5.2, R6.2, SW1.2, U9.4 (GND), U?.2 (VN)
- net SCLK: now also U9.6 (CLK)
- net SD0: now also U9.5 (DI(IO0))
- net SD1: now also U9.2 (DO(IO1))
- net SD2: now also U9.3 (IO2)
- net SD3: now also U9.7 (IO3)
- net D+ renamed DP
- net DP: now also J1.A6 (D+), J1.B6 (D+), U?.1 (IO1)
- net D- renamed DN
- net DN: now also J1.A7 (D-), J1.B7 (D-), U?.4 (IO3)
- new net: J1.B5 (CC2), R6.1
- new net: R4.1, SW1.1
- new net: J1.A5 (CC1), R5.1
- new net: R4.2, U9.1 (~{CS})
- new net +5V: F1.1, U?.5 (VP)
- new net VBUS: F1.2, J1.A4 (VBUS), J1.A9 (VBUS), J1.B4 (VBUS), J1.B9 (VBUS)
- no-connect marks 0 -> 2
Other:
- moved on the sheet: C1, C2, R1, R10, R2, R3, U?, Y1

Commit message: break
Parts:
- added U?: XC6206PxxxMR, Package_TO_SOT_SMD:SOT-23, symbol Regulator_Linear:XC6206PxxxMR
Changed lines of the file:
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@@
     (pin "2")
+  )
+  (symbol (lib_id "Regulator_Linear:XC6206PxxxMR") (at 134.62 62.23 0) (unit 1)
+    (in_bom yes) (on_board yes) (fields_autoplaced)
+    (property "Reference" "U?" (id 0) (at 134.62 54.61 0))
+    (property "Value" "XC6206PxxxMR" (id 1) (at 134.62 57.15 0))
+    (property "Footprint" "Package_TO_SOT_SMD:SOT-23" (id 2) (at 134.62 56.515 0)
+      (effects (font (size 1.27 1.27) italic) hide)
+    )
+    (property "Datasheet" "https://www.torexsemi.com/file/xc6206/XC6206.pdf" (id 3) (at 134.62 62.23 0)
+      (effects (font (size 1.27 1.27)) hide)
+    )
+    (pin "1")
+    (pin "2")
+    (pin "3")
   )
   (symbol (lib_id "Device:R_Small") (at 118.11 25.4 90) (unit 1)
@@
       (reference "U?") (unit 1) (value "SRV05-4") (footprint "Package_TO_SOT_SMD:SOT-23-6")
     )
+    (path "/eef7ba55-7070-42d9-a12b-8fed33840e53"
+      (reference "U?") (unit 1) (value "XC6206PxxxMR") (footprint "Package_TO_SOT_SMD:SOT-23")
+    )
     (path "/637a8555-7a36-4b19-a129-832a8e1482c7"

Commit message: pcb
Parts:
- added C10: 10uF, Capacitor_SMD:C_0805_2012Metric, symbol Device:C_Small
- added C11, C12, C13, C14, C15, C16, C17, C7, C8: 100nF, Capacitor_SMD:C_0805_2012Metric, symbol Device:C_Small
- added C4, C5, C6, C9: 1uF, Capacitor_SMD:C_0805_2012Metric, symbol Device:C_Small
- added D1, D10, D2, D3, D4, D5, D6, D7, D8, D9: D_Small, Diode_SMD:D_SOD-123, symbol Device:D_Small
- added J2: Conn_01x05, Connector_PinHeader_2.00mm:PinHeader_1x05_P2.00mm_Vertical, symbol Connector_Generic:Conn_01x05
- added M1, M10, M2, M3, M4, M5, M6, M7, M8, M9: MX-NoLED, Button_Switch_Keyboard:SW_Cherry_MX_1.00u_PCB, symbol MX_Alps_Hybrid:MX-NoLED
- C1, C2, C3: footprint (none) -> Capacitor_SMD:C_0805_2012Metric
- F1: footprint (none) -> Fuse:Fuse_1206_3216Metric
- J1: footprint (none) -> Connector_USB:USB_C_Receptacle_HRO_TYPE-C-31-M-12
- R1, R2, R3, R4, R5, R6: footprint (none) -> Resistor_SMD:R_0805_2012Metric
- SW1: footprint (none) -> random-keyboard-parts:Reset_Pretty
- Y1: footprint (none) -> Crystal:Crystal_SMD_3225-4Pin_3.2x2.5mm
- gave numbers to parts that had none: 3
- renumbered U9 to U4
Connections:
- net +1V1: now also C6.1, C7.1, C8.1
- net +3.3V: now also C10.1, C11.1, C12.1, C13.1, C14.1, C15.1, C16.1, C17.1, C9.1, J2.3 (Pin_3)
- net CLK: now also J2.5 (Pin_5)
- net DIO: now also J2.4 (Pin_4)
- net GND: now also U2.1 (GND), Y1.2, Y1.4, C10.2, C11.2, C12.2, C13.2, C14.2, C15.2, C16.2, C17.2, C4.2, C5.2, C6.2, C7.2, C8.2, C9.2, J2.2 (Pin_2)
- net Reset: now also J2.1 (Pin_1)
- net SS: now also R4.2, U4.1 (~{CS})
- net at U2.2 (VO): now also C5.1
- net at U2.3 (VI): now also C4.1
- new net: M10.1 (COL), M6.1 (COL), M7.1 (COL), M8.1 (COL), M9.1 (COL)
- new net: D9.2 (A), M9.2 (ROW)
- new net: D10.1 (K), D5.1 (K)
- new net: D5.2 (A), M5.2 (ROW)
- new net: D4.1 (K), D9.1 (K)
- new net: D2.1 (K), D7.1 (K)
- new net: D7.2 (A), M7.2 (ROW)
- new net: D4.2 (A), M4.2 (ROW)
- new net: D10.2 (A), M10.2 (ROW)
- new net: D1.1 (K), D6.1 (K)
- new net: D6.2 (A), M6.2 (ROW)
- new net: M1.1 (COL), M2.1 (COL), M3.1 (COL), M4.1 (COL), M5.1 (COL)
- new net: D8.2 (A), M8.2 (ROW)
- new net: D3.1 (K), D8.1 (K)
- new net: D1.2 (A), M1.2 (ROW)
- new net: D2.2 (A), M2.2 (ROW)
- new net: D3.2 (A), M3.2 (ROW)
- no-connect marks 2 -> 4
Other:
- moved on the sheet: U2

Commit message: done
Connections:
- net +3.3V: now also C5.1, U2.2 (VO)
- net +5V: now also C4.1, U2.3 (VI)
Changed lines of the file:
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@@
   (junction (at 16.51 85.09) (diameter 0) (color 0 0 0 0)
   )
+  (junction (at 135.89 63.5) (diameter 0) (color 0 0 0 0)
+  )
   (junction (at 184.15 66.04) (diameter 0) (color 0 0 0 0)
   )
@@
   )
   (junction (at 26.67 80.01) (diameter 0) (color 0 0 0 0)
+  )
+  (junction (at 118.11 63.5) (diameter 0) (color 0 0 0 0)
   )
   (junction (at 143.51 53.34) (diameter 0) (color 0 0 0 0)
@@
     (pin "1")
     (pin "2")
+  )
+  (symbol (lib_id "power:+5V") (at 118.11 63.5 0) (unit 1)
+    (in_bom yes) (on_board yes) (fields_autoplaced)
+    (property "Reference" "#PWR?" (id 0) (at 118.11 67.31 0)
+      (effects (font (size 1.27 1.27)) hide)
+    )
+    (property "Value" "+5V" (id 1) (at 118.11 58.42 0))
+    (property "Footprint" "" (id 2) (at 118.11 63.5 0)
+      (effects (font (size 1.27 1.27)) hide)
+    )
+    (property "Datasheet" "" (id 3) (at 118.11 63.5 0)
+      (effects (font (size 1.27 1.27)) hide)
+    )
+    (pin "1")
   )
   (symbol (lib_id "Device:D_Small") (at 113.03 137.16 90) (unit 1)
@@
     (pin "6")
   )
+  (symbol (lib_id "power:+3.3V") (at 135.89 63.5 0) (unit 1)
+    (in_bom yes) (on_board yes) (fields_autoplaced)
+    (property "Reference" "#PWR?" (id 0) (at 135.89 67.31 0)
+      (effects (font (size 1.27 1.27)) hide)
+    )
+    (property "Value" "+3.3V" (id 1) (at 135.89 58.42 0))
+    (property "Footprint" "" (id 2) (at 135.89 63.5 0)
+      (effects (font (size 1.27 1.27)) hide)
+    )
+    (property "Datasheet" "" (id 3) (at 135.89 63.5 0)
+      (effects (font (size 1.27 1.27)) hide)
+    )
+    (pin "1")
+  )
   (symbol (lib_id "power:VBUS") (at 246.38 21.59 0) (unit 1)
     (in_bom yes) (on_board yes) (fields_autoplaced)
@@
       (reference "#PWR0120") (unit 1) (value "+3.3V") (footprint "")
     )
+    (path "/15de0215-7c77-4ba5-8c5f-8fca5dc3523a"
+      (reference "#PWR?") (unit 1) (value "+5V") (footprint "")
+    )
+    (path "/8f90d403-b642-4b2a-a6b5-c82f9725b6a4"
+      (reference "#PWR?") (unit 1) (value "+3.3V") (footprint "")
+    )
     (path "/7b149139-36e7-45ac-98c2-3ce40f1aa7e2"
