File: Rart60xt.kicad_pcb (KiCad board)
At the start: 2 copper layers, 38.1 x 95.2 mm, 53 parts, among them J1 USB_C_Receptacle_USB2.0, J2 Conn_01x05, M1 MX-NoLED, M10 MX-NoLED, M2 MX-NoLED, M3 MX-NoLED, M4 MX-NoLED, M5 MX-NoLED, M6 MX-NoLED, M7 MX-NoLED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

Commit message: add
Other:
- board size 38.1 x 95.2 mm -> 38.4 x 95.5 mm
Changed lines of the file:
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@@
     )
   )
-  (gr_line (start 61.11875 115.09375) (end 58.7375 117.475) (layer "Edge.Cuts") (width 0.1))
-  (gr_line (start 23.01875 115.09375) (end 23.01875 24.60625) (layer "Edge.Cuts") (width 0.1))
-  (gr_line (start 25.4 117.475) (end 23.01875 115.09375) (layer "Edge.Cuts") (width 0.1))
+  (gr_line (start 22.86 117.602) (end 22.86 26.67) (layer "Edge.Cuts") (width 0.1))
+  (gr_line (start 22.86 22.098) (end 61.214 22.098) (layer "Edge.Cuts") (width 0.1))
   (gr_line (start 58.7375 117.475) (end 25.4 117.475) (layer "Edge.Cuts") (width 0.1))
-  (gr_line (start 23.01875 24.60625) (end 25.4 22.225) (layer "Edge.Cuts") (width 0.1))
+  (gr_arc (start 58.674 22.098) (mid 60.470051 22.841949) (end 61.214 24.638) (layer "Edge.Cuts") (width 0.1))
   (gr_line (start 61.11875 24.60625) (end 61.11875 115.09375) (layer "Edge.Cuts") (width 0.1))
-  (gr_line (start 57.15 22.225) (end 58.7375 22.225) (layer "Edge.Cuts") (width 0.1))
-  (gr_line (start 25.4 22.225) (end 57.15 22.225) (layer "Edge.Cuts") (width 0.1))
-  (gr_line (start 58.7375 22.225) (end 61.11875 24.60625) (layer "Edge.Cuts") (width 0.1))
+  (gr_arc (start 22.86 24.638) (mid 23.603949 22.841949) (end 25.4 22.098) (layer "Edge.Cuts") (width 0.1))
+  (gr_line (start 22.86 26.67) (end 22.86 22.098) (layer "Edge.Cuts") (width 0.1))
+  (gr_line (start 61.214 117.602) (end 22.86 117.602) (layer "Edge.Cuts") (width 0.1))
+  (gr_line (start 61.214 22.098) (end 61.214 117.602) (layer "Edge.Cuts") (width 0.1))
 )
