File: New folder/DB.brd (EAGLE design)
At the start: 94.1 x 95.2 mm, 20 parts, among them J1 TYPE-C-31-M-12, U3 LTC4054, U6 DW01A, U7 FS8205, X2 BM06B-SRSS-TB

Commit message: add
Parts:
- turned E1 to 180 degrees
- turned F1 to 270 degrees
Connections:
- net GND: now also BAT1.2
- net N$82: now also BAT1.1
- net VCC: now also X2.6
- net VUSB: no longer X2.6
Routing:
- net VBAT: track 0.00 -> 44.0 mm, vias 0 -> 4
- net N$82: track 0.00 -> 38.4 mm, vias 0 -> 1
- net VUSB: track 0.00 -> 25.3 mm, vias 0 -> 2
- net VCC: track 0.00 -> 24.0 mm, vias 0 -> 2
- net DN: track 0.00 -> 16.9 mm
- net DP: track 0.00 -> 15.7 mm, vias 0 -> 2
- net GND: track 0.00 -> 14.5 mm
- net N$85: track 0.00 -> 7.54 mm
- net N$83: track 0.00 -> 7.29 mm
- net N$110: track 0.00 -> 6.50 mm
- net N$111: track 0.00 -> 5.94 mm
- net N$88: track 0.00 -> 4.97 mm
- net N$113: track 0.00 -> 2.21 mm
- net N$112: track 0.00 -> 2.21 mm
- net N$89: track 0.00 -> 1.99 mm
Other:
- outline, holes or cut-outs redrawn

Commit message: add
Parts:
- added BAT2, BAT3, CHG1: (no value), adafruit:JST-PH-2-THM-RA
- added C2: 4.7uf, Components:C0805
- added C3: 100nF, Components:C0805
- added E2: SRV05-4.TCT, SRV05-4.TCT:SOT95P280X145-6N
- added F2: 500mA, fuse:RESC3216X125N
- added J2: TYPE-C-31-M-12, TYPE-C-31-M-12:HRO_TYPE-C-31-M-12
- added LED2: (no value), adafruit:CHIPLED_1206
- added R10: (no value), Components:R0805
- added R3, R4: 5.1k, Components:R0805
- added R5: 10k/2k, Components:R0805
- added R8: 1k, Components:R0805
- added R9: 100ohm, Components:R0805
- added S1: MSK-12C02_SMD_SPDT_SWITCH, MSK-12C02 SMD Micro Slider Switch SPDT:MSK-12C02
- added U1: LTC4054, LTC4054:LTC4054
- added U2: DW01A, DW01A:SOT23-6
- added U4: FS8205, FS8205:SOT95P280X145-6N
- added X1: BM06B-SRSS-TB, con-JST SH:BM06B-SRSS-TB
Connections:
- new net DN1: E2.4, J2.A7, J2.B7, X1.5
- new net DP1: E2.1, J2.A6, J2.B6, X1.4
- new net N$41: J2.A5, R4.2
- new net N$42: J2.B5, R3.2
- new net N$43: R5.2, U1.5
- new net N$44: LED2.C, U1.1
- new net N$45: LED2.A, R8.1
- new net N$46: BAT2.1, BAT3.1, S1.L2
- new net N$47: C3.2, R9.2, U2.5
- new net N$48: R10.1, U2.2
- new net N$49: U2.1, U4.6
- new net N$50: U2.3, U4.4
- new net VBAT1: C2.2, R9.1, S1.COM, U1.3, X1.2
- new net VCC1: F2.2, R8.2, U1.4, X1.6
- new net VUSB1: CHG1.1, E2.5, F2.1, J2.A4B9, J2.B4A9
- net GND: now also BAT2.2, BAT3.2, C2.1, C3.1, CHG1.2, E2.2, J2.A1B12, J2.B1A12, J2.S1, J2.S2, J2.S3, J2.S4, R10.2, R3.1, R4.1, R5.1, U1.2, U2.6, U4.1, U4.3, X1.3
Other:
- outline, holes or cut-outs redrawn
