File: DB/DBS.brd (EAGLE design)
At the start: 98 x 96.5 mm, 20 parts, among them J1 TYPE-C-31-M-12, J10 TYPE-C-31-M-12, J2 TYPE-C-31-M-12, J3 TYPE-C-31-M-12, J4 TYPE-C-31-M-12, J5 TYPE-C-31-M-12, J6 TYPE-C-31-M-12, J7 TYPE-C-31-M-12, J8 TYPE-C-31-M-12, J9 TYPE-C-31-M-12, X1 SM04B-SRSS-TB, X10 SM04B-SRSS-TB, X2 SM04B-SRSS-TB, X3 SM04B-SRSS-TB, X4 SM04B-SRSS-TB, X5 SM04B-SRSS-TB, X6 SM04B-SRSS-TB, X7 SM04B-SRSS-TB, X8 SM04B-SRSS-TB, X9 SM04B-SRSS-TB

Commit message: add
Parts:
- added E1, E2: SRV05-4.TCT, SRV05-4.TCT:SOT95P280X145-6N
- added F1, F2: 500mA, fuse:RESC3216X125N
- added J11, J12, J13, J14, J15, J16, J17, J18, J19, J20, J21, J22, J23, J24, J25: TYPE-C-31-M-12, TYPE-C-31-M-12:HRO_TYPE-C-31-M-12
- added R1, R2, R3, R4: 5.1k, Components:R0603
- added X11, X12, X13, X14, X15, X16, X17, X18, X19, X20, X21, X22, X23, X24, X25: SM04B-SRSS-TB, con-JST SH:SM04B-SRSS-TB
- renumbered J2 to J26, X2 to X26
Connections:
- new net DN1: E1.1, J1.A7, J1.B7, X1.2
- new net DN2: E2.1, J26.A7, J26.B7, X26.2
- new net DP1: E1.4, J1.A6, J1.B6, X1.3
- new net DP2: E2.4, J26.A6, J26.B6, X26.3
- new net N$1: J1.A5, R1.2
- new net N$101: E1.5, F1.2, J1.A4B9, J1.B4A9
- new net N$102: J26.A5, R3.2
- new net N$103: F1.1, X1.1
- new net N$104: J26.B5, R4.1
- new net N$2: J1.B5, R2.1
- new net N$3: E2.5, F2.2, J26.A4B9, J26.B4A9
- new net N$4: F2.1, X26.1
- net GND: now also E1.2, E2.2, J1.S1, J1.S2, J1.S3, J1.S4, J11.A1B12, J11.B1A12, J12.A1B12, J12.B1A12, J13.A1B12, J13.B1A12, J14.A1B12, J14.B1A12, J15.A1B12, J15.B1A12, J16.A1B12, J16.B1A12, J17.A1B12, J17.B1A12, J18.A1B12, J18.B1A12, J19.A1B12, J19.B1A12, J20.A1B12, J20.B1A12, J21.A1B12, J21.B1A12, J22.A1B12, J22.B1A12, J23.A1B12, J23.B1A12, J24.A1B12, J24.B1A12, J25.A1B12, J25.B1A12, J26.S1, J26.S2, J26.S3, J26.S4, R1.1, R2.2, R3.1, R4.2, X1.4, X26.4
- net VBUS: now also J11.A4B9, J11.B4A9, J12.A4B9, J12.B4A9, J13.A4B9, J13.B4A9, J14.A4B9, J14.B4A9, J15.A4B9, J15.B4A9, J16.A4B9, J16.B4A9, J17.A4B9, J17.B4A9, J18.A4B9, J18.B4A9, J19.A4B9, J19.B4A9, J20.A4B9, J20.B4A9, J21.A4B9, J21.B4A9, J22.A4B9, J22.B4A9, J23.A4B9, J23.B4A9, J24.A4B9, J24.B4A9, J25.A4B9, J25.B4A9; no longer J1.A4B9, J1.B4A9, J26.A4B9, J26.B4A9
