File: DB/DBS.sch (EAGLE design)
At the start: 20 parts, among them J1 TYPE-C-31-M-12, J10 TYPE-C-31-M-12, J2 TYPE-C-31-M-12, J3 TYPE-C-31-M-12, J4 TYPE-C-31-M-12, J5 TYPE-C-31-M-12, J6 TYPE-C-31-M-12, J7 TYPE-C-31-M-12, J8 TYPE-C-31-M-12, J9 TYPE-C-31-M-12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

Commit message: add
Parts:
- removed J2: TYPE-C-31-M-12, TYPE-C-31-M-12:TYPE-C-31-M-12
- removed X2: SM04B-SRSS-TB, con-JST SH:SM04B-SRSS-TB
- added E1, E2: SRV05-4.TCT, SRV05-4.TCT:SRV05-4.TCT
- added F1, F2: 500mA, fuse:0ZCJ0075AF2E
- added J11, J12, J13, J14, J15, J16, J17, J18, J19, J20, J21, J22, J23, J24, J25, J26: TYPE-C-31-M-12, TYPE-C-31-M-12:TYPE-C-31-M-12
- added R1, R2, R3, R4: 5.1k, Components:RESISTOR-0603
- added X11, X12, X13, X14, X15, X16, X17, X18, X19, X20, X21, X22, X23, X24, X25, X26: SM04B-SRSS-TB, con-JST SH:SM04B-SRSS-TB
Connections:
- new net DN1: E1.1, J1.DN1, J1.DN2, X1.2
- new net DN2: E2.1, J26.DN1, J26.DN2, X26.2
- new net DP1: E1.4, J1.DP1, J1.DP2, X1.3
- new net DP2: E2.4, J26.DP1, J26.DP2, X26.3
- new net GND: E1.2, E2.2, J1.GND, J1.SHIELD, J26.GND, J26.SHIELD, R1.1, R2.2, R3.1, R4.2, X1.4, X26.4
- new net N$1: J1.CC1, R1.2
- new net N$101: E1.5, F1.2, J1.VBUS
- new net N$102: J26.CC1, R3.2
- new net N$103: F1.1, X1.1
- new net N$104: J26.CC2, R4.1
- new net N$2: J1.CC2, R2.1
- new net N$3: E2.5, F2.2, J26.VBUS
- new net N$4: F2.1, X26.1
Other:
- moved on the sheet: J1, X1
