File: New folder/DB/DBS.brd (EAGLE design)
At the start: 98 x 96.5 mm, 58 parts, among them J1 TYPE-C-31-M-12, J10 TYPE-C-31-M-12, J11 TYPE-C-31-M-12, J12 TYPE-C-31-M-12, J13 TYPE-C-31-M-12, J14 TYPE-C-31-M-12, J15 TYPE-C-31-M-12, J16 TYPE-C-31-M-12, J17 TYPE-C-31-M-12, J18 TYPE-C-31-M-12, J19 TYPE-C-31-M-12, J20 TYPE-C-31-M-12, J21 TYPE-C-31-M-12, J22 TYPE-C-31-M-12, J23 TYPE-C-31-M-12, J24 TYPE-C-31-M-12, J25 TYPE-C-31-M-12, J26 TYPE-C-31-M-12, J3 TYPE-C-31-M-12, J4 TYPE-C-31-M-12, J5 TYPE-C-31-M-12, J6 TYPE-C-31-M-12, J7 TYPE-C-31-M-12, J8 TYPE-C-31-M-12, J9 TYPE-C-31-M-12, X1 SM04B-SRSS-TB, X10 SM04B-SRSS-TB, X11 SM04B-SRSS-TB, X12 SM04B-SRSS-TB, X13 SM04B-SRSS-TB, X14 SM04B-SRSS-TB, X15 SM04B-SRSS-TB, X16 SM04B-SRSS-TB, X17 SM04B-SRSS-TB, X18 SM04B-SRSS-TB, X19 SM04B-SRSS-TB, X20 SM04B-SRSS-TB, X21 SM04B-SRSS-TB, X22 SM04B-SRSS-TB, X23 SM04B-SRSS-TB, X24 SM04B-SRSS-TB, X25 SM04B-SRSS-TB, X26 SM04B-SRSS-TB, X3 SM04B-SRSS-TB, X4 SM04B-SRSS-TB, X5 SM04B-SRSS-TB, X6 SM04B-SRSS-TB, X7 SM04B-SRSS-TB, X8 SM04B-SRSS-TB, X9 SM04B-SRSS-TB

Commit message: add
Parts:
- removed J7: TYPE-C-31-M-12, TYPE-C-31-M-12:HRO_TYPE-C-31-M-12
- removed X7: SM04B-SRSS-TB, con-JST SH:SM04B-SRSS-TB
- added E3, E4, E5, E6, E7: SRV05-4.TCT, SRV05-4.TCT:SOT95P280X145-6N
- added F3, F4, F5, F6, F7: 500mA, fuse:RESC3216X125N
- added J2: TYPE-C-31-M-12, TYPE-C-31-M-12:HRO_TYPE-C-31-M-12
- added R10, R11, R12, R13, R14, R5, R6, R7, R8, R9: 5.1k, Components:R0603
- added X2: SM04B-SRSS-TB, con-JST SH:SM04B-SRSS-TB
- moved J5 82.5 mm to (10.0, 76.2)
- moved X5 82.5 mm to (10.0, 66.5)
- moved J3 20.0 mm to (70.0, 96.2)
- moved J4 20.0 mm to (90.0, 96.2)
- moved J6 20.0 mm to (30.0, 76.2)
- moved X3 20.0 mm to (70.0, 86.5)
- moved X4 20.0 mm to (90.0, 86.5)
- moved X6 20.0 mm to (30.0, 66.5)
- moved F1 0.62 mm to (2.50, 88.1)
- moved F2 0.62 mm to (22.5, 88.1)
Connections:
- new net DN3: E3.1, J2.A7, J2.B7, X2.2
- new net DN4: E4.1, J3.A7, J3.B7, X3.2
- new net DN5: E5.1, J4.A7, J4.B7, X4.2
- new net DN6: E6.1, J5.A7, J5.B7, X5.2
- new net DN7: E7.1, J6.A7, J6.B7, X6.2
- new net DP3: E3.4, J2.A6, J2.B6, X2.3
- new net DP4: E4.4, J3.A6, J3.B6, X3.3
- new net DP5: E5.4, J4.A6, J4.B6, X4.3
- new net DP6: E6.4, J5.A6, J5.B6, X5.3
- new net DP7: E7.4, J6.A6, J6.B6, X6.3
- new net GND1: E3.2, J2.A1B12, J2.B1A12, J2.S1, J2.S2, J2.S3, J2.S4, R5.1, R6.2, X2.4
- new net GND2: E4.2, J3.A1B12, J3.B1A12, J3.S1, J3.S2, J3.S3, J3.S4, R7.1, R8.2, X3.4
- new net GND3: E5.2, J4.A1B12, J4.B1A12, J4.S1, J4.S2, J4.S3, J4.S4, R10.2, R9.1, X4.4
- new net GND4: E6.2, J5.A1B12, J5.B1A12, J5.S1, J5.S2, J5.S3, J5.S4, R11.1, R12.2, X5.4
- new net GND5: E7.2, J6.A1B12, J6.B1A12, J6.S1, J6.S2, J6.S3, J6.S4, R13.1, R14.2, X6.4
- new net N$105: E3.5, F3.2, J2.A4B9, J2.B4A9
- new net N$106: F3.1, X2.1
- new net N$107: J2.A5, R5.2
- new net N$108: J2.B5, R6.1
- new net N$109: E4.5, F4.2, J3.A4B9, J3.B4A9
- new net N$110: F4.1, X3.1
- new net N$111: J3.A5, R7.2
- new net N$112: J3.B5, R8.1
- new net N$113: E5.5, F5.2, J4.A4B9, J4.B4A9
- new net N$114: F5.1, X4.1
- new net N$115: J4.A5, R9.2
- new net N$116: J4.B5, R10.1
- new net N$117: E6.5, F6.2, J5.A4B9, J5.B4A9
- new net N$118: F6.1, X5.1
- new net N$119: J5.A5, R11.2
- new net N$120: J5.B5, R12.1
- new net N$121: E7.5, F7.2, J6.A4B9, J6.B4A9
- new net N$122: F7.1, X6.1
- new net N$123: J6.A5, R13.2
- new net N$124: J6.B5, R14.1
- net GND: no longer J3.A1B12, J3.B1A12, J4.A1B12, J4.B1A12, J5.A1B12, J5.B1A12, J6.A1B12, J6.B1A12, J7.A1B12, J7.B1A12
- net VBUS: no longer J3.A4B9, J3.B4A9, J4.A4B9, J4.B4A9, J5.A4B9, J5.B4A9, J6.A4B9, J6.B4A9, J7.A4B9, J7.B4A9

Commit message: add
Parts:
- removed J22, J23, J24, J25: TYPE-C-31-M-12, TYPE-C-31-M-12:HRO_TYPE-C-31-M-12
- removed X22, X23, X24, X25: SM04B-SRSS-TB, con-JST SH:SM04B-SRSS-TB
- added E10, E11, E12, E13, E14, E15, E16, E17, E18, E19, E20, E21, E22, E8, E9: SRV05-4.TCT, SRV05-4.TCT:SOT95P280X145-6N
- added F10, F11, F12, F13, F14, F15, F16, F17, F18, F19, F20, F21, F22, F8, F9: 500mA, fuse:RESC3216X125N
- added J7: TYPE-C-31-M-12, TYPE-C-31-M-12:HRO_TYPE-C-31-M-12
- added R15, R16, R17, R18, R19, R20, R21, R22, R23, R24, R25, R26, R27, R28, R29, R30, R31, R32, R33, R34, R35, R36, R37, R38, R39, R40, R41, R42, R43, R44: 5.1k, Components:R0603
- added X7: SM04B-SRSS-TB, con-JST SH:SM04B-SRSS-TB
- moved J10 82.5 mm to (10.0, 56.2)
- moved J15 82.5 mm to (10.0, 36.2)
- moved J20 82.5 mm to (10.0, 16.2)
- moved X10 82.5 mm to (10.0, 46.5)
- moved X15 82.5 mm to (10.0, 26.5)
- moved X20 82.5 mm to (10.0, 6.50)
- moved J11 20.0 mm to (30.0, 56.2)
- moved J12 20.0 mm to (50.0, 56.2)
- moved J13 20.0 mm to (70.0, 56.2)
- moved J14 20.0 mm to (90.0, 56.2)
- moved J16 20.0 mm to (30.0, 36.2)
- moved J17 20.0 mm to (50.0, 36.2)
- moved J18 20.0 mm to (70.0, 36.2)
- moved J19 20.0 mm to (90.0, 36.2)
- moved J21 20.0 mm to (30.0, 16.2)
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Connections:
- removed net GND1: E3.2, J2.A1B12, J2.B1A12, J2.S1, J2.S2, J2.S3, J2.S4, R5.1, R6.2, X2.4
- removed net GND2: E4.2, J3.A1B12, J3.B1A12, J3.S1, J3.S2, J3.S3, J3.S4, R7.1, R8.2, X3.4
- removed net GND3: E5.2, J4.A1B12, J4.B1A12, J4.S1, J4.S2, J4.S3, J4.S4, R10.2, R9.1, X4.4
- removed net GND4: E6.2, J5.A1B12, J5.B1A12, J5.S1, J5.S2, J5.S3, J5.S4, R11.1, R12.2, X5.4
- removed net GND5: E7.2, J6.A1B12, J6.B1A12, J6.S1, J6.S2, J6.S3, J6.S4, R13.1, R14.2, X6.4
- removed net VBUS: J10.A4B9, J10.B4A9, J11.A4B9, J11.B4A9, J12.A4B9, J12.B4A9, J13.A4B9, J13.B4A9, J14.A4B9, J14.B4A9, J15.A4B9, J15.B4A9, J16.A4B9, J16.B4A9, J17.A4B9, J17.B4A9, J18.A4B9, J18.B4A9, J19.A4B9, J19.B4A9, J20.A4B9, J20.B4A9, J21.A4B9, J21.B4A9, J22.A4B9, J22.B4A9, J23.A4B9, J23.B4A9, J24.A4B9, J24.B4A9, J25.A4B9, J25.B4A9, J8.A4B9, J8.B4A9, J9.A4B9, J9.B4A9
- new net DN10: E10.1, J9.A7, J9.B7, X9.2
- new net DN11: E11.1, J10.A7, J10.B7, X10.2
- new net DN12: E12.1, J11.A7, J11.B7, X11.2
- new net DN13: E13.1, J12.A7, J12.B7, X12.2
- new net DN14: E14.1, J13.A7, J13.B7, X13.2
- new net DN15: E15.1, J14.A7, J14.B7, X14.2
- new net DN16: E16.1, J15.A7, J15.B7, X15.2
- new net DN17: E17.1, J16.A7, J16.B7, X16.2
- new net DN18: E18.1, J17.A7, J17.B7, X17.2
- new net DN19: E19.1, J18.A7, J18.B7, X18.2
- new net DN20: E20.1, J19.A7, J19.B7, X19.2
- new net DN21: E21.1, J20.A7, J20.B7, X20.2
- new net DN22: E22.1, J21.A7, J21.B7, X21.2
- new net DN8: E8.1, J7.A7, J7.B7, X7.2
- new net DN9: E9.1, J8.A7, J8.B7, X8.2
- new net DP10: E10.4, J9.A6, J9.B6, X9.3
- new net DP11: E11.4, J10.A6, J10.B6, X10.3
- new net DP12: E12.4, J11.A6, J11.B6, X11.3
- new net DP13: E13.4, J12.A6, J12.B6, X12.3
- new net DP14: E14.4, J13.A6, J13.B6, X13.3
- new net DP15: E15.4, J14.A6, J14.B6, X14.3
- new net DP16: E16.4, J15.A6, J15.B6, X15.3
- new net DP17: E17.4, J16.A6, J16.B6, X16.3
- new net DP18: E18.4, J17.A6, J17.B6, X17.3
- new net DP19: E19.4, J18.A6, J18.B6, X18.3
- new net DP20: E20.4, J19.A6, J19.B6, X19.3
- new net DP21: E21.4, J20.A6, J20.B6, X20.3
- new net DP22: E22.4, J21.A6, J21.B6, X21.3
- new net DP8: E8.4, J7.A6, J7.B6, X7.3
- new net DP9: E9.4, J8.A6, J8.B6, X8.3
- new net N$125: E8.5, F8.2, J7.A4B9, J7.B4A9
- new net N$126: F8.1, X7.1
- new net N$127: J7.A5, R15.2
- new net N$128: J7.B5, R16.1
- new net N$129: E9.5, F9.2, J8.A4B9, J8.B4A9
- new net N$130: F9.1, X8.1
- new net N$131: J8.A5, R17.2
- new net N$132: J8.B5, R18.1
- new net N$133: E10.5, F10.2, J9.A4B9, J9.B4A9
- new net N$134: F10.1, X9.1
- new net N$135: J9.A5, R19.2
- new net N$136: J9.B5, R20.1
- new net N$137: E11.5, F11.2, J10.A4B9, J10.B4A9
- new net N$138: F11.1, X10.1
- new net N$139: J10.A5, R21.2
- new net N$140: J10.B5, R22.1
- new net N$141: E12.5, F12.2, J11.A4B9, J11.B4A9
- new net N$142: F12.1, X11.1
- new net N$143: J11.A5, R23.2
- new net N$144: J11.B5, R24.1
- new net N$145: E13.5, F13.2, J12.A4B9, J12.B4A9
- new net N$146: F13.1, X12.1
- new net N$147: J12.A5, R25.2
- new net N$148: J12.B5, R26.1
- new net N$149: E14.5, F14.2, J13.A4B9, J13.B4A9
- new net N$150: F14.1, X13.1
- new net N$151: J13.A5, R27.2
- new net N$152: J13.B5, R28.1
- new net N$153: E15.5, F15.2, J14.A4B9, J14.B4A9
- new net N$154: F15.1, X14.1
- new net N$155: J14.A5, R29.2
- new net N$156: J14.B5, R30.1
- new net N$157: E16.5, F16.2, J15.A4B9, J15.B4A9
- new net N$158: F16.1, X15.1
- new net N$159: J15.A5, R31.2
- new net N$160: J15.B5, R32.1
- new net N$161: E17.5, F17.2, J16.A4B9, J16.B4A9
- new net N$162: F17.1, X16.1
- new net N$163: J16.A5, R33.2
- new net N$164: J16.B5, R34.1
- new net N$165: E18.5, F18.2, J17.A4B9, J17.B4A9
- new net N$166: F18.1, X17.1
- new net N$167: J17.A5, R35.2
- new net N$168: J17.B5, R36.1
- new net N$169: E19.5, F19.2, J18.A4B9, J18.B4A9
- new net N$170: F19.1, X18.1
- new net N$171: J18.A5, R37.2
- new net N$172: J18.B5, R38.1
- new net N$173: E20.5, F20.2, J19.A4B9, J19.B4A9
- new net N$174: F20.1, X19.1
- new net N$175: J19.A5, R39.2
- new net N$176: J19.B5, R40.1
- new net N$177: E21.5, F21.2, J20.A4B9, J20.B4A9
- new net N$178: F21.1, X20.1
- new net N$179: J20.A5, R41.2
- new net N$180: J20.B5, R42.1
- new net N$181: E22.5, F22.2, J21.A4B9, J21.B4A9
- new net N$182: F22.1, X21.1
- new net N$183: J21.A5, R43.2
- new net N$184: J21.B5, R44.1
- net GND: now also E10.2, E11.2, E12.2, E13.2, E14.2, E15.2, E16.2, E17.2, E18.2, E19.2, E20.2, E21.2, E22.2, E3.2, E4.2, E5.2, E6.2, E7.2, E8.2, E9.2, J10.S1, J10.S2, J10.S3, J10.S4, J11.S1, J11.S2, J11.S3, J11.S4, J12.S1, J12.S2, J12.S3, J12.S4, J13.S1, J13.S2, J13.S3, J13.S4, J14.S1, J14.S2, J14.S3, J14.S4, J15.S1, J15.S2, J15.S3, J15.S4, J16.S1, J16.S2, J16.S3, J16.S4, J17.S1, J17.S2, J17.S3, J17.S4, J18.S1, J18.S2, J18.S3, J18.S4, J19.S1, J19.S2, J19.S3, J19.S4, J2.A1B12, J2.B1A12, J2.S1, J2.S2, J2.S3, J2.S4, J20.S1, J20.S2, J20.S3, J20.S4, J21.S1, J21.S2, J21.S3, J21.S4, J3.A1B12, J3.B1A12, J3.S1, J3.S2, J3.S3, J3.S4, J4.A1B12, J4.B1A12, J4.S1, J4.S2, J4.S3, J4.S4, J5.A1B12, J5.B1A12, J5.S1, J5.S2, J5.S3, J5.S4, J6.A1B12, J6.B1A12, J6.S1, J6.S2, J6.S3, J6.S4, J7.A1B12, J7.B1A12, J7.S1, J7.S2, J7.S3, J7.S4, J8.S1, J8.S2, J8.S3, J8.S4, J9.S1, J9.S2, J9.S3, J9.S4, R10.2, R11.1, R12.2, R13.1, R14.2, R15.1, R16.2, R17.1, R18.2, R19.1, R20.2, R21.1, R22.2, R23.1, R24.2, R25.1, R26.2, R27.1, R28.2, R29.1, R30.2, R31.1, R32.2, R33.1, R34.2, R35.1, R36.2, R37.1, R38.2, R39.1, R40.2, R41.1, R42.2, R43.1, R44.2, R5.1, R6.2, R7.1, R8.2, R9.1, X10.4, X11.4, X12.4, X13.4, X14.4, X15.4, X16.4, X17.4, X18.4, X19.4, X2.4, X20.4, X21.4, X3.4, X4.4, X5.4, X6.4, X7.4, X8.4, X9.4; no longer J22.A1B12, J22.B1A12, J23.A1B12, J23.B1A12, J24.A1B12, J24.B1A12, J25.A1B12, J25.B1A12
Other:
- outline, holes or cut-outs redrawn

Commit message: add
Parts:
- added E23, E24, E25: SRV05-4.TCT, SRV05-4.TCT:SOT95P280X145-6N
- added F23, F24, F25: 500mA, fuse:RESC3216X125N
- added J22, J23, J24: TYPE-C-31-M-12, TYPE-C-31-M-12:HRO_TYPE-C-31-M-12
- added R45, R46, R47, R48, R49, R50: 5.1k, Components:R0603
- added X22, X23, X24: SM04B-SRSS-TB, con-JST SH:SM04B-SRSS-TB
Connections:
- new net DN23: E23.1, J22.A7, J22.B7, X22.2
- new net DN24: E24.1, J23.A7, J23.B7, X23.2
- new net DN25: E25.1, J24.A7, J24.B7, X24.2
- new net DP23: E23.4, J22.A6, J22.B6, X22.3
- new net DP24: E24.4, J23.A6, J23.B6, X23.3
- new net DP25: E25.4, J24.A6, J24.B6, X24.3
- new net N$185: E23.5, F23.2, J22.A4B9, J22.B4A9
- new net N$186: F23.1, X22.1
- new net N$187: J22.A5, R45.2
- new net N$188: J22.B5, R46.1
- new net N$189: E24.5, F24.2, J23.A4B9, J23.B4A9
- new net N$190: F24.1, X23.1
- new net N$191: J23.A5, R47.2
- new net N$192: J23.B5, R48.1
- new net N$193: E25.5, F25.2, J24.A4B9, J24.B4A9
- new net N$194: F25.1, X24.1
- new net N$195: J24.A5, R49.2
- new net N$196: J24.B5, R50.1
- net GND: now also E23.2, E24.2, E25.2, J22.A1B12, J22.B1A12, J22.S1, J22.S2, J22.S3, J22.S4, J23.A1B12, J23.B1A12, J23.S1, J23.S2, J23.S3, J23.S4, J24.A1B12, J24.B1A12, J24.S1, J24.S2, J24.S3, J24.S4, R45.1, R46.2, R47.1, R48.2, R49.1, R50.2, X22.4, X23.4, X24.4
Other:
- outline, holes or cut-outs redrawn
