File: New folder/DB/DBS.brd (EAGLE design)
At the start: 98 x 96.5 mm, 150 parts, among them J1 TYPE-C-31-M-12, J10 TYPE-C-31-M-12, J11 TYPE-C-31-M-12, J12 TYPE-C-31-M-12, J13 TYPE-C-31-M-12, J14 TYPE-C-31-M-12, J15 TYPE-C-31-M-12, J16 TYPE-C-31-M-12, J17 TYPE-C-31-M-12, J18 TYPE-C-31-M-12, J19 TYPE-C-31-M-12, J2 TYPE-C-31-M-12, J20 TYPE-C-31-M-12, J21 TYPE-C-31-M-12, J22 TYPE-C-31-M-12, J23 TYPE-C-31-M-12, J24 TYPE-C-31-M-12, J26 TYPE-C-31-M-12, J3 TYPE-C-31-M-12, J4 TYPE-C-31-M-12, J5 TYPE-C-31-M-12, J6 TYPE-C-31-M-12, J7 TYPE-C-31-M-12, J8 TYPE-C-31-M-12, J9 TYPE-C-31-M-12, X1 SM04B-SRSS-TB, X10 SM04B-SRSS-TB, X11 SM04B-SRSS-TB, X12 SM04B-SRSS-TB, X13 SM04B-SRSS-TB, X14 SM04B-SRSS-TB, X15 SM04B-SRSS-TB, X16 SM04B-SRSS-TB, X17 SM04B-SRSS-TB, X18 SM04B-SRSS-TB, X19 SM04B-SRSS-TB, X2 SM04B-SRSS-TB, X20 SM04B-SRSS-TB, X21 SM04B-SRSS-TB, X22 SM04B-SRSS-TB, X23 SM04B-SRSS-TB, X24 SM04B-SRSS-TB, X26 SM04B-SRSS-TB, X3 SM04B-SRSS-TB, X4 SM04B-SRSS-TB, X5 SM04B-SRSS-TB, X6 SM04B-SRSS-TB, X7 SM04B-SRSS-TB, X8 SM04B-SRSS-TB, X9 SM04B-SRSS-TB

Commit message: add
Parts:
- turned E10 to 90 degrees
- turned E11 to 90 degrees
- turned E12 to 90 degrees
- turned E13 to 90 degrees
- turned E14 to 90 degrees
- turned E15 to 90 degrees
- turned E16 to 90 degrees
- turned E17 to 90 degrees
- turned E18 to 90 degrees
- turned E19 to 90 degrees
- turned E2 to 90 degrees
- turned E20 to 90 degrees
- turned E21 to 90 degrees
- turned E22 to 90 degrees
- turned E23 to 90 degrees
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Routing:
- net DP1: track 0.00 -> 28.8 mm
- net DN1: track 0.00 -> 26.9 mm, vias 0 -> 2
- net DN2: track 0.00 -> 22.8 mm
- net N$101: track 0.00 -> 21.5 mm, vias 0 -> 3
- net DP2: track 0.00 -> 18.0 mm
- net N$141: track 0.00 -> 17.4 mm, vias 0 -> 3
- net N$125: track 0.00 -> 16.9 mm, vias 0 -> 3
- net N$121: track 0.00 -> 16.8 mm, vias 0 -> 3
- net N$105: track 0.00 -> 16.8 mm, vias 0 -> 3
- net N$149: track 0.00 -> 16.8 mm, vias 0 -> 3
- net N$133: track 0.00 -> 16.7 mm, vias 0 -> 3
- net N$113: track 0.00 -> 16.7 mm, vias 0 -> 3
- net N$173: track 0.00 -> 16.7 mm, vias 0 -> 3
- net N$169: track 0.00 -> 16.7 mm, vias 0 -> 3
- net N$129: track 0.00 -> 16.7 mm, vias 0 -> 3
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
Commit message: add
Routing:
- net DN3: track 0.00 -> 23.0 mm
- net DP3: track 0.00 -> 21.5 mm
- net N$177: track 0.00 -> 16.7 mm, vias 0 -> 3
- net N$185: track 0.00 -> 16.7 mm, vias 0 -> 3
- net N$189: track 0.00 -> 16.7 mm, vias 0 -> 3
- net N$193: track 0.00 -> 16.7 mm, vias 0 -> 3
- net N$161: track 0.00 -> 16.6 mm, vias 0 -> 3
- net N$157: track 0.00 -> 16.6 mm, vias 0 -> 3
- net N$181: track 0.00 -> 16.6 mm, vias 0 -> 3
- net N$107: track 0.00 -> 8.00 mm
- net N$111: track 0.00 -> 7.80 mm
- net N$112: track 0.00 -> 7.66 mm
- net N$108: track 0.00 -> 7.66 mm
- net N$186: track 0.00 -> 6.05 mm
- net N$178: track 0.00 -> 6.05 mm
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
Commit message: add
Parts:
- moved F1 1.25 mm to (3.75, 88.1)
- moved F10 1.25 mm to (83.8, 68.1)
- moved F11 1.25 mm to (3.75, 48.1)
- moved F12 1.25 mm to (23.8, 48.1)
- moved F13 1.25 mm to (43.8, 48.1)
- moved F14 1.25 mm to (63.8, 48.1)
- moved F15 1.25 mm to (83.8, 48.1)
- moved F16 1.25 mm to (3.75, 28.1)
- moved F17 1.25 mm to (23.8, 28.1)
- moved F18 1.25 mm to (43.8, 28.1)
- moved F19 1.25 mm to (63.8, 28.1)
- moved F2 1.25 mm to (23.8, 88.1)
- moved F20 1.25 mm to (83.8, 28.1)
- moved F21 1.25 mm to (3.75, 8.12)
- moved F22 1.25 mm to (23.8, 8.12)
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Routing:
- net GND: track 4.96 -> 280.0 mm, vias 7 -> 32
- net DN12: track 0.00 -> 24.1 mm
- net DN11: track 0.00 -> 22.9 mm
- net DN19: track 0.00 -> 22.9 mm
- net DN24: track 0.00 -> 22.8 mm
- net DN5: track 0.00 -> 22.8 mm
- net DN17: track 0.00 -> 22.8 mm
- net DN20: track 0.00 -> 22.7 mm
- net DN15: track 0.00 -> 22.7 mm
- net DN13: track 0.00 -> 22.7 mm
- net DN18: track 0.00 -> 22.6 mm
- net DN9: track 0.00 -> 22.6 mm
- net DN25: track 0.00 -> 22.6 mm
- net DN8: track 0.00 -> 22.6 mm
- net DN16: track 0.00 -> 22.5 mm
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- added copper zone on layer 1, net GND
- added copper zone on layer 16, net GND
