File: New folder/DB/DBS.brd (EAGLE design)
At the start: 98 x 96.5 mm, 150 parts, among them J1 TYPE-C-31-M-12, J10 TYPE-C-31-M-12, J11 TYPE-C-31-M-12, J12 TYPE-C-31-M-12, J13 TYPE-C-31-M-12, J14 TYPE-C-31-M-12, J15 TYPE-C-31-M-12, J16 TYPE-C-31-M-12, J17 TYPE-C-31-M-12, J18 TYPE-C-31-M-12, J19 TYPE-C-31-M-12, J2 TYPE-C-31-M-12, J20 TYPE-C-31-M-12, J21 TYPE-C-31-M-12, J22 TYPE-C-31-M-12, J23 TYPE-C-31-M-12, J24 TYPE-C-31-M-12, J26 TYPE-C-31-M-12, J3 TYPE-C-31-M-12, J4 TYPE-C-31-M-12, J5 TYPE-C-31-M-12, J6 TYPE-C-31-M-12, J7 TYPE-C-31-M-12, J8 TYPE-C-31-M-12, J9 TYPE-C-31-M-12, X1 SM04B-SRSS-TB, X10 SM04B-SRSS-TB, X11 SM04B-SRSS-TB, X12 SM04B-SRSS-TB, X13 SM04B-SRSS-TB, X14 SM04B-SRSS-TB, X15 SM04B-SRSS-TB, X16 SM04B-SRSS-TB, X17 SM04B-SRSS-TB, X18 SM04B-SRSS-TB, X19 SM04B-SRSS-TB, X2 SM04B-SRSS-TB, X20 SM04B-SRSS-TB, X21 SM04B-SRSS-TB, X22 SM04B-SRSS-TB, X23 SM04B-SRSS-TB, X24 SM04B-SRSS-TB, X26 SM04B-SRSS-TB, X3 SM04B-SRSS-TB, X4 SM04B-SRSS-TB, X5 SM04B-SRSS-TB, X6 SM04B-SRSS-TB, X7 SM04B-SRSS-TB, X8 SM04B-SRSS-TB, X9 SM04B-SRSS-TB

Commit message: add
Parts:
- moved E1 48.8 mm to (16.9, 136.2)
- moved E10 48.8 mm to (96.9, 116.2)
- moved E11 48.8 mm to (16.9, 96.2)
- moved E12 48.8 mm to (37.5, 96.2)
- moved E13 48.8 mm to (56.9, 96.2)
- moved E14 48.8 mm to (76.9, 96.2)
- moved E15 48.8 mm to (96.9, 96.2)
- moved E16 48.8 mm to (16.9, 76.2)
- moved E17 48.8 mm to (36.9, 76.2)
- moved E18 48.8 mm to (56.9, 76.2)
- moved E19 48.8 mm to (76.9, 76.2)
- moved E2 48.8 mm to (36.9, 136.2)
- moved E20 48.8 mm to (96.9, 76.2)
- moved E21 48.8 mm to (16.9, 56.2)
- moved E22 48.8 mm to (36.9, 56.2)
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