File: New folder/DB/DBS.sch (EAGLE design)
At the start: 58 parts, among them J1 TYPE-C-31-M-12, J10 TYPE-C-31-M-12, J11 TYPE-C-31-M-12, J12 TYPE-C-31-M-12, J13 TYPE-C-31-M-12, J14 TYPE-C-31-M-12, J15 TYPE-C-31-M-12, J16 TYPE-C-31-M-12, J17 TYPE-C-31-M-12, J18 TYPE-C-31-M-12, J19 TYPE-C-31-M-12, J20 TYPE-C-31-M-12, J21 TYPE-C-31-M-12, J22 TYPE-C-31-M-12, J23 TYPE-C-31-M-12, J24 TYPE-C-31-M-12, J25 TYPE-C-31-M-12, J26 TYPE-C-31-M-12, J3 TYPE-C-31-M-12, J4 TYPE-C-31-M-12, J5 TYPE-C-31-M-12, J6 TYPE-C-31-M-12, J7 TYPE-C-31-M-12, J8 TYPE-C-31-M-12, J9 TYPE-C-31-M-12, X1 SM04B-SRSS-TB, X10 SM04B-SRSS-TB, X11 SM04B-SRSS-TB, X12 SM04B-SRSS-TB, X13 SM04B-SRSS-TB, X14 SM04B-SRSS-TB, X15 SM04B-SRSS-TB, X16 SM04B-SRSS-TB, X17 SM04B-SRSS-TB, X18 SM04B-SRSS-TB, X19 SM04B-SRSS-TB, X20 SM04B-SRSS-TB, X21 SM04B-SRSS-TB, X22 SM04B-SRSS-TB, X23 SM04B-SRSS-TB, X24 SM04B-SRSS-TB, X25 SM04B-SRSS-TB, X26 SM04B-SRSS-TB, X3 SM04B-SRSS-TB, X4 SM04B-SRSS-TB, X5 SM04B-SRSS-TB, X6 SM04B-SRSS-TB, X7 SM04B-SRSS-TB, X8 SM04B-SRSS-TB, X9 SM04B-SRSS-TB

Commit message: add
Parts:
- removed J7: TYPE-C-31-M-12, TYPE-C-31-M-12:TYPE-C-31-M-12
- removed X7: SM04B-SRSS-TB, con-JST SH:SM04B-SRSS-TB
- added E3, E4, E5, E6, E7: SRV05-4.TCT, SRV05-4.TCT:SRV05-4.TCT
- added F3, F4, F5, F6, F7: 500mA, fuse:0ZCJ0075AF2E
- added J2: TYPE-C-31-M-12, TYPE-C-31-M-12:TYPE-C-31-M-12
- added R10, R11, R12, R13, R14, R5, R6, R7, R8, R9: 5.1k, Components:RESISTOR-0603
- added X2: SM04B-SRSS-TB, con-JST SH:SM04B-SRSS-TB
Connections:
- new net DN3: E3.1, J2.DN1, J2.DN2, X2.2
- new net DN4: E4.1, J3.DN1, J3.DN2, X3.2
- new net DN5: E5.1, J4.DN1, J4.DN2, X4.2
- new net DN6: E6.1, J5.DN1, J5.DN2, X5.2
- new net DN7: E7.1, J6.DN1, J6.DN2, X6.2
- new net DP3: E3.4, J2.DP1, J2.DP2, X2.3
- new net DP4: E4.4, J3.DP1, J3.DP2, X3.3
- new net DP5: E5.4, J4.DP1, J4.DP2, X4.3
- new net DP6: E6.4, J5.DP1, J5.DP2, X5.3
- new net DP7: E7.4, J6.DP1, J6.DP2, X6.3
- new net GND1: E3.2, J2.GND, J2.SHIELD, R5.1, R6.2, X2.4
- new net GND2: E4.2, J3.GND, J3.SHIELD, R7.1, R8.2, X3.4
- new net GND3: E5.2, J4.GND, J4.SHIELD, R10.2, R9.1, X4.4
- new net GND4: E6.2, J5.GND, J5.SHIELD, R11.1, R12.2, X5.4
- new net GND5: E7.2, J6.GND, J6.SHIELD, R13.1, R14.2, X6.4
- new net N$105: E3.5, F3.2, J2.VBUS
- new net N$106: F3.1, X2.1
- new net N$107: J2.CC1, R5.2
- new net N$108: J2.CC2, R6.1
- new net N$109: E4.5, F4.2, J3.VBUS
- new net N$110: F4.1, X3.1
- new net N$111: J3.CC1, R7.2
- new net N$112: J3.CC2, R8.1
- new net N$113: E5.5, F5.2, J4.VBUS
- new net N$114: F5.1, X4.1
- new net N$115: J4.CC1, R9.2
- new net N$116: J4.CC2, R10.1
- new net N$117: E6.5, F6.2, J5.VBUS
- new net N$118: F6.1, X5.1
- new net N$119: J5.CC1, R11.2
- new net N$120: J5.CC2, R12.1
- new net N$121: E7.5, F7.2, J6.VBUS
- new net N$122: F7.1, X6.1
- new net N$123: J6.CC1, R13.2
- new net N$124: J6.CC2, R14.1
Other:
- moved on the sheet: J3, J4, J5, J6, X3, X4, X5, X6

Commit message: add
Parts:
- removed J22, J23, J24, J25: TYPE-C-31-M-12, TYPE-C-31-M-12:TYPE-C-31-M-12
- removed X22, X23, X24, X25: SM04B-SRSS-TB, con-JST SH:SM04B-SRSS-TB
- added E10, E11, E12, E13, E14, E15, E16, E17, E18, E19, E20, E21, E22, E8, E9: SRV05-4.TCT, SRV05-4.TCT:SRV05-4.TCT
- added F10, F11, F12, F13, F14, F15, F16, F17, F18, F19, F20, F21, F22, F8, F9: 500mA, fuse:0ZCJ0075AF2E
- added J7: TYPE-C-31-M-12, TYPE-C-31-M-12:TYPE-C-31-M-12
- added R15, R16, R17, R18, R19, R20, R21, R22, R23, R24, R25, R26, R27, R28, R29, R30, R31, R32, R33, R34, R35, R36, R37, R38, R39, R40, R41, R42, R43, R44: 5.1k, Components:RESISTOR-0603
- added X7: SM04B-SRSS-TB, con-JST SH:SM04B-SRSS-TB
Connections:
- removed net GND1: E3.2, J2.GND, J2.SHIELD, R5.1, R6.2, X2.4
- removed net GND2: E4.2, J3.GND, J3.SHIELD, R7.1, R8.2, X3.4
- removed net GND3: E5.2, J4.GND, J4.SHIELD, R10.2, R9.1, X4.4
- removed net GND4: E6.2, J5.GND, J5.SHIELD, R11.1, R12.2, X5.4
- removed net GND5: E7.2, J6.GND, J6.SHIELD, R13.1, R14.2, X6.4
- new net DN10: E10.1, J9.DN1, J9.DN2, X9.2
- new net DN11: E11.1, J10.DN1, J10.DN2, X10.2
- new net DN12: E12.1, J11.DN1, J11.DN2, X11.2
- new net DN13: E13.1, J12.DN1, J12.DN2, X12.2
- new net DN14: E14.1, J13.DN1, J13.DN2, X13.2
- new net DN15: E15.1, J14.DN1, J14.DN2, X14.2
- new net DN16: E16.1, J15.DN1, J15.DN2, X15.2
- new net DN17: E17.1, J16.DN1, J16.DN2, X16.2
- new net DN18: E18.1, J17.DN1, J17.DN2, X17.2
- new net DN19: E19.1, J18.DN1, J18.DN2, X18.2
- new net DN20: E20.1, J19.DN1, J19.DN2, X19.2
- new net DN21: E21.1, J20.DN1, J20.DN2, X20.2
- new net DN22: E22.1, J21.DN1, J21.DN2, X21.2
- new net DN8: E8.1, J7.DN1, J7.DN2, X7.2
- new net DN9: E9.1, J8.DN1, J8.DN2, X8.2
- new net DP10: E10.4, J9.DP1, J9.DP2, X9.3
- new net DP11: E11.4, J10.DP1, J10.DP2, X10.3
- new net DP12: E12.4, J11.DP1, J11.DP2, X11.3
- new net DP13: E13.4, J12.DP1, J12.DP2, X12.3
- new net DP14: E14.4, J13.DP1, J13.DP2, X13.3
- new net DP15: E15.4, J14.DP1, J14.DP2, X14.3
- new net DP16: E16.4, J15.DP1, J15.DP2, X15.3
- new net DP17: E17.4, J16.DP1, J16.DP2, X16.3
- new net DP18: E18.4, J17.DP1, J17.DP2, X17.3
- new net DP19: E19.4, J18.DP1, J18.DP2, X18.3
- new net DP20: E20.4, J19.DP1, J19.DP2, X19.3
- new net DP21: E21.4, J20.DP1, J20.DP2, X20.3
- new net DP22: E22.4, J21.DP1, J21.DP2, X21.3
- new net DP8: E8.4, J7.DP1, J7.DP2, X7.3
- new net DP9: E9.4, J8.DP1, J8.DP2, X8.3
- new net N$125: E8.5, F8.2, J7.VBUS
- new net N$126: F8.1, X7.1
- new net N$127: J7.CC1, R15.2
- new net N$128: J7.CC2, R16.1
- new net N$129: E9.5, F9.2, J8.VBUS
- new net N$130: F9.1, X8.1
- new net N$131: J8.CC1, R17.2
- new net N$132: J8.CC2, R18.1
- new net N$133: E10.5, F10.2, J9.VBUS
- new net N$134: F10.1, X9.1
- new net N$135: J9.CC1, R19.2
- new net N$136: J9.CC2, R20.1
- new net N$137: E11.5, F11.2, J10.VBUS
- new net N$138: F11.1, X10.1
- new net N$139: J10.CC1, R21.2
- new net N$140: J10.CC2, R22.1
- new net N$141: E12.5, F12.2, J11.VBUS
- new net N$142: F12.1, X11.1
- new net N$143: J11.CC1, R23.2
- new net N$144: J11.CC2, R24.1
- new net N$145: E13.5, F13.2, J12.VBUS
- new net N$146: F13.1, X12.1
- new net N$147: J12.CC1, R25.2
- new net N$148: J12.CC2, R26.1
- new net N$149: E14.5, F14.2, J13.VBUS
- new net N$150: F14.1, X13.1
- new net N$151: J13.CC1, R27.2
- new net N$152: J13.CC2, R28.1
- new net N$153: E15.5, F15.2, J14.VBUS
- new net N$154: F15.1, X14.1
- new net N$155: J14.CC1, R29.2
- new net N$156: J14.CC2, R30.1
- new net N$157: E16.5, F16.2, J15.VBUS
- new net N$158: F16.1, X15.1
- new net N$159: J15.CC1, R31.2
- new net N$160: J15.CC2, R32.1
- new net N$161: E17.5, F17.2, J16.VBUS
- new net N$162: F17.1, X16.1
- new net N$163: J16.CC1, R33.2
- new net N$164: J16.CC2, R34.1
- new net N$165: E18.5, F18.2, J17.VBUS
- new net N$166: F18.1, X17.1
- new net N$167: J17.CC1, R35.2
- new net N$168: J17.CC2, R36.1
- new net N$169: E19.5, F19.2, J18.VBUS
- new net N$170: F19.1, X18.1
- new net N$171: J18.CC1, R37.2
- new net N$172: J18.CC2, R38.1
- new net N$173: E20.5, F20.2, J19.VBUS
- new net N$174: F20.1, X19.1
- new net N$175: J19.CC1, R39.2
- new net N$176: J19.CC2, R40.1
- new net N$177: E21.5, F21.2, J20.VBUS
- new net N$178: F21.1, X20.1
- new net N$179: J20.CC1, R41.2
- new net N$180: J20.CC2, R42.1
- new net N$181: E22.5, F22.2, J21.VBUS
- new net N$182: F22.1, X21.1
- new net N$183: J21.CC1, R43.2
- new net N$184: J21.CC2, R44.1
- net GND: now also E10.2, E11.2, E12.2, E13.2, E14.2, E15.2, E16.2, E17.2, E18.2, E19.2, E20.2, E21.2, E22.2, E3.2, E4.2, E5.2, E6.2, E7.2, E8.2, E9.2, J10.GND, J10.SHIELD, J11.GND, J11.SHIELD, J12.GND, J12.SHIELD, J13.GND, J13.SHIELD, J14.GND, J14.SHIELD, J15.GND, J15.SHIELD, J16.GND, J16.SHIELD, J17.GND, J17.SHIELD, J18.GND, J18.SHIELD, J19.GND, J19.SHIELD, J2.GND, J2.SHIELD, J20.GND, J20.SHIELD, J21.GND, J21.SHIELD, J3.GND, J3.SHIELD, J4.GND, J4.SHIELD, J5.GND, J5.SHIELD, J6.GND, J6.SHIELD, J7.GND, J7.SHIELD, J8.GND, J8.SHIELD, J9.GND, J9.SHIELD, R10.2, R11.1, R12.2, R13.1, R14.2, R15.1, R16.2, R17.1, R18.2, R19.1, R20.2, R21.1, R22.2, R23.1, R24.2, R25.1, R26.2, R27.1, R28.2, R29.1, R30.2, R31.1, R32.2, R33.1, R34.2, R35.1, R36.2, R37.1, R38.2, R39.1, R40.2, R41.1, R42.2, R43.1, R44.2, R5.1, R6.2, R7.1, R8.2, R9.1, X10.4, X11.4, X12.4, X13.4, X14.4, X15.4, X16.4, X17.4, X18.4, X19.4, X2.4, X20.4, X21.4, X3.4, X4.4, X5.4, X6.4, X7.4, X8.4, X9.4
Other:
- moved on the sheet: J10, J11, J12, J13, J14, J15, J16, J17, J18, J19, J20, J21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

Commit message: add
Parts:
- added E23, E24, E25: SRV05-4.TCT, SRV05-4.TCT:SRV05-4.TCT
- added F23, F24, F25: 500mA, fuse:0ZCJ0075AF2E
- added J22, J23, J24: TYPE-C-31-M-12, TYPE-C-31-M-12:TYPE-C-31-M-12
- added R45, R46, R47, R48, R49, R50: 5.1k, Components:RESISTOR-0603
- added X22, X23, X24: SM04B-SRSS-TB, con-JST SH:SM04B-SRSS-TB
Connections:
- new net DN23: E23.1, J22.DN1, J22.DN2, X22.2
- new net DN24: E24.1, J23.DN1, J23.DN2, X23.2
- new net DN25: E25.1, J24.DN1, J24.DN2, X24.2
- new net DP23: E23.4, J22.DP1, J22.DP2, X22.3
- new net DP24: E24.4, J23.DP1, J23.DP2, X23.3
- new net DP25: E25.4, J24.DP1, J24.DP2, X24.3
- new net N$185: E23.5, F23.2, J22.VBUS
- new net N$186: F23.1, X22.1
- new net N$187: J22.CC1, R45.2
- new net N$188: J22.CC2, R46.1
- new net N$189: E24.5, F24.2, J23.VBUS
- new net N$190: F24.1, X23.1
- new net N$191: J23.CC1, R47.2
- new net N$192: J23.CC2, R48.1
- new net N$193: E25.5, F25.2, J24.VBUS
- new net N$194: F25.1, X24.1
- new net N$195: J24.CC1, R49.2
- new net N$196: J24.CC2, R50.1
- net GND: now also E23.2, E24.2, E25.2, J22.GND, J22.SHIELD, J23.GND, J23.SHIELD, J24.GND, J24.SHIELD, R45.1, R46.2, R47.1, R48.2, R49.1, R50.2, X22.4, X23.4, X24.4
