File: New folder/Rable/Rable.brd (EAGLE design)
At the start: 283.5 x 94.6 mm, 199 parts, among them J1 TYPE-C-31-M-12, J3 I2C-HEADER, J4 I2C-HEADER, J5 I2C-HEADER, U1 HOLYIOT-18010-NRF52840, U2 AP2112K-3.3TRG1, U3 LTC4054, U4 AO3401, U5 AO3401, X1 SM04B-SRSS-TB, X2 BM06B-SRSS-TB, X3 BM06B-SRSS-TB, X4 BM06B-SRSS-TB

Commit message: add
Parts:
- added Q1: 2N7002, 2N7002:SOT95P240X111-3N
- added R12: 100, Components:R0805
- added R13: 10k, Components:R0805
- R8: value 2M -> 10k
- moved U5 162.8 mm to (99.4, 182.8), flipped to the bottom
- moved U4 159.1 mm to (171.4, 134.5), flipped to the bottom
- moved R8 152.2 mm to (172.6, 130.4), flipped to the bottom
- moved C1 8.29 mm to (64.9, 182.8), turned to 270 degrees
- moved LED1 7.14 mm to (56.6, 182.8)
- moved R7 6.58 mm to (67.9, 182.8)
- moved U3 4.21 mm to (61.3, 182.8), turned to 180 degrees
- moved R6 0.60 mm to (53.0, 182.8), turned to 90 degrees
Connections:
- new net N$51: Q1.1, R12.1, R8.2
- new net N$53: Q1.3, R13.1, U4.1
- new net UG_EN: R12.2
- new net UG_PWR: U4.2
- net EXT_VCC: no longer U4.3
- net GND: now also Q1.2
- net POWER_PIN: no longer R8.2, U4.1
- net VCCNRF: now also R13.2, U4.3; no longer U4.2

Commit message: add
Parts:
- added R15: 100, Components:R0805
- R12: value 100 -> (none); device Components:R0805 -> Components:R0402
- moved S1 148.4 mm to (174.4, 133.3), flipped to the bottom
- moved R12 136.7 mm to (51.1, 184.6), turned to 90 degrees
- moved R4 89.8 mm to (121.4, 200.6), turned to 180 degrees
- moved R3 85.9 mm to (121.4, 203.0), turned to 180 degrees
- moved E1 83.0 mm to (116.7, 201.8), turned to 90 degrees
- moved U4 26.0 mm to (197.3, 137.2)
- moved R8 24.4 mm to (196.8, 133.9)
- moved R1 22.7 mm to (19.1, 214.3), turned to 180 degrees
- moved D11 20.8 mm to (57.1, 133.3)
- moved D1 15.6 mm to (41.1, 214.3)
- moved R5 15.5 mm to (92.3, 183.4)
- moved R13 14.0 mm to (190.2, 133.1)
- moved C3 13.7 mm to (103.0, 183.4), turned to 90 degrees
- moved X2 12.7 mm to (29.8, 184.5), turned to 90 degrees
- moved R9 12.6 mm to (117.3, 183.4), turned to 270 degrees
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Connections:
- net 1 renamed X4
- removed net N$102: 6.25U.MX1, 7U.MX2, D8.A
- removed net N$8: RALT.MX1, RALT.P$1, RALT.P$2, RALT1.MX2, RALT1.P$3, RALT1.P$4
- removed net POWER_PIN: U1.13
- new net VBAT2: S3.1, X4.2
- new net VSS: R12.1, R6.2, U3.4
- new net X16: U1.29
- new net X17: U1.30
- new net X18: U1.28
- new net X19: U1.33
- new net X20: U1.34
- new net X5: U1.36
- net C1: now also U1.9, ~.MX2, ~.P$3, ~.P$4; no longer U1.19, ~.MX1, ~.P$1, ~.P$2
- net C10: now also U1.20; no longer U1.33
- net C11: now also RALT.MX1, RALT.P$1, RALT.P$2, RALT1.MX2, RALT1.P$3, RALT1.P$4, U1.19; no longer U1.30
- net C12: now also RWIN.MX1, RWIN.P$1, RWIN.P$2, RWIN1.MX2, RWIN1.P$3, RWIN1.P$4, U1.18; no longer U1.29
- net C13: now also RWIN2.MX1, RWIN2.P$1, RWIN2.P$2, U1.15; no longer U1.28
- net C14: now also U1.17; no longer U1.27
- net C15: now also U1.16; no longer U1.26
- net C16: now also U1.8
- net C2: now also 1.MX2, 1.P$3, 1.P$4, U1.10; no longer 1.MX1, 1.P$1, 1.P$2, U1.18
- net C3: now also U1.7; no longer U1.17
- net C4: now also U1.6; no longer U1.16
- net C5: now also U1.3; no longer U1.15
- net C6: no longer U1.11
- net C7: now also 6.25U.MX1, 7U.MX2, U1.13; no longer 6.25U.MX2, 7U.MX1, U1.10
- net C8: now also U1.27; no longer U1.9
- net C9: now also U1.26; no longer U1.34
- net CAPS: no longer U1.4
- net DN: now also X1.2; no longer X1.3
- net DP: now also X1.3; no longer X1.2
- net GND: now also X1.4; no longer X1.1
- net LED: no longer U1.36
- net N$1: now also 6.25U.MX2, 7U.MX1, D8.A; no longer RWIN.MX1, RWIN.P$1, RWIN.P$2, RWIN1.MX2, RWIN1.P$3, RWIN1.P$4
- net N$2: now also ~.MX1, ~.P$1, ~.P$2; no longer ~.MX2, ~.P$3, ~.P$4
- net N$24: now also 1.MX1, 1.P$1, 1.P$2; no longer 1.MX2, 1.P$3, 1.P$4
- net N$51: now also R15.1; no longer R12.1
- net N1: no longer U1.7
- net N2: no longer U1.6
- net R1: now also U1.5; no longer U1.8
- net R2: now also U1.4; no longer U1.20
- net R3: now also U1.2; no longer U1.5
- net R4: now also U1.11; no longer U1.2
- net R5: no longer U1.3
- net UG_EN: now also R15.2; no longer R12.2
- net VBAT: no longer X4.2
- net VCC: now also R12.2; no longer R6.2, U3.4, X4.6
- net VUSB: now also X1.1, X4.6; no longer X1.4
Routing:
- net R1: track 0.00 -> 356.8 mm, vias 0 -> 2
- net R2: track 0.00 -> 345.6 mm, vias 0 -> 2
- net R3: track 0.00 -> 314.8 mm, vias 0 -> 2
- net C14: track 0.00 -> 304.0 mm
- net C13: track 0.00 -> 266.9 mm, vias 0 -> 2
- net R4: track 0.00 -> 243.7 mm
- net C1: track 0.00 -> 241.7 mm, vias 0 -> 2
- net C12: track 0.00 -> 231.2 mm, vias 0 -> 1
- net C11: track 0.00 -> 202.5 mm, vias 0 -> 1
- net C15: track 0.00 -> 200.0 mm, vias 0 -> 2
- net C2: track 0.00 -> 194.0 mm, vias 0 -> 1
- net VCC: track 0.00 -> 190.8 mm, vias 0 -> 4
- net C16: track 0.00 -> 183.6 mm, vias 0 -> 2
- net C3: track 0.00 -> 175.4 mm, vias 0 -> 1
- net VUSB: track 0.00 -> 150.9 mm, vias 0 -> 3
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Other:
- outline, holes or cut-outs redrawn

Commit message: add
Parts:
- moved U4 92.7 mm to (104.8, 141.1), turned to 270 degrees
- moved R8 92.0 mm to (104.8, 133.3)
- moved R15 87.7 mm to (104.8, 130.4), turned to 180 degrees
- moved R13 86.1 mm to (104.8, 144.1)
- moved Q1 79.5 mm to (104.8, 136.9)
- moved RGB1 61.4 mm to (83.3, 126.8), flipped to the bottom
- moved D8 1.19 mm to (160.1, 132.2)
Connections:
- net X4 renamed UG
- removed net X16: U1.29
- removed net X18: U1.28
- removed net X5: U1.36
- net C6: now also U1.13
- net C7: now also U1.27; no longer U1.13
- net C8: now also U1.28; no longer U1.27
- net R5: now also U1.29
- net UG_EN: now also U1.36
Routing:
- net R5: track 99.0 -> 225.9 mm
- net VCCNRF: track 94.3 -> 134.9 mm, vias 2 -> 4
- net RST: track 24.9 -> 55.6 mm
- net C6: track 70.8 -> 91.3 mm, vias 0 -> 1
- net UG: track 0.00 -> 13.2 mm
- net N$53: track 0.00 -> 9.72 mm
- net N$51: track 0.00 -> 8.56 mm
- net UG_EN: track 0.00 -> 8.19 mm
- net C7: track 138.6 -> 145.3 mm
- net C8: track 124.7 -> 127.5 mm
- net GND: track 16.6 -> 19.3 mm, vias 0 -> 1
- net N$1: track 24.5 -> 25.7 mm

Commit message: addadd
Parts:
- removed C10, C11, C12, C13, C14, C4, C5, C6, C7, C8, C9: (no value), Components:C0805
- removed RGB1, RGB10, RGB11, RGB2, RGB3, RGB4, RGB5, RGB6, RGB7, RGB8, RGB9: WS2812B, LED:WS2812B
- added C15, C16, C17, C18, C19, C20, C21, C22, C23, C24, C25, C26, C27, C28, C29: (no value), Components:C0603
- added U10, U11, U12, U13, U14, U15, U16, U17, U18, U19, U20, U6, U7, U8, U9: WS2812-2020, WS2812-2020:LED_WS2812-2020
- moved J5 101.8 mm to (76.8, 103.0)
- moved CAPS1 101.8 mm to (114.3, 117.3)
- moved JP1 101.8 mm to (121.4, 112.5)
- moved PWR 101.8 mm to (76.2, 112.5)
- moved R11 101.8 mm to (90.5, 117.3)
- moved R14 101.8 mm to (95.2, 117.3)
Connections:
- removed net EXT_VCC: C10.2, C11.2, C12.2, C13.2, C14.2, C4.2, C5.2, C6.2, C7.2, C8.2, C9.2, RGB1.1-VDD, RGB10.1-VDD, RGB11.1-VDD, RGB2.1-VDD, RGB3.1-VDD, RGB4.1-VDD, RGB5.1-VDD, RGB6.1-VDD, RGB7.1-VDD, RGB8.1-VDD, RGB9.1-VDD
- removed net LED: RGB1.4-DIN
- removed net N$104: RGB10.4-DIN, RGB9.2-DOUT
- removed net N$12: RGB1.2-DOUT, RGB2.4-DIN
- removed net N$13: RGB2.2-DOUT, RGB3.4-DIN
- removed net N$14: RGB5.2-DOUT, RGB6.4-DIN
- removed net N$15: RGB6.2-DOUT, RGB7.4-DIN
- removed net N$16: RGB7.2-DOUT, RGB8.4-DIN
- removed net N$17: RGB8.2-DOUT, RGB9.4-DIN
- removed net N$19: RGB10.2-DOUT, RGB11.4-DIN
- removed net N$98: RGB3.2-DOUT, RGB4.4-DIN
- removed net N$99: RGB4.2-DOUT, RGB5.4-DIN
- new net N$102: U18.1, U19.3
- new net N$105: U19.1, U20.3
- new net N$50: U7.1, U8.3
- new net N$52: U8.1, U9.3
- new net N$61: U10.3, U9.1
- new net N$67: U10.1, U11.3
- new net N$74: U11.1, U12.3
- new net N$75: U12.1, U13.3
- new net N$76: U13.1, U14.3
- new net N$79: U14.1, U15.3
- new net N$8: U6.1, U7.3
- new net N$80: U15.1, U16.3
- new net N$81: U16.1, U17.3
- new net N$84: U17.1, U18.3
- net GND: now also C15.1, C16.1, C17.1, C18.1, C19.1, C20.1, C21.1, C22.1, C23.1, C24.1, C25.1, C26.1, C27.1, C28.1, C29.1, U10.2, U11.2, U12.2, U13.2, U14.2, U15.2, U16.2, U17.2, U18.2, U19.2, U20.2, U6.2, U7.2, U8.2, U9.2; no longer C10.1, C11.1, C12.1, C13.1, C14.1, C4.1, C5.1, C6.1, C7.1, C8.1, C9.1, RGB1.3-GND, RGB10.3-GND, RGB11.3-GND, RGB2.3-GND, RGB3.3-GND, RGB4.3-GND, RGB5.3-GND, RGB6.3-GND, RGB7.3-GND, RGB8.3-GND, RGB9.3-GND
- net UG: now also U6.3
- net UG_PWR: now also C15.2, C16.2, C17.2, C18.2, C19.2, C20.2, C21.2, C22.2, C23.2, C24.2, C25.2, C26.2, C27.2, C28.2, C29.2, U10.4, U11.4, U12.4, U13.4, U14.4, U15.4, U16.4, U17.4, U18.4, U19.4, U20.4, U6.4, U7.4, U8.4, U9.4
Routing:
- net UG_PWR: track 0.00 -> 345.9 mm, vias 0 -> 7
- net N$67: track 0.00 -> 80.8 mm, vias 0 -> 2
- net N$8: track 0.00 -> 48.3 mm, vias 0 -> 2
- net N$50: track 0.00 -> 44.4 mm
- net R5: track 225.9 -> 269.6 mm, vias 0 -> 2
- net N$61: track 0.00 -> 37.8 mm
- net N$52: track 0.00 -> 36.9 mm
- net UG: track 13.2 -> 35.1 mm
- net GND: track 19.3 -> 34.6 mm, vias 1 -> 2
- net BAT_PIN: track 49.5 -> 61.1 mm
- net C16: track 183.6 -> 181.8 mm
- net C6: track 91.3 -> 92.5 mm
- net C1: track 241.7 -> 241.2 mm, vias 2 -> 3

Commit message: add
Parts:
- moved D25 0.84 mm to (103.0, 210.1)
- moved D27 0.84 mm to (141.1, 210.1)
- moved D36 0.84 mm to (198.2, 210.1)
Routing:
- net UG_PWR: track 345.9 -> 507.3 mm, vias 7 -> 9
- net N$75: track 0.00 -> 110.6 mm
- net N$74: track 0.00 -> 44.3 mm
- net R1: track 356.8 -> 359.4 mm

Commit message: add
Parts:
- moved D31 0.84 mm to (236.3, 210.1)
- moved D47 0.60 mm to (264.3, 191.1)
- moved D32 0.60 mm to (254.8, 210.1)
Routing:
- net UG_PWR: track 507.3 -> 919.4 mm, vias 9 -> 16
- net R5: track 269.6 -> 344.7 mm, vias 2 -> 4
- net R4: track 243.7 -> 313.4 mm, vias 0 -> 2
- net N$81: track 0.00 -> 68.9 mm, vias 0 -> 2
- net N$84: track 0.00 -> 59.7 mm, vias 0 -> 2
- net N$76: track 0.00 -> 57.0 mm
- net N$79: track 0.00 -> 46.3 mm, vias 0 -> 2
- net R3: track 314.8 -> 360.3 mm
- net R2: track 345.6 -> 383.0 mm, vias 2 -> 4
- net R1: track 359.4 -> 396.2 mm, vias 2 -> 4
- net N$105: track 0.00 -> 34.4 mm
- net N$102: track 0.00 -> 31.2 mm
- net N$80: track 0.00 -> 30.3 mm
- net GND: track 34.6 -> 60.4 mm, vias 2 -> 7
- net C14: track 304.0 -> 306.9 mm
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
Commit message: add
Parts:
- removed CAPS1, PWR: (no value), adafruit:LED3MM
- removed J5: I2C-HEADER, Headers:HEADER-4X1-2.54
- removed R11, R14: 75R, Components:R0805
- moved JP1 14.9 mm to (114.3, 125.6)
- moved D49 0.60 mm to (59.5, 172.0)
- moved D52 0.60 mm to (78.6, 172.0)
- moved D53 0.60 mm to (97.6, 172.0)
- moved R1 0.60 mm to (19.1, 213.7)
- moved X2 0.60 mm to (29.8, 184.0)
- moved X3 0.60 mm to (275.0, 184.0)
- moved D23 0.60 mm to (64.3, 210.1)
- moved D24 0.60 mm to (83.3, 210.1)
- moved D26 0.60 mm to (121.4, 210.1)
- moved D28 0.60 mm to (159.5, 210.1)
- moved D29 0.60 mm to (178.6, 210.1)
- moved D30 0.60 mm to (216.7, 210.1)
Connections:
- removed net CAPS: R11.1
- removed net N$11: CAPS1.A, R11.2
- removed net N$20: PWR.A, R14.2
- removed net N1: JP1.1
- removed net N2: JP1.2
- net GND: no longer CAPS1.K, J5.1, PWR.K
- net SCL: no longer J5.3
- net SDA: no longer J5.4
- net VBAT: no longer R14.1
- net VCCNRF: no longer J5.2
- net X19: now also JP1.2
- net X20: now also JP1.1
Routing:
- net R5: track 344.7 -> 437.0 mm, vias 4 -> 6
- net R4: track 313.4 -> 389.2 mm, vias 2 -> 4
- net R1: track 396.2 -> 452.8 mm, vias 4 -> 6
- net GND: track 60.4 -> 110.3 mm, vias 7 -> 37
- net R3: track 360.3 -> 393.2 mm, vias 2 -> 4
- net R2: track 383.0 -> 403.1 mm
- net X20: track 0.00 -> 6.21 mm
- net X19: track 0.00 -> 5.84 mm
- net N$60: track 0.00 -> 4.89 mm
- net N$67: track 80.8 -> 83.4 mm
- net N$86: track 60.0 -> 62.5 mm
- net N$81: track 68.9 -> 70.6 mm
- net C11: track 202.5 -> 203.3 mm
- net N$46: track 27.3 -> 28.0 mm
- net C1: track 241.2 -> 242.0 mm
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- added copper zone on layer 1, net GND
- added copper zone on layer 16, net GND

Commit message: add
Parts:
- renumbered BAT1 to BAT, BAT2 to CHG, R12 to HERE
Routing:
- net N$67: track 83.4 -> 89.5 mm
