File: New folder/Rable/Rable.brd (EAGLE design)
At the start: 283.5 x 94.6 mm, 206 parts, among them J1 TYPE-C-31-M-12, J3 I2C-HEADER, J4 I2C-HEADER, Q1 2N7002, U1 HOLYIOT-18010-NRF52840, U10 WS2812-2020, U11 WS2812-2020, U12 WS2812-2020, U13 WS2812-2020, U14 WS2812-2020, U15 WS2812-2020, U16 WS2812-2020, U17 WS2812-2020, U18 WS2812-2020, U19 WS2812-2020, U2 AP2112K-3.3TRG1, U20 WS2812-2020, U3 LTC4054, U4 AO3401, U5 AO3401, U6 WS2812-2020, U7 WS2812-2020, U8 WS2812-2020, U9 WS2812-2020, X1 SM04B-SRSS-TB, X2 BM06B-SRSS-TB, X3 BM06B-SRSS-TB, X4 BM06B-SRSS-TB

Commit message: add
Parts:
- removed C15, C16, C17, C18, C19, C20, C21, C22, C23, C24, C25, C26, C27, C28, C29: (no value), Components:C0603
- removed RALT: KEYSWITCH-PLAIN-MXHSPCB-1U, Keyboard:MXHSPCB-1U
- removed U10, U11, U12, U13, U14, U15, U16, U17, U18, U19, U20, U6, U7, U8, U9: WS2812-2020, WS2812-2020:LED_WS2812-2020
- added =1, =2, =3, =4, =5, RWIN3, TAB1, TAB2, TAB3, TAB4, ~1: KEYSWITCH-PLAIN-MXHSPCB-1U, Keyboard:MXHSPCB-1U
- added D64: (no value), Components:SOD-123
- 7U: value KEYSWITCH-PLAIN-MXHSPCB-7U-FLIPPED -> KEYSWITCH-PLAIN-MXHSPCB-7U; device Keyboard:MXHSPCB-7U-FLIPPED -> Keyboard:MXHSPCB-7U
- RSHIFT1: value KEYSWITCH-PLAIN-MXHSPCB-2U -> KEYSWITCH-PLAIN-MXHSPCB-2U-FLIPPED; device Keyboard:MXHSPCB-2U -> Keyboard:MXHSPCB-2U-FLIPPED
- moved D6 26.2 mm to (214.3, 133.3)
- moved D7 24.9 mm to (243.5, 136.3)
- moved RWIN 23.8 mm to (233.4, 133.3)
- moved D9 17.3 mm to (292.3, 138.7)
- moved X2 14.0 mm to (16.1, 186.9), turned to 0 degrees
- moved RALT1 11.9 mm to (211.9, 133.3), turned to 0 degrees
- moved RWIN1 11.9 mm to (235.7, 133.3)
- moved RWIN2 9.52 mm to (257.2, 133.3), turned to 0 degrees
- moved X3 4.21 mm to (272.1, 186.9), turned to 0 degrees
- moved D10 2.38 mm to (78.6, 133.3)
- moved D11 2.38 mm to (54.8, 133.3)
- turned 7U to 180 degrees
- turned FN to 0 degrees
- turned LALT to 180 degrees
- turned LALT1 to 0 degrees
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Connections:
- net X17 renamed 17
- removed net N$102: U18.1, U19.3
- removed net N$105: U19.1, U20.3
- removed net N$50: U7.1, U8.3
- removed net N$52: U8.1, U9.3
- removed net N$61: U10.3, U9.1
- removed net N$67: U10.1, U11.3
- removed net N$68: D14.A, RSHIFT1.MX2, RSHIFT1.P$3, RSHIFT1.P$4, RSHIFT2.MX1, RSHIFT2.P$1, RSHIFT2.P$2
- removed net N$74: U11.1, U12.3
- removed net N$75: U12.1, U13.3
- removed net N$76: U13.1, U14.3
- removed net N$79: U14.1, U15.3
- removed net N$80: U15.1, U16.3
- removed net N$81: U16.1, U17.3
- removed net N$84: U17.1, U18.3
- new net 01: U1.7
- new net 010: U1.18
- new net 011: U1.8
- new net 012: U1.9
- new net 013: U1.10
- new net 014: U1.11
- new net 02: U1.6
- new net 03: U1.12
- new net 04: U1.13
- new net 05: U1.15
- new net 06: U1.17
- new net 07: U1.20
- new net 08: U1.19
- new net 09: U1.26
- new net 15: U1.27
- new net 16: U1.29
- new net 18: U1.28
- new net 19: U1.33
- new net 20: U1.34
- new net 21: U1.16
- new net 22: U1.3
- new net 23: U1.2
- new net 24: U1.4
- new net 25: U1.5
- new net N$11: D64.A, RWIN2.MX2, RWIN2.P$3, RWIN2.P$4, RWIN3.MX1, RWIN3.P$1, RWIN3.P$2
- net BAT_PIN: no longer U1.12
- net C1: no longer U1.9
- net C10: no longer U1.20
- net C11: now also RALT1.MX1, RALT1.P$1, RALT1.P$2; no longer RALT.MX1, RALT.P$1, RALT.P$2, RALT1.MX2, RALT1.P$3, RALT1.P$4, U1.19
- net C12: no longer U1.18
- net C13: now also RSHIFT1.MX2, RSHIFT1.P$3, RSHIFT1.P$4, RSHIFT2.MX1, RSHIFT2.P$1, RSHIFT2.P$2, RWIN3.MX2, RWIN3.P$3, RWIN3.P$4; no longer RSHIFT1.MX1, RSHIFT1.P$1, RSHIFT1.P$2, RSHIFT2.MX2, RSHIFT2.P$3, RSHIFT2.P$4, U1.15
- net C14: no longer U1.17
- net C15: now also =1.MX1, =1.P$1, =1.P$2, =2.MX1, =2.P$1, =2.P$2, =3.MX1, =3.P$1, =3.P$2, =4.MX1, =4.P$1, =4.P$2, =5.MX1, =5.P$1, =5.P$2; no longer U1.16
- net C16: now also TAB1.MX1, TAB1.P$1, TAB1.P$2, TAB2.MX1, TAB2.P$1, TAB2.P$2, TAB3.MX1, TAB3.P$1, TAB3.P$2, TAB4.MX1, TAB4.P$1, TAB4.P$2, ~1.MX1, ~1.P$1, ~1.P$2; no longer U1.8
- net C2: no longer U1.10
- net C3: no longer U1.7
- net C4: no longer U1.6
- net C5: no longer U1.3
- net C6: no longer U1.13
- net C7: no longer U1.27
- net C8: no longer U1.28
- net C9: no longer U1.26
- net GND: no longer C15.1, C16.1, C17.1, C18.1, C19.1, C20.1, C21.1, C22.1, C23.1, C24.1, C25.1, C26.1, C27.1, C28.1, C29.1, U10.2, U11.2, U12.2, U13.2, U14.2, U15.2, U16.2, U17.2, U18.2, U19.2, U20.2, U6.2, U7.2, U8.2, U9.2
- net N$22: now also RALT1.MX2, RALT1.P$3, RALT1.P$4; no longer RALT.MX2, RALT.P$3, RALT.P$4, RALT1.MX1, RALT1.P$1, RALT1.P$2
- net N$8: now also D14.A, RSHIFT1.MX1, RSHIFT1.P$1, RSHIFT1.P$2, RSHIFT2.MX2, RSHIFT2.P$3, RSHIFT2.P$4; no longer U6.1, U7.3
- net R1: no longer U1.5
- net R2: no longer U1.4
- net R3: no longer U1.2
- net R4: no longer U1.11
- net R5: now also D64.C; no longer U1.29
- net UG: no longer U6.3
- net UG_PWR: no longer C15.2, C16.2, C17.2, C18.2, C19.2, C20.2, C21.2, C22.2, C23.2, C24.2, C25.2, C26.2, C27.2, C28.2, C29.2, U10.4, U11.4, U12.4, U13.4, U14.4, U15.4, U16.4, U17.4, U18.4, U19.4, U20.4, U6.4, U7.4, U8.4, U9.4
- net X19: no longer U1.33
- net X20: no longer U1.34
Routing:
- net UG_PWR: track 919.5 -> 0.00 mm, vias 16 -> 0
- net R1: track 452.8 -> 0.00 mm, vias 6 -> 0
- net R5: track 437.0 -> 0.00 mm, vias 6 -> 0
- net R2: track 403.1 -> 0.00 mm, vias 4 -> 0
- net R3: track 392.7 -> 0.00 mm, vias 4 -> 0
- net R4: track 389.2 -> 0.00 mm, vias 4 -> 0
- net C14: track 306.9 -> 0.00 mm
- net C13: track 267.5 -> 0.00 mm, vias 2 -> 0
- net C1: track 242.0 -> 0.00 mm, vias 3 -> 0
- net C12: track 232.9 -> 0.00 mm, vias 1 -> 0
- net C11: track 203.3 -> 0.00 mm, vias 1 -> 0
- net C15: track 200.0 -> 0.00 mm, vias 2 -> 0
- net C2: track 194.0 -> 0.00 mm, vias 1 -> 0
- net VCC: track 190.8 -> 0.00 mm, vias 4 -> 0
- net C16: track 182.0 -> 0.00 mm, vias 2 -> 0
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- removed copper zone on layer 1, net GND
- removed copper zone on layer 16, net GND

Commit message: add
Parts:
- moved TAB1 4.76 mm to (-4.76, 190.5)
- moved TAB2 4.76 mm to (-4.76, 171.4)
- moved TAB3 4.76 mm to (-4.76, 152.4)
- moved TAB4 4.76 mm to (-4.76, 133.3)
- moved ~1 4.76 mm to (-4.76, 209.6)
- moved D24 0.84 mm to (83.9, 209.6)
- moved D26 0.84 mm to (122.0, 209.6)
- moved D28 0.84 mm to (160.1, 209.6)
- moved D29 0.84 mm to (179.2, 209.6)
- moved D30 0.84 mm to (217.3, 209.6)
- moved D23 0.84 mm to (64.9, 209.6)
- moved D25 0.60 mm to (103.0, 209.6)
- moved D27 0.60 mm to (141.1, 209.6)
- moved D31 0.60 mm to (236.3, 209.6)
- moved D32 0.60 mm to (254.8, 209.6)
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Connections:
- removed net N$100: D11.A, LWIN.MX2, LWIN.P$3, LWIN.P$4, LWIN1.MX1, LWIN1.P$1, LWIN1.P$2
- removed net N$101: D10.A, LALT.MX2, LALT.P$3, LALT.P$4, LALT1.MX1, LALT1.P$1, LALT1.P$2
- removed net N$86: D13.A, FN.MX1, FN.P$1, FN.P$2
- new net N$12: D11.A, LWIN.MX1, LWIN.P$1, LWIN.P$2, LWIN1.MX2, LWIN1.P$3, LWIN1.P$4
- new net N$13: D10.A, LALT.MX1, LALT.P$1, LALT.P$2, LALT1.MX2, LALT1.P$3, LALT1.P$4
- new net N$14: D13.A, FN.MX2, FN.P$3, FN.P$4
- net C1: now also LCTRL.MX2, LCTRL.P$3, LCTRL.P$4, LCTRL1.MX1, LCTRL1.P$1, LCTRL1.P$2; no longer LCTRL.MX1, LCTRL.P$1, LCTRL.P$2, LCTRL1.MX2, LCTRL1.P$3, LCTRL1.P$4
- net C14: now also FN.MX1, FN.P$1, FN.P$2; no longer FN.MX2, FN.P$3, FN.P$4
- net C2: now also LWIN.MX2, LWIN.P$3, LWIN.P$4, LWIN1.MX1, LWIN1.P$1, LWIN1.P$2; no longer LWIN.MX1, LWIN.P$1, LWIN.P$2, LWIN1.MX2, LWIN1.P$3, LWIN1.P$4
- net C3: now also LALT.MX2, LALT.P$3, LALT.P$4, LALT1.MX1, LALT1.P$1, LALT1.P$2; no longer LALT.MX1, LALT.P$1, LALT.P$2, LALT1.MX2, LALT1.P$3, LALT1.P$4
- net N$6: now also LCTRL.MX1, LCTRL.P$1, LCTRL.P$2, LCTRL1.MX2, LCTRL1.P$3, LCTRL1.P$4; no longer LCTRL.MX2, LCTRL.P$3, LCTRL.P$4, LCTRL1.MX1, LCTRL1.P$1, LCTRL1.P$2
Routing:
- net R1: track 0.00 -> 229.7 mm
- net C13: track 0.00 -> 114.5 mm, vias 0 -> 1
- net C7: track 0.00 -> 109.4 mm, vias 0 -> 2
- net C1: track 0.00 -> 106.9 mm, vias 0 -> 2
- net C14: track 0.00 -> 105.8 mm
- net C3: track 0.00 -> 103.2 mm
- net C12: track 0.00 -> 100.3 mm
- net C2: track 0.00 -> 93.0 mm
- net C11: track 0.00 -> 92.1 mm
- net C15: track 0.00 -> 80.7 mm
- net C4: track 0.00 -> 71.5 mm
- net C6: track 0.00 -> 70.8 mm
- net C9: track 0.00 -> 70.8 mm
- net C5: track 0.00 -> 70.8 mm
- net C8: track 0.00 -> 70.8 mm
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Other:
- board size 283.5 x 94.6 mm -> 327.4 x 95.2 mm
