File: New folder/Rable/Rable.brd (EAGLE design)
At the start: 327.4 x 95.2 mm, 187 parts, among them J1 TYPE-C-31-M-12, J3 I2C-HEADER, J4 I2C-HEADER, Q1 2N7002, U1 HOLYIOT-18010-NRF52840, U2 AP2112K-3.3TRG1, U3 LTC4054, U4 AO3401, U5 AO3401, X1 SM04B-SRSS-TB, X2 BM06B-SRSS-TB, X3 BM06B-SRSS-TB, X4 BM06B-SRSS-TB

Commit message: add
Parts:
- added D65, D66, D67, D68, D69, D70, D71, D72, D73, D74: (no value), Components:SOD-123
- added X5, X6: BM02B-SRSS-TB, con-JST SH:BM02B-SRSS-TB
- moved D9 21.2 mm to (271.5, 142.9), turned to 0 degrees
- moved D7 21.0 mm to (222.6, 133.3)
- moved D6 4.76 mm to (219.1, 133.3)
- moved D10 3.57 mm to (82.2, 133.3)
- moved D11 3.57 mm to (58.3, 133.3)
- moved D64 3.21 mm to (246.5, 132.8)
- moved CHG 2.98 mm to (141.1, 182.8)
- moved D8 2.98 mm to (163.1, 132.2)
- moved F1 1.88 mm to (36.9, 198.2), turned to 270 degrees
- moved D1 1.19 mm to (41.1, 213.1)
- moved D22 1.19 mm to (43.5, 213.1)
- moved D5 1.19 mm to (34.5, 133.3)
- moved R1 1.19 mm to (19.1, 212.5)
- moved D24 0.60 mm to (83.3, 209.6)
- moved D25 0.60 mm to (102.4, 209.6)
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Connections:
- new net N$15: D65.A, ~1.MX2, ~1.P$3, ~1.P$4
- new net N$16: D66.A, TAB1.MX2, TAB1.P$3, TAB1.P$4
- new net N$17: D67.A, TAB2.MX2, TAB2.P$3, TAB2.P$4
- new net N$19: D68.A, TAB3.MX2, TAB3.P$3, TAB3.P$4
- new net N$20: D69.A, TAB4.MX2, TAB4.P$3, TAB4.P$4
- new net N$21: =1.MX2, =1.P$3, =1.P$4, D70.A
- new net N$23: =2.MX2, =2.P$3, =2.P$4, D71.A
- new net N$35: =3.MX2, =3.P$3, =3.P$4, D72.A
- new net N$37: =4.MX2, =4.P$3, =4.P$4, D73.A
- new net N$47: =5.MX2, =5.P$3, =5.P$4, D74.A
- net GND: now also X4.1, X5.1, X6.1
- net N$82: now also X6.2
- net R1: now also D65.C
- net R2: now also D66.C
- net R3: now also D67.C
- net R4: now also D68.C
- net R5: now also D69.C
- net VUSB: now also X5.2
Routing:
- net VUSB: track 0.00 -> 164.8 mm, vias 0 -> 3
- net DN: track 0.00 -> 117.3 mm, vias 0 -> 2
- net DP: track 0.00 -> 115.2 mm
- net VBAT: track 0.00 -> 109.7 mm, vias 0 -> 1
- net C16: track 0.00 -> 80.7 mm
- net VCC: track 0.00 -> 78.5 mm, vias 0 -> 3
- net VBAT2: track 0.00 -> 66.6 mm, vias 0 -> 1
- net N$14: track 0.00 -> 55.1 mm
- net N$82: track 0.00 -> 53.1 mm, vias 0 -> 1
- net GND: track 0.00 -> 46.8 mm, vias 0 -> 1
- net N$11: track 0.00 -> 41.9 mm
- net N$8: track 0.00 -> 41.1 mm
- net N$103: track 0.00 -> 32.9 mm
- net N$46: track 0.00 -> 30.9 mm
- net N$36: track 0.00 -> 24.8 mm
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
Commit message: add
Parts:
- added HERE1: (no value), Components:R0402
- added R17: 22R, Components:R0805
- added U10, U11, U12, U13, U14, U15, U16, U17, U18, U19, U20, U21, U22, U23, U6, U7, U8, U9: WS2812-2020, WS2812-2020:LED_WS2812-2020
- added X7, X8: BM06B-SRSS-TB, con-JST SH:BM06B-SRSS-TB
- moved D71 9.54 mm to (312.5, 200.0), turned to 90 degrees
- moved X3 3.77 mm to (275.6, 188.1)
- moved X2 2.66 mm to (18.5, 188.1)
- moved D8 2.38 mm to (165.5, 132.2)
- turned R5 to 90 degrees
Connections:
- removed net 01: U1.7
- removed net 010: U1.18
- removed net 011: U1.8
- removed net 012: U1.9
- removed net 013: U1.10
- removed net 014: U1.11
- removed net 02: U1.6
- removed net 03: U1.12
- removed net 04: U1.13
- removed net 05: U1.15
- removed net 06: U1.17
- removed net 07: U1.20
- removed net 08: U1.19
- removed net 09: U1.26
- removed net 15: U1.27
- removed net 16: U1.29
- removed net 18: U1.28
- removed net 21: U1.16
- removed net 22: U1.3
- removed net 23: U1.2
- removed net 24: U1.4
- removed net 25: U1.5
- new net N$102: U10.3, U9.1
- new net N$104: U10.1, U11.3
- new net N$105: U11.1, U12.3
- new net N$106: U12.1, U13.3
- new net N$107: U13.1, U14.3
- new net N$108: U14.1, U15.3
- new net N$109: U15.1, U16.3
- new net N$110: U16.1, U17.3
- new net N$111: U17.1, U18.3
- new net N$112: U18.1, U19.3
- new net N$113: U19.1, U20.3
- new net N$114: U20.1, U21.3
- new net N$115: U21.1, U22.3
- new net N$116: U22.1, U23.3
- new net N$117: R17.2, U8.3
- new net N$80: U6.1, U7.3
- new net N$81: U23.1, U6.3
- new net N$98: U8.1, U9.3
- net BAT_PIN: now also U1.13
- net C1: now also U1.10
- net C10: now also U1.20
- net C11: now also U1.19
- net C12: now also U1.18
- net C13: now also U1.17
- net C14: now also U1.16
- net C15: now also U1.15, X8.1
- net C16: now also U1.9, X7.1
- net C2: now also U1.11
- net C3: now also U1.8
- net C4: now also U1.7
- net C5: now also U1.2
- net C6: now also U1.6
- net C7: now also U1.26
- net C8: now also U1.28
- net C9: now also U1.27
- net GND: now also U10.2, U11.2, U12.2, U13.2, U14.2, U15.2, U16.2, U17.2, U18.2, U19.2, U20.2, U21.2, U22.2, U23.2, U6.2, U7.2, U8.2, U9.2
- net R1: now also D70.C, U1.3, X7.6, X8.6
- net R2: now also D71.C, U1.4, X7.5, X8.5
- net R3: now also D72.C, U1.5, X7.4, X8.4
- net R4: now also D73.C, U1.12, X7.3, X8.3
- net R5: now also D74.C, U1.29, X7.2, X8.2
- net UG: now also R17.1
- net UG_PWR: now also U10.4, U11.4, U12.4, U13.4, U14.4, U15.4, U16.4, U17.4, U18.4, U19.4, U20.4, U21.4, U22.4, U23.4, U6.4, U7.4, U8.4, U9.4
- net VBAT: now also HERE1.2
- net VBAT2: now also HERE1.1
Routing:
- net UG_PWR: track 0.00 -> 896.6 mm, vias 0 -> 21
- net R5: track 0.00 -> 678.0 mm, vias 0 -> 9
- net R1: track 232.8 -> 589.2 mm, vias 0 -> 12
- net R3: track 259.2 -> 613.3 mm, vias 0 -> 9
- net R4: track 231.4 -> 576.6 mm, vias 0 -> 7
- net R2: track 247.7 -> 517.0 mm, vias 0 -> 7
- net C15: track 80.7 -> 319.1 mm, vias 0 -> 5
- net C16: track 80.7 -> 281.9 mm, vias 0 -> 2
- net C14: track 125.6 -> 295.3 mm
- net C13: track 114.5 -> 264.5 mm, vias 1 -> 2
- net GND: track 46.8 -> 182.0 mm, vias 1 -> 14
- net VCCNRF: track 3.00 -> 135.5 mm, vias 0 -> 3
- net C1: track 106.9 -> 226.5 mm
- net VCC: track 78.5 -> 195.3 mm, vias 3 -> 5
- net C12: track 100.3 -> 206.4 mm, vias 0 -> 1
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- added copper zone on layer 1, net GND
- added copper zone on layer 16, net GND
Other:
- outline, holes or cut-outs redrawn

Commit message: add
Parts:
- renumbered HERE to USB_INT, HERE1 to USB_EXT, LED1 to LED_CHG
Routing:
- net GND: track 182.0 -> 194.2 mm, vias 14 -> 17
- net C1: track 226.5 -> 229.7 mm
- net R2: track 517.0 -> 514.9 mm
- net R5: track 678.0 -> 676.8 mm
- net C2: track 184.6 -> 185.8 mm
- net R4: track 576.6 -> 577.4 mm
- net N$115: track 31.7 -> 32.3 mm
Other:
- outline, holes or cut-outs redrawn

Commit message: add
Routing:
- net N$6: track 16.5 -> 18.5 mm
- net GND: vias 17 -> 19
Changed lines of the file:
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@@
 <wire x1="20.3" y1="189.4" x2="21.36565" y2="189.4" width="0.254" layer="16"/>
 <wire x1="22.77365" y1="187.992" x2="27.208" y2="187.992" width="0.254" layer="16"/>
-<wire x1="28.6" y1="187.992" x2="31.82925" y2="187.992" width="0.254" layer="16"/>
+<wire x1="27.208" y1="187.992" x2="31.82925" y2="187.992" width="0.254" layer="16"/>
 <wire x1="21.36565" y1="189.4" x2="22.77365" y2="187.992" width="0.254" layer="16"/>
-<wire x1="25.49185" y1="192.69185" x2="25.1757" y2="193.008" width="0.254" layer="16"/>
 <wire x1="25.1757" y1="193.008" x2="22.87424375" y2="193.008" width="0.254" layer="16"/>
 <contactref element="X7" pad="5"/>
@@
 <wire x1="310.9599375" y1="197.588" x2="311.5" y2="198.1280625" width="0.254" layer="16"/>
 <wire x1="311.5" y1="198.1280625" x2="311.5" y2="200.6209375" width="0.254" layer="16"/>
-<wire x1="25.49185" y1="192.69185" x2="26.4" y2="191.7837" width="0.254" layer="16"/>
-<wire x1="27.208" y1="187.992" x2="28.6" y2="187.992" width="0.254" layer="16"/>
+<wire x1="25.1757" y1="193.008" x2="26.4" y2="191.7837" width="0.254" layer="16"/>
 <wire x1="26.4" y1="191.7837" x2="26.4" y2="188.8" width="0.254" layer="16"/>
 <wire x1="26.4" y1="188.8" x2="27.208" y2="187.992" width="0.254" layer="16"/>
@@
 <wire x1="12.6" y1="148.7" x2="13" y2="149.1" width="0.254" layer="16"/>
 <wire x1="13" y1="149.1" x2="17.6" y2="149.1" width="0.254" layer="16"/>
-<wire x1="17.6" y1="149.1" x2="17.8" y2="149.3" width="0.254" layer="16"/>
-<wire x1="17.8" y1="149.3" x2="18.15483125" y2="149.65483125" width="0.254" layer="16"/>
+<wire x1="17.6" y1="149.1" x2="18.15483125" y2="149.65483125" width="0.254" layer="16"/>
 <wire x1="18.15483125" y1="149.65483125" x2="20.05483125" y2="149.65483125" width="0.254" layer="16"/>
 </signal>
@@
 <via x="51" y="215.8" extent="1-16" drill="0.35"/>
 <via x="43.6" y="149.3" extent="1-16" drill="0.35"/>
-<wire x1="292.8484375" y1="193.79625" x2="292.8484375" y2="172.365" width="0" layer="19" extent="16-16"/>
+<via x="27.9" y="145.9" extent="1-16" drill="0.35"/>
+<via x="286.2" y="185.5" extent="1-16" drill="0.35"/>
 </signal>
 <signal name="VCC">
@@
 <wire x1="37.06115" y1="207.042" x2="35.592" y2="208.51115" width="0.254" layer="16"/>
 <wire x1="35.592" y1="208.51115" x2="35.592" y2="210.58885" width="0.254" layer="16"/>
-<wire x1="35.592" y1="210.58885" x2="37.512525" y2="212.509375" width="0.254" layer="16"/>
-<wire x1="37.512525" y1="212.509375" x2="38.19675" y2="213.1936" width="0.254" layer="16"/>
+<wire x1="35.592" y1="210.58885" x2="38.19675" y2="213.1936" width="0.254" layer="16"/>
 <wire x1="42.7514125" y1="213.1936" x2="43.4578125" y2="213.9" width="0.254" layer="16"/>
 <wire x1="38.19675" y1="213.1936" x2="42.7514125" y2="213.1936" width="0.254" layer="16"/>
@@
 <wire x1="31.4265" y1="130.81" x2="31.4265" y2="131.439" width="0.254" layer="16"/>
 <wire x1="31.4265" y1="131.439" x2="31.4325" y2="131.445" width="0.254" layer="16"/>
-<wire x1="34.528125" y1="134.985" x2="31.4265" y2="131.883375" width="0.254" layer="16"/>
 <wire x1="31.4265" y1="131.883375" x2="31.4265" y2="131.439" width="0.254" layer="16"/>
+<wire x1="31.4265" y1="130.81" x2="32.9936" y2="132.3771" width="0.254" layer="16"/>
+<wire x1="32.9936" y1="132.3771" x2="32.9936" y2="132.7683375" width="0.254" layer="16"/>
+<wire x1="32.9936" y1="132.7683375" x2="33.8316625" y2="133.6064" width="0.254" layer="16"/>
+<wire x1="34.7064" y1="133.6064" x2="35" y2="133.9" width="0.254" layer="16"/>
+<wire x1="35" y1="133.9" x2="35" y2="134.513125" width="0.254" layer="16"/>
+<wire x1="35" y1="134.513125" x2="34.528125" y2="134.985" width="0.254" layer="16"/>
+<wire x1="33.8316625" y1="133.6064" x2="34.7064" y2="133.6064" width="0.254" layer="16"/>
 </signal>
 <signal name="N$12">

Commit message: add
Connections:
- removed net X19: JP1.2
- removed net X20: JP1.1
- net 19: now also JP1.2
- net 20: now also JP1.1
Routing:
- net 19: track 0.00 -> 7.13 mm
- net 20: track 0.00 -> 6.21 mm
Changed lines of the file:
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@@
 <setting verticaltext="up"/>
 </settings>
-<grid distance="0.1" unitdist="mm" unit="mm" style="lines" multiple="8" display="yes" altdistance="2.38125" altunitdist="mm" altunit="mm"/>
+<grid distance="2.38125" unitdist="mm" unit="mm" style="lines" multiple="8" display="yes" altdistance="2.38125" altunitdist="mm" altunit="mm"/>
 <layers>
 <layer number="1" name="Top" color="4" fill="1" visible="yes" active="yes"/>
@@
 </element>
 <element name="LED_CHG" library="adafruit" package="CHIPLED_1206" value="" x="53.578125" y="181.5703125" smashed="yes" rot="MR270">
-<attribute name="NAME" x="50.085625" y="181.054375" size="0.8128" layer="26" rot="MR0"/>
+<attribute name="NAME" x="56.379375" y="179.579375" size="0.8128" layer="26" rot="MR0"/>
 <attribute name="VALUE" x="54.848125" y="179.0303125" size="1.27" layer="28" rot="MR0"/>
 </element>
@@
 <contactref element="U1" pad="30"/>
 </signal>
-<signal name="X19">
-<contactref element="JP1" pad="2"/>
-</signal>
-<signal name="X20">
-<contactref element="JP1" pad="1"/>
-</signal>
 <signal name="VSS">
 <contactref element="U3" pad="4"/>
@@
 <signal name="19">
 <contactref element="U1" pad="33"/>
+<contactref element="JP1" pad="2"/>
+<wire x1="115.3" y1="125.6109375" x2="115.3" y2="126.3" width="0.254" layer="16"/>
+<wire x1="115.3" y1="126.3" x2="114.2064" y2="127.3936" width="0.254" layer="16"/>
+<wire x1="115.8" y1="130" x2="116" y2="130.2" width="0.254" layer="16"/>
+<wire x1="116" y1="130.2" x2="116" y2="131.14375" width="0.254" layer="16"/>
+<wire x1="116" y1="131.14375" x2="115.9765625" y2="131.1671875" width="0.254" layer="16"/>
+<wire x1="114.2064" y1="127.3936" x2="114.2064" y2="129.0316625" width="0.254" layer="16"/>
+<wire x1="114.2064" y1="129.0316625" x2="115.1747375" y2="130" width="0.254" layer="16"/>
+<wire x1="115.1747375" y1="130" x2="115.8" y2="130" width="0.254" layer="16"/>
 </signal>
 <signal name="20">
 <contactref element="U1" pad="34"/>
+<contactref element="JP1" pad="1"/>
+<wire x1="113.3" y1="125.6109375" x2="113.3" y2="126.8" width="0.254" layer="16"/>
+<wire x1="113.3" y1="126.8" x2="113.8" y2="127.3" width="0.254" layer="16"/>
+<wire x1="114.8765625" y1="130.2765625" x2="114.8765625" y2="131.1671875" width="0.254" layer="16"/>
+<wire x1="113.8" y1="127.3" x2="113.8" y2="129.2" width="0.254" layer="16"/>
+<wire x1="113.8" y1="129.2" x2="114.8765625" y2="130.2765625" width="0.254" layer="16"/>
 </signal>
 <signal name="N$8">

Commit message: add
Parts:
- removed R17: 22R, Components:R0805
- removed U3: LTC4054, LTC4054:LTC4054
- added Q5: 2N7002, 2N7002:SOT95P240X111-3N
- added R11: 10k, Components:R0805
- Q1: value 2N7002 -> LTC4054; device 2N7002:SOT95P240X111-3N -> LTC4054:LTC4054
- R10: value 2M -> 10k
- R13: value 10k -> 330
- R5: value 10k -> 1k
- R6: value 1k -> 10k/2k
- R7: value 10k/2k -> 10k
- R8: value 10k -> 2M
- moved Q1 63.2 mm to (61.3, 182.8)
- moved R8 50.9 mm to (114.3, 183.4), turned to 90 degrees
- moved R10 40.4 mm to (104.8, 144.1), turned to 0 degrees
- moved R5 34.5 mm to (57.7, 182.8)
- moved R13 26.3 mm to (78.6, 141.7)
- moved R7 24.4 mm to (92.3, 183.4), turned to 90 degrees
- moved R6 10.1 mm to (67.9, 182.8), turned to 270 degrees
- renumbered R15 to R12, U10 to RGB3, U11 to RGB4, U12 to RGB5, U13 to RGB6, U14 to RGB7, U15 to RGB8, U16 to RGB9, U17 to RGB10, U18 to RGB11, U19 to RGB12, U2 to Q3, U20 to RGB13, U21 to RGB14, U22 to RGB15, U23 to RGB16, U4 to Q4, U5 to Q2, U6 to RGB17, U7 to RGB18, U8 to RGB1, U9 to RGB2
Connections:
- net BAT_PIN: now also R8.1; no longer R10.1
- net GND: now also Q5.2, R11.1, R6.1, R8.2; no longer R10.2, R5.1, R8.1, U3.2
- net N$117: now also R13.2; no longer R17.2
- net N$51: now also Q5.1, R11.2; no longer Q1.1, R8.2
- net N$53: now also Q5.3, R10.1; no longer Q1.3, R13.1
- net N$7: now also Q1.1; no longer U3.1
- net N$87: now also Q1.5, R6.2; no longer R7.2, U3.5
- net N$9: now also R5.1; no longer R6.1
- net UG: now also R13.1; no longer R17.1
- net VBAT: now also Q1.3; no longer U3.3
- net VCC: now also R7.2; no longer R5.2
- net VCCNRF: now also R10.2; no longer R13.2
- net VSS: now also Q1.4, R5.2; no longer R6.2, U3.4
Routing:
- net GND: track 194.2 -> 199.0 mm
Other:
- outline, holes or cut-outs redrawn
