File: New folder/Rable/Rable.sch (EAGLE design)
At the start: 200 parts, among them J1 TYPE-C-31-M-12, J3 I2C-HEADER, J4 I2C-HEADER, J5 I2C-HEADER, U1 HOLYIOT-18010-NRF52840, U2 AP2112K-3.3TRG1, U3 LTC4054, U4 AO3401, U5 AO3401, X1 SM04B-SRSS-TB, X2 BM06B-SRSS-TB, X3 BM06B-SRSS-TB, X4 BM06B-SRSS-TB

Commit message: add
Parts:
- removed CHGR: (no value), adafruit:LED3MM
- removed D98: SS14, SS14:SS14
- added LED1: (no value), adafruit:LEDCHIPLED_1206
Connections:
- net N$10: no longer D98.K
- net N$7: now also LED1.C; no longer CHGR.C
- net N$9: now also LED1.A; no longer CHGR.A
- net VCC: no longer D98.A
Changed lines of the file:
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@@
 <part name="JP1" library="pinhead" deviceset="PINHD-1X2" device="M"/>
 <part name="PWR" library="adafruit" deviceset="LED" device="3MM"/>
-<part name="CHGR" library="adafruit" deviceset="LED" device="3MM"/>
 <part name="CAPS1" library="adafruit" deviceset="LED" device="3MM"/>
 <part name="RGB1" library="LED" deviceset="WS2812B" device=""/>
@@
 <part name="C14" library="Components" deviceset="CAPACITOR" device="-C0805"/>
 <part name="J5" library="Headers" deviceset="I2C-HEADER" device=""/>
-<part name="D98" library="SS14" deviceset="SS14" device=""/>
 <part name="R14" library="Components" deviceset="RESISTOR" device="-0805" value="75R"/>
 <part name="BAT1" library="adafruit" deviceset="JST_2PIN" device="-THM-RA"/>
@@
 <part name="X4" library="con-JST SH" deviceset="BM06B-SRSS" device="-TB"/>
 <part name="BAT2" library="adafruit" deviceset="JST_2PIN" device="-THM-RA"/>
+<part name="LED1" library="adafruit" deviceset="LED" device="CHIPLED_1206"/>
 </parts>
 <sheets>
@@
 </instance>
 <instance part="C1" gate="G$1" x="-177.8" y="60.96" smashed="yes" rot="R90">
-<attribute name="NAME" x="-178.308" y="55.88" size="1.778" layer="95" rot="R90"/>
+<attribute name="NAME" x="-173.228" y="58.42" size="1.778" layer="95" rot="R90"/>
 <attribute name="VALUE" x="-177.546" y="61.976" size="1.778" layer="96" rot="R90" align="top-left"/>
 </instance>
@@
 <attribute name="VALUE" x="-111.125" y="48.768" size="1.778" layer="96" rot="R90"/>
 </instance>
-<instance part="CHGR" gate="G$1" x="-208.28" y="68.58" smashed="yes">
-<attribute name="NAME" x="-204.724" y="64.008" size="1.778" layer="95" rot="R90"/>
-<attribute name="VALUE" x="-202.565" y="64.008" size="1.778" layer="96" rot="R90"/>
-</instance>
 <instance part="CAPS1" gate="G$1" x="-116.84" y="30.48" smashed="yes" rot="R180">
 <attribute name="NAME" x="-120.396" y="35.052" size="1.778" layer="95" rot="R270"/>
@@
 </instance>
 <instance part="J5" gate="G$1" x="-203.2" y="2.54" smashed="yes" rot="R180"/>
-<instance part="D98" gate="G$1" x="-281.94" y="58.42" smashed="yes">
-<attribute name="NAME" x="-284.226" y="60.325" size="1.778" layer="95"/>
-<attribute name="VALUE" x="-284.226" y="54.991" size="1.778" layer="96"/>
-</instance>
 <instance part="R14" gate="G$1" x="-111.76" y="55.88" smashed="yes" rot="R180">
 <attribute name="NAME" x="-107.95" y="54.3814" size="1.778" layer="95" rot="R180"/>
@@
 <attribute name="NAME" x="-120.65" y="95.885" size="1.778" layer="95" rot="R180"/>
 <attribute name="VALUE" x="-120.65" y="106.68" size="1.778" layer="96" rot="R180"/>
+</instance>
+<instance part="LED1" gate="G$1" x="-208.28" y="68.58" smashed="yes">
+<attribute name="NAME" x="-204.724" y="66.548" size="1.778" layer="95" rot="R90"/>
+<attribute name="VALUE" x="-202.565" y="64.008" size="1.778" layer="96" rot="R90"/>
 </instance>
 </instances>
@@
 <junction x="-287.02" y="60.96"/>
 <label x="-289.56" y="66.04" size="1.778" layer="95" rot="R180" xref="yes"/>
-<pinref part="D98" gate="G$1" pin="A"/>
-<wire x1="-284.48" y1="58.42" x2="-287.02" y2="58.42" width="0.1524" layer="91"/>
-<wire x1="-287.02" y1="58.42" x2="-287.02" y2="60.96" width="0.1524" layer="91"/>
 </segment>
 <segment>
@@
 <segment>
 <pinref part="U3" gate="G$1" pin="CHRG"/>
-<pinref part="CHGR" gate="G$1" pin="C"/>
+<pinref part="LED1" gate="G$1" pin="C"/>
 </segment>
 </net>
@@
 <segment>
 <pinref part="R6" gate="G$1" pin="1"/>
-<pinref part="CHGR" gate="G$1" pin="A"/>
+<pinref part="LED1" gate="G$1" pin="A"/>
 </segment>
 </net>
@@
 <pinref part="D99" gate="D$1" pin="C"/>
 <junction x="-276.86" y="60.96"/>
-<pinref part="D98" gate="G$1" pin="K"/>
-<wire x1="-279.4" y1="58.42" x2="-276.86" y2="58.42" width="0.1524" layer="91"/>
-<wire x1="-276.86" y1="58.42" x2="-276.86" y2="60.96" width="0.1524" layer="91"/>
-</segment>
-</net>
+</segment>
+</net>

Commit message: add
Parts:
- added Q1: 2N7002, 2N7002:2N7002
- added R12: 100, Components:RESISTOR-0805
- added R13: 10k, Components:RESISTOR-0805
- R8: value 2M -> 10k
Connections:
- new net N$51: Q1.G, R12.1, R8.2
- new net N$53: Q1.D, R13.1, U4.G
- new net UG_EN: R12.2
- new net UG_PWR: U4.S
- net EXT_VCC: no longer U4.D
- net GND: now also Q1.S
- net POWER_PIN: no longer R8.2, U4.G
- net VCCNRF: now also R13.2, U4.D; no longer U4.S
Other:
- moved on the sheet: CAPS1, R11, R8, U4
Changed lines of the file:
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@@
 <part name="E1" library="SRV05-4.TCT" deviceset="SRV05-4.TCT" device=""/>
 <part name="U4" library="AO3401" deviceset="AO3401" device=""/>
-<part name="R8" library="Components" deviceset="RESISTOR" device="-0805" value="2M"/>
+<part name="R8" library="Components" deviceset="RESISTOR" device="-0805" value="10k"/>
 <part name="J3" library="Headers" deviceset="I2C-HEADER" device=""/>
 <part name="R11" library="Components" deviceset="RESISTOR" device="-0805" value="75R"/>
@@
 <part name="BAT2" library="adafruit" deviceset="JST_2PIN" device="-THM-RA"/>
 <part name="LED1" library="adafruit" deviceset="LED" device="CHIPLED_1206"/>
+<part name="Q1" library="2N7002" deviceset="2N7002" device=""/>
+<part name="R12" library="Components" deviceset="RESISTOR" device="-0805" value="100"/>
+<part name="R13" library="Components" deviceset="RESISTOR" device="-0805" value="10k"/>
 </parts>
 <sheets>
@@
 <attribute name="VALUE" x="-219.71" y="119.38" size="1.778" layer="96" align="center-left"/>
 </instance>
-<instance part="U4" gate="G$1" x="-137.16" y="63.5" smashed="yes">
-<attribute name="VALUE" x="-148.59" y="63.5" size="1.778" layer="96"/>
-<attribute name="NAME" x="-148.59" y="66.04" size="1.778" layer="95"/>
-</instance>
-<instance part="R8" gate="G$1" x="-144.78" y="55.88" smashed="yes" rot="R90">
-<attribute name="NAME" x="-146.2786" y="52.07" size="1.778" layer="95" rot="R90"/>
-<attribute name="VALUE" x="-149.098" y="54.61" size="1.778" layer="96" rot="R90"/>
+<instance part="U4" gate="G$1" x="-142.24" y="55.88" smashed="yes">
+<attribute name="VALUE" x="-135.89" y="58.42" size="1.778" layer="96"/>
+<attribute name="NAME" x="-133.35" y="55.88" size="1.778" layer="95"/>
+</instance>
+<instance part="R8" gate="G$1" x="-152.4" y="35.56" smashed="yes" rot="R90">
+<attribute name="NAME" x="-153.8986" y="31.75" size="1.778" layer="95" rot="R90"/>
+<attribute name="VALUE" x="-148.59" y="36.322" size="1.778" layer="96" rot="R180"/>
 </instance>
 <instance part="J3" gate="G$1" x="-149.86" y="91.44" smashed="yes" rot="R180"/>
-<instance part="R11" gate="G$1" x="-111.76" y="27.94" smashed="yes" rot="R180">
-<attribute name="NAME" x="-107.95" y="26.4414" size="1.778" layer="95" rot="R180"/>
-<attribute name="VALUE" x="-107.95" y="31.242" size="1.778" layer="96" rot="R180"/>
+<instance part="R11" gate="G$1" x="-111.76" y="35.56" smashed="yes" rot="R180">
+<attribute name="NAME" x="-107.95" y="34.0614" size="1.778" layer="95" rot="R180"/>
+<attribute name="VALUE" x="-107.95" y="38.862" size="1.778" layer="96" rot="R180"/>
 </instance>
 <instance part="JP1" gate="G$1" x="-114.3" y="83.82" smashed="yes">
@@
 <attribute name="VALUE" x="-111.125" y="48.768" size="1.778" layer="96" rot="R90"/>
 </instance>
-<instance part="CAPS1" gate="G$1" x="-116.84" y="30.48" smashed="yes" rot="R180">
-<attribute name="NAME" x="-120.396" y="35.052" size="1.778" layer="95" rot="R270"/>
-<attribute name="VALUE" x="-122.555" y="35.052" size="1.778" layer="96" rot="R270"/>
+<instance part="CAPS1" gate="G$1" x="-116.84" y="38.1" smashed="yes" rot="R180">
+<attribute name="NAME" x="-120.396" y="42.672" size="1.778" layer="95" rot="R270"/>
+<attribute name="VALUE" x="-122.555" y="42.672" size="1.778" layer="96" rot="R270"/>
 </instance>
 <instance part="RGB1" gate="G$1" x="-281.94" y="165.1" smashed="yes">
@@
 <attribute name="NAME" x="-204.724" y="66.548" size="1.778" layer="95" rot="R90"/>
 <attribute name="VALUE" x="-202.565" y="64.008" size="1.778" layer="96" rot="R90"/>
+</instance>
+<instance part="Q1" gate="G$1" x="-149.86" y="45.72" smashed="yes">
+<attribute name="VALUE" x="-148.59" y="45.72" size="1.778" layer="96"/>
+<attribute name="NAME" x="-158.75" y="48.26" size="1.778" layer="95"/>
+</instance>
+<instance part="R12" gate="G$1" x="-160.02" y="43.18" smashed="yes" rot="R180">
+<attribute name="NAME" x="-156.21" y="41.6814" size="1.778" layer="95" rot="R180"/>
+<attribute name="VALUE" x="-158.75" y="46.482" size="1.778" layer="96" rot="R180"/>
+</instance>
+<instance part="R13" gate="G$1" x="-147.32" y="60.96" smashed="yes" rot="R90">
+<attribute name="NAME" x="-148.8186" y="57.15" size="1.778" layer="95" rot="R90"/>
+<attribute name="VALUE" x="-143.51" y="61.722" size="1.778" layer="96" rot="R180"/>
 </instance>
 </instances>
@@
 </segment>
 <segment>
-<pinref part="R8" gate="G$1" pin="1"/>
-<wire x1="-144.78" y1="50.8" x2="-147.32" y2="50.8" width="0.1524" layer="91"/>
-<label x="-147.32" y="50.8" size="1.016" layer="95" rot="R180" xref="yes"/>
-</segment>
-<segment>
 <pinref part="U1" gate="G$1" pin="GND"/>
 <wire x1="-248.92" y1="-53.34" x2="-246.38" y2="-53.34" width="0.1524" layer="91"/>
@@
 </segment>
 <segment>
-<label x="-104.14" y="35.56" size="1.778" layer="95" xref="yes"/>
+<label x="-104.14" y="43.18" size="1.778" layer="95" xref="yes"/>
 <pinref part="CAPS1" gate="G$1" pin="C"/>
-<wire x1="-116.84" y1="35.56" x2="-104.14" y2="35.56" width="0.1524" layer="91"/>
+<wire x1="-116.84" y1="43.18" x2="-104.14" y2="43.18" width="0.1524" layer="91"/>
 </segment>
 <segment>
@@
 <wire x1="-101.6" y1="116.84" x2="-88.9" y2="116.84" width="0.1524" layer="91"/>
 </segment>
+<segment>
+<pinref part="R8" gate="G$1" pin="1"/>
+<pinref part="Q1" gate="G$1" pin="S"/>
+<wire x1="-152.4" y1="30.48" x2="-147.32" y2="30.48" width="0.1524" layer="91"/>
+<wire x1="-147.32" y1="30.48" x2="-147.32" y2="40.64" width="0.1524" layer="91"/>
+<wire x1="-147.32" y1="30.48" x2="-147.32" y2="27.94" width="0.1524" layer="91"/>
+<junction x="-147.32" y="30.48"/>
+<label x="-147.32" y="27.94" size="1.778" layer="95" rot="R180" xref="yes"/>
+</segment>
 </net>
 <net name="VCC" class="0">
@@
 </segment>
 <segment>
-<pinref part="U4" gate="G$1" pin="S"/>
-<wire x1="-134.62" y1="55.88" x2="-134.62" y2="53.34" width="0.1524" layer="91"/>
-<label x="-134.62" y="53.34" size="1.016" layer="95" rot="R180" xref="yes"/>
-</segment>
-<segment>
 <pinref part="J5" gate="G$1" pin="SCL"/>
 <wire x1="-205.74" y1="2.54" x2="-215.9" y2="2.54" width="0.1524" layer="91"/>
@@
 <wire x1="-152.4" y1="91.44" x2="-154.94" y2="91.44" width="0.1524" layer="91"/>
 <label x="-154.94" y="91.44" size="1.016" layer="95" rot="R180" xref="yes"/>
+</segment>
+<segment>
+<pinref part="R13" gate="G$1" pin="2"/>
+<wire x1="-147.32" y1="66.04" x2="-147.32" y2="68.58" width="0.1524" layer="91"/>
+<pinref part="U4" gate="G$1" pin="D"/>
+<wire x1="-147.32" y1="68.58" x2="-139.7" y2="68.58" width="0.1524" layer="91"/>
+<wire x1="-139.7" y1="68.58" x2="-139.7" y2="63.5" width="0.1524" layer="91"/>
+<wire x1="-147.32" y1="68.58" x2="-149.86" y2="68.58" width="0.1524" layer="91"/>
+<junction x="-147.32" y="68.58"/>
+<label x="-149.86" y="68.58" size="1.778" layer="95" rot="R180" xref="yes"/>
 </segment>
 </net>
@@
 <net name="POWER_PIN" class="0">
 <segment>
-<pinref part="U4" gate="G$1" pin="G"/>
-<wire x1="-142.24" y1="60.96" x2="-144.78" y2="60.96" width="0.1524" layer="91"/>
-<pinref part="R8" gate="G$1" pin="2"/>
-<wire x1="-144.78" y1="60.96" x2="-147.32" y2="60.96" width="0.1524" layer="91"/>
-<junction x="-144.78" y="60.96"/>
-<label x="-147.32" y="60.96" size="1.016" layer="95" rot="R180" xref="yes"/>
-</segment>
-<segment>
 <pinref part="U1" gate="G$1" pin="P0.05"/>
 <wire x1="-294.64" y1="15.24" x2="-297.18" y2="15.24" width="0.1524" layer="91"/>
@@
 </net>
 <net name="EXT_VCC" class="0">
-<segment>
-<pinref part="U4" gate="G$1" pin="D"/>
-<wire x1="-134.62" y1="71.12" x2="-134.62" y2="73.66" width="0.1524" layer="91"/>
-<label x="-134.62" y="73.66" size="1.016" layer="95" rot="R180" xref="yes"/>
-</segment>
 <segment>
 <pinref part="RGB1" gate="G$1" pin="VDD"/>
@@
 <segment>
 <pinref part="R11" gate="G$1" pin="1"/>
-<wire x1="-106.68" y1="27.94" x2="-104.14" y2="27.94" width="0.1524" layer="91"/>
-<label x="-104.14" y="27.94" size="1.778" layer="95" xref="yes"/>
+<wire x1="-106.68" y1="35.56" x2="-104.14" y2="35.56" width="0.1524" layer="91"/>
+<label x="-104.14" y="35.56" size="1.778" layer="95" xref="yes"/>
 </segment>
 <segment>
@@
 </segment>
 </net>
+<net name="UG_EN" class="0">
+<segment>
+<pinref part="R12" gate="G$1" pin="2"/>
+<wire x1="-165.1" y1="43.18" x2="-167.64" y2="43.18" width="0.1524" layer="91"/>
+<label x="-167.64" y="43.18" size="1.778" layer="95" rot="R180" xref="yes"/>
+</segment>
+</net>
+<net name="N$53" class="0">
+<segment>
+<pinref part="R13" gate="G$1" pin="1"/>
+<pinref part="Q1" gate="G$1" pin="D"/>
+<wire x1="-147.32" y1="55.88" x2="-147.32" y2="53.34" width="0.1524" layer="91"/>
+<pinref part="U4" gate="G$1" pin="G"/>
+<wire x1="-147.32" y1="53.34" x2="-147.32" y2="50.8" width="0.1524" layer="91"/>
+<junction x="-147.32" y="53.34"/>
+</segment>
+</net>
+<net name="UG_PWR" class="0">
+<segment>
+<pinref part="U4" gate="G$1" pin="S"/>
+<wire x1="-139.7" y1="48.26" x2="-139.7" y2="45.72" width="0.1524" layer="91"/>
+<label x="-139.7" y="45.72" size="1.778" layer="95" xref="yes"/>
+</segment>
+</net>
+<net name="N$51" class="0">
+<segment>
+<pinref part="R12" gate="G$1" pin="1"/>
+<pinref part="R12" gate="G$1" pin="1"/>
+<pinref part="Q1" gate="G$1" pin="G"/>
+<wire x1="-154.94" y1="43.18" x2="-152.4" y2="43.18" width="0.1524" layer="91"/>
+<junction x="-154.94" y="43.18"/>
+<pinref part="R8" gate="G$1" pin="2"/>
+<wire x1="-152.4" y1="43.18" x2="-152.4" y2="40.64" width="0.1524" layer="91"/>
+<junction x="-152.4" y="43.18"/>
+</segment>
+</net>

Commit message: add
Parts:
- added R15: 100, Components:RESISTOR-0805
- R12: value 100 -> (none); device Components:RESISTOR-0805 -> Components:RESISTOR-0405
Connections:
- net 1 renamed X4
- removed net N$102: 6.25U.P0, 7U.P1, D8.A
- removed net N$8: RALT.P0, RALT1.P1
- removed net POWER_PIN: U1.P0.05
- new net VBAT2: S3.O, X4.2
- new net VSS: R12.1, R6.2, U3.VCC
- new net X16: U1.P1.01
- new net X17: U1.P1.02
- new net X18: U1.P1.03
- new net X19: U1.P1.04
- new net X20: U1.P1.06
- new net X5: U1.P0.10
- net C1: now also U1.P0.29, ~.P1; no longer U1.P0.21, ~.P0
- net C10: now also U1.P0.19; no longer U1.P1.04
- net C11: now also RALT.P0, RALT1.P1, U1.P0.21; no longer U1.P1.02
- net C12: now also RWIN.P0, RWIN1.P1, U1.P0.23; no longer U1.P1.01
- net C13: now also RWIN2.P0, U1.P0.07; no longer U1.P1.03
- net C14: now also U1.P0.12; no longer U1.P1.00
- net C15: now also U1.P1.09; no longer U1.P0.22
- net C16: now also U1.P0.28
- net C2: now also 1.P1, U1.P0.30; no longer 1.P0, U1.P0.23
- net C3: now also U1.P0.02; no longer U1.P0.12
- net C4: now also U1.P0.03; no longer U1.P1.09
- net C5: now also U1.P1.10; no longer U1.P0.07
- net C6: no longer U1.P0.31
- net C7: now also 6.25U.P0, 7U.P1, U1.P0.05; no longer 6.25U.P1, 7U.P0, U1.P0.30
- net C8: now also U1.P1.00; no longer U1.P0.29
- net C9: now also U1.P0.22; no longer U1.P1.06
- net CAPS: no longer U1.P1.13
- net DN: now also X1.2; no longer X1.3
- net DP: now also X1.3; no longer X1.2
- net GND: now also X1.4; no longer X1.1
- net LED: no longer U1.P0.10
- net N$1: now also 6.25U.P1, 7U.P0, D8.A; no longer RWIN.P0, RWIN1.P1
- net N$2: now also ~.P0; no longer ~.P1
- net N$24: now also 1.P0; no longer 1.P1
- net N$51: now also R15.1; no longer R12.1
- net N1: no longer U1.P0.02
- net N2: no longer U1.P0.03
- net R1: now also U1.P1.15; no longer U1.P0.28
- net R2: now also U1.P1.13; no longer U1.P0.19
- net R3: now also U1.P1.11; no longer U1.P1.15
- net R4: now also U1.P0.31; no longer U1.P1.11
- net R5: no longer U1.P1.10
- net UG_EN: now also R15.2; no longer R12.2
- net VBAT: no longer X4.2
- net VCC: now also R12.2; no longer R6.2, U3.VCC, X4.6
- net VUSB: now also X1.1, X4.6; no longer X1.4
Other:
- moved on the sheet: 1, 6.25U, 7U, R12, ~

Commit message: add
Connections:
- net X4 renamed UG
- removed net X16: U1.P1.01
- removed net X18: U1.P1.03
- removed net X5: U1.P0.10
- net C6: now also U1.P0.05
- net C7: now also U1.P1.00; no longer U1.P0.05
- net C8: now also U1.P1.03; no longer U1.P1.00
- net R5: now also U1.P1.01
- net UG_EN: now also U1.P0.10
Changed lines of the file:
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@@
 <label x="157.48" y="121.92" size="1.27" layer="95" rot="R90" xref="yes"/>
+</segment>
+<segment>
+<pinref part="U1" gate="G$1" pin="P0.05"/>
+<wire x1="-294.64" y1="15.24" x2="-297.18" y2="15.24" width="0.1524" layer="91"/>
+<label x="-297.18" y="15.24" size="1.016" layer="95" rot="R180" xref="yes"/>
 </segment>
 </net>
@@
 </segment>
 <segment>
-<pinref part="U1" gate="G$1" pin="P0.05"/>
-<wire x1="-294.64" y1="15.24" x2="-297.18" y2="15.24" width="0.1524" layer="91"/>
-<label x="-297.18" y="15.24" size="1.016" layer="95" rot="R180" xref="yes"/>
+<pinref part="U1" gate="G$1" pin="P1.00"/>
+<wire x1="-248.92" y1="2.54" x2="-246.38" y2="2.54" width="0.1524" layer="91"/>
+<label x="-246.38" y="2.54" size="1.016" layer="95" xref="yes"/>
 </segment>
 </net>
@@
 </segment>
 <segment>
-<pinref part="U1" gate="G$1" pin="P1.00"/>
-<wire x1="-248.92" y1="2.54" x2="-246.38" y2="2.54" width="0.1524" layer="91"/>
-<label x="-246.38" y="2.54" size="1.016" layer="95" xref="yes"/>
+<pinref part="U1" gate="G$1" pin="P1.03"/>
+<wire x1="-248.92" y1="-5.08" x2="-246.38" y2="-5.08" width="0.1524" layer="91"/>
+<label x="-246.38" y="-5.08" size="1.016" layer="95" xref="yes"/>
 </segment>
 </net>
@@
 <wire x1="-335.28" y1="27.94" x2="-332.74" y2="27.94" width="0.1524" layer="91"/>
 <label x="-332.74" y="27.94" size="1.27" layer="95" xref="yes"/>
+</segment>
+<segment>
+<pinref part="U1" gate="G$1" pin="P1.01"/>
+<wire x1="-248.92" y1="0" x2="-246.38" y2="0" width="0.1524" layer="91"/>
+<label x="-246.38" y="0" size="1.016" layer="95" xref="yes"/>
 </segment>
 </net>
@@
 </segment>
 </net>
-<net name="X4" class="0">
+<net name="UG" class="0">
 <segment>
 <pinref part="U1" gate="G$1" pin="P0.09"/>
@@
 <wire x1="-167.64" y1="43.18" x2="-170.18" y2="43.18" width="0.1524" layer="91"/>
 <label x="-170.18" y="43.18" size="1.778" layer="95" rot="R180" xref="yes"/>
+</segment>
+<segment>
+<pinref part="U1" gate="G$1" pin="P0.10"/>
+<wire x1="-294.64" y1="2.54" x2="-297.18" y2="2.54" width="0.1524" layer="91"/>
+<label x="-297.18" y="2.54" size="1.016" layer="95" rot="R180" xref="yes"/>
 </segment>
 </net>
@@
 </segment>
 </net>
-<net name="X5" class="0">
-<segment>
-<pinref part="U1" gate="G$1" pin="P0.10"/>
-<wire x1="-294.64" y1="2.54" x2="-297.18" y2="2.54" width="0.1524" layer="91"/>
-<label x="-297.18" y="2.54" size="1.016" layer="95" rot="R180" xref="yes"/>
-</segment>
-</net>
-<net name="X16" class="0">
-<segment>
-<pinref part="U1" gate="G$1" pin="P1.01"/>
-<wire x1="-248.92" y1="0" x2="-246.38" y2="0" width="0.1524" layer="91"/>
-<label x="-246.38" y="0" size="1.016" layer="95" xref="yes"/>
-</segment>
-</net>
 <net name="X17" class="0">
 <segment>
@@
 </segment>
 </net>
-<net name="X18" class="0">
-<segment>
-<pinref part="U1" gate="G$1" pin="P1.03"/>
-<wire x1="-248.92" y1="-5.08" x2="-246.38" y2="-5.08" width="0.1524" layer="91"/>
-<label x="-246.38" y="-5.08" size="1.016" layer="95" xref="yes"/>
-</segment>
-</net>

Commit message: addadd
Parts:
- removed C10, C11, C12, C13, C14, C4, C5, C6, C7, C8, C9: (no value), Components:CAPACITOR-C0805
- removed RGB1, RGB10, RGB11, RGB2, RGB3, RGB4, RGB5, RGB6, RGB7, RGB8, RGB9: WS2812B, LED:WS2812B
- added C15, C16, C17, C18, C19, C20, C21, C22, C23, C24, C25, C26, C27, C28, C29: (no value), Components:CAPACITOR-0603
- added U10, U11, U12, U13, U14, U15, U16, U17, U18, U19, U20, U6, U7, U8, U9: WS2812-2020, WS2812-2020:WS2812-2020
Connections:
- removed net EXT_VCC: C10.2, C11.2, C12.2, C13.2, C14.2, C4.2, C5.2, C6.2, C7.2, C8.2, C9.2, RGB1.VDD, RGB10.VDD, RGB11.VDD, RGB2.VDD, RGB3.VDD, RGB4.VDD, RGB5.VDD, RGB6.VDD, RGB7.VDD, RGB8.VDD, RGB9.VDD
- removed net LED: RGB1.DIN
- removed net N$104: RGB10.DIN, RGB9.DOUT
- removed net N$12: RGB1.DOUT, RGB2.DIN
- removed net N$13: RGB2.DOUT, RGB3.DIN
- removed net N$14: RGB5.DOUT, RGB6.DIN
- removed net N$15: RGB6.DOUT, RGB7.DIN
- removed net N$16: RGB7.DOUT, RGB8.DIN
- removed net N$17: RGB8.DOUT, RGB9.DIN
- removed net N$19: RGB10.DOUT, RGB11.DIN
- removed net N$98: RGB3.DOUT, RGB4.DIN
- removed net N$99: RGB4.DOUT, RGB5.DIN
- new net N$102: U18.DO, U19.DI
- new net N$105: U19.DO, U20.DI
- new net N$50: U7.DO, U8.DI
- new net N$52: U8.DO, U9.DI
- new net N$61: U10.DI, U9.DO
- new net N$67: U10.DO, U11.DI
- new net N$74: U11.DO, U12.DI
- new net N$75: U12.DO, U13.DI
- new net N$76: U13.DO, U14.DI
- new net N$79: U14.DO, U15.DI
- new net N$8: U6.DO, U7.DI
- new net N$80: U15.DO, U16.DI
- new net N$81: U16.DO, U17.DI
- new net N$84: U17.DO, U18.DI
- net GND: now also C15.1, C16.1, C17.1, C18.1, C19.1, C20.1, C21.1, C22.1, C23.1, C24.1, C25.1, C26.1, C27.1, C28.1, C29.1, U10.GND, U11.GND, U12.GND, U13.GND, U14.GND, U15.GND, U16.GND, U17.GND, U18.GND, U19.GND, U20.GND, U6.GND, U7.GND, U8.GND, U9.GND; no longer C10.1, C11.1, C12.1, C13.1, C14.1, C4.1, C5.1, C6.1, C7.1, C8.1, C9.1, RGB1.GND, RGB10.GND, RGB11.GND, RGB2.GND, RGB3.GND, RGB4.GND, RGB5.GND, RGB6.GND, RGB7.GND, RGB8.GND, RGB9.GND
- net UG: now also U6.DI
- net UG_PWR: now also C15.2, C16.2, C17.2, C18.2, C19.2, C20.2, C21.2, C22.2, C23.2, C24.2, C25.2, C26.2, C27.2, C28.2, C29.2, U10.VDD, U11.VDD, U12.VDD, U13.VDD, U14.VDD, U15.VDD, U16.VDD, U17.VDD, U18.VDD, U19.VDD, U20.VDD, U6.VDD, U7.VDD, U8.VDD, U9.VDD
