File: New folder/Rable/Rable.sch (EAGLE design)
At the start: 211 parts, among them J1 TYPE-C-31-M-12, J3 I2C-HEADER, J4 I2C-HEADER, J5 I2C-HEADER, Q1 2N7002, U1 HOLYIOT-18010-NRF52840, U10 WS2812-2020, U11 WS2812-2020, U12 WS2812-2020, U13 WS2812-2020, U14 WS2812-2020, U15 WS2812-2020, U16 WS2812-2020, U17 WS2812-2020, U18 WS2812-2020, U19 WS2812-2020, U2 AP2112K-3.3TRG1, U20 WS2812-2020, U3 LTC4054, U4 AO3401, U5 AO3401, U6 WS2812-2020, U7 WS2812-2020, U8 WS2812-2020, U9 WS2812-2020, X1 SM04B-SRSS-TB, X2 BM06B-SRSS-TB, X3 BM06B-SRSS-TB, X4 BM06B-SRSS-TB

Commit message: add
Parts:
- removed CAPS1, PWR: (no value), adafruit:LED3MM
- removed J5: I2C-HEADER, Headers:I2C-HEADER
- removed R11, R14: 75R, Components:RESISTOR-0805
Connections:
- removed net CAPS: R11.1
- removed net N$11: CAPS1.A, R11.2
- removed net N$20: PWR.A, R14.2
- removed net N1: JP1.1
- removed net N2: JP1.2
- net GND: no longer CAPS1.C, J5.GND, PWR.C
- net SCL: no longer J5.SDA
- net SDA: no longer J5.VCC
- net VBAT: no longer R14.1
- net VCCNRF: no longer J5.SCL
- net X19: now also JP1.2
- net X20: now also JP1.1
Changed lines of the file:
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@@
 <part name="R8" library="Components" deviceset="RESISTOR" device="-0805" value="10k"/>
 <part name="J3" library="Headers" deviceset="I2C-HEADER" device=""/>
-<part name="R11" library="Components" deviceset="RESISTOR" device="-0805" value="75R"/>
 <part name="JP1" library="pinhead" deviceset="PINHD-1X2" device="M"/>
-<part name="PWR" library="adafruit" deviceset="LED" device="3MM"/>
-<part name="CAPS1" library="adafruit" deviceset="LED" device="3MM"/>
-<part name="J5" library="Headers" deviceset="I2C-HEADER" device=""/>
-<part name="R14" library="Components" deviceset="RESISTOR" device="-0805" value="75R"/>
 <part name="BAT1" library="adafruit" deviceset="JST_2PIN" device="-THM-RA"/>
 <part name="S3" library="SparkFun-Switches" deviceset="SWITCH-SPDT" device="-SMD-AYZ0202"/>
@@
 </instance>
 <instance part="J3" gate="G$1" x="-149.86" y="91.44" smashed="yes" rot="R180"/>
-<instance part="R11" gate="G$1" x="-111.76" y="35.56" smashed="yes" rot="R180">
-<attribute name="NAME" x="-107.95" y="34.0614" size="1.778" layer="95" rot="R180"/>
-<attribute name="VALUE" x="-107.95" y="38.862" size="1.778" layer="96" rot="R180"/>
-</instance>
 <instance part="JP1" gate="G$1" x="-114.3" y="83.82" smashed="yes">
 <attribute name="NAME" x="-120.65" y="89.535" size="1.778" layer="95"/>
 <attribute name="VALUE" x="-120.65" y="78.74" size="1.778" layer="96"/>
-</instance>
-<instance part="PWR" gate="G$1" x="-116.84" y="53.34" smashed="yes">
-<attribute name="NAME" x="-113.284" y="48.768" size="1.778" layer="95" rot="R90"/>
-<attribute name="VALUE" x="-111.125" y="48.768" size="1.778" layer="96" rot="R90"/>
-</instance>
-<instance part="CAPS1" gate="G$1" x="-116.84" y="38.1" smashed="yes" rot="R180">
-<attribute name="NAME" x="-120.396" y="42.672" size="1.778" layer="95" rot="R270"/>
-<attribute name="VALUE" x="-122.555" y="42.672" size="1.778" layer="96" rot="R270"/>
-</instance>
-<instance part="J5" gate="G$1" x="-203.2" y="2.54" smashed="yes" rot="R180"/>
-<instance part="R14" gate="G$1" x="-111.76" y="55.88" smashed="yes" rot="R180">
-<attribute name="NAME" x="-107.95" y="54.3814" size="1.778" layer="95" rot="R180"/>
-<attribute name="VALUE" x="-107.95" y="59.182" size="1.778" layer="96" rot="R180"/>
 </instance>
 <instance part="BAT1" gate="G$1" x="-165.1" y="119.38" smashed="yes">
@@
 <wire x1="-198.12" y1="30.48" x2="-195.58" y2="30.48" width="0.1524" layer="91"/>
 <label x="-195.58" y="30.48" size="1.016" layer="95" xref="yes"/>
-</segment>
-<segment>
-<label x="-104.14" y="43.18" size="1.778" layer="95" xref="yes"/>
-<pinref part="CAPS1" gate="G$1" pin="C"/>
-<wire x1="-116.84" y1="43.18" x2="-104.14" y2="43.18" width="0.1524" layer="91"/>
-</segment>
-<segment>
-<pinref part="J5" gate="G$1" pin="GND"/>
-<wire x1="-205.74" y1="5.08" x2="-208.28" y2="5.08" width="0.1524" layer="91"/>
-<label x="-208.28" y="5.08" size="1.778" layer="95" rot="R180" xref="yes"/>
-</segment>
-<segment>
-<pinref part="PWR" gate="G$1" pin="C"/>
-<wire x1="-116.84" y1="48.26" x2="-104.14" y2="48.26" width="0.1524" layer="91"/>
-<label x="-104.14" y="48.26" size="1.778" layer="95" xref="yes"/>
 </segment>
 <segment>
@@
 <label x="-276.86" y="78.74" size="1.778" layer="95" rot="R180" xref="yes"/>
 </segment>
-<segment>
-<pinref part="R14" gate="G$1" pin="1"/>
-<wire x1="-106.68" y1="55.88" x2="-104.14" y2="55.88" width="0.1524" layer="91"/>
-<label x="-104.14" y="55.88" size="1.778" layer="95" xref="yes"/>
-</segment>
 </net>
 <net name="N$87" class="0">
@@
 <wire x1="-248.92" y1="25.4" x2="-246.38" y2="25.4" width="0.1524" layer="91"/>
 <label x="-246.38" y="25.4" size="1.016" layer="95" xref="yes"/>
-</segment>
-<segment>
-<pinref part="J5" gate="G$1" pin="SCL"/>
-<wire x1="-205.74" y1="2.54" x2="-215.9" y2="2.54" width="0.1524" layer="91"/>
-<label x="-215.9" y="2.54" size="1.778" layer="95" rot="R180" xref="yes"/>
 </segment>
 <segment>
@@
 </segment>
 </net>
-<net name="CAPS" class="0">
-<segment>
-<pinref part="R11" gate="G$1" pin="1"/>
-<wire x1="-106.68" y1="35.56" x2="-104.14" y2="35.56" width="0.1524" layer="91"/>
-<label x="-104.14" y="35.56" size="1.778" layer="95" xref="yes"/>
-</segment>
-</net>
 <net name="CLK" class="0">
 <segment>
@@
 </segment>
 </net>
-<net name="N$11" class="0">
-<segment>
-<pinref part="R11" gate="G$1" pin="2"/>
-<pinref part="CAPS1" gate="G$1" pin="A"/>
-</segment>
-</net>
-<net name="N1" class="0">
-<segment>
-<pinref part="JP1" gate="G$1" pin="1"/>
-<wire x1="-116.84" y1="86.36" x2="-121.92" y2="86.36" width="0.1524" layer="91"/>
-<label x="-121.92" y="86.36" size="1.016" layer="95" rot="R180" xref="yes"/>
-</segment>
-</net>
-<net name="N2" class="0">
-<segment>
-<pinref part="JP1" gate="G$1" pin="2"/>
-<wire x1="-116.84" y1="83.82" x2="-121.92" y2="83.82" width="0.1524" layer="91"/>
-<label x="-121.92" y="83.82" size="1.016" layer="95" rot="R180" xref="yes"/>
-</segment>
-</net>
 <net name="SDA" class="0">
 <segment>
@@
 <label x="-297.18" y="-10.16" size="1.016" layer="95" rot="R180" xref="yes"/>
 </segment>
-<segment>
-<pinref part="J5" gate="G$1" pin="VCC"/>
-<wire x1="-205.74" y1="-2.54" x2="-215.9" y2="-2.54" width="0.1524" layer="91"/>
-<label x="-215.9" y="-2.54" size="1.778" layer="95" rot="R180" xref="yes"/>
-</segment>
 </net>
 <net name="SCL" class="0">
@@
 <label x="-297.18" y="-15.24" size="1.016" layer="95" rot="R180" xref="yes"/>
 </segment>
-<segment>
-<pinref part="J5" gate="G$1" pin="SDA"/>
-<wire x1="-205.74" y1="0" x2="-208.28" y2="0" width="0.1524" layer="91"/>
-<label x="-208.28" y="0" size="1.778" layer="95" rot="R180" xref="yes"/>
-</segment>
 </net>
 <net name="UG" class="0">
@@
 <wire x1="-304.8" y1="200.66" x2="-307.34" y2="200.66" width="0.1524" layer="91"/>
 <label x="-307.34" y="200.66" size="1.778" layer="95" rot="R180" xref="yes"/>
-</segment>
-</net>
-<net name="N$20" class="0">
-<segment>
-<pinref part="R14" gate="G$1" pin="2"/>
-<pinref part="PWR" gate="G$1" pin="A"/>
 </segment>
 </net>
@@
 <label x="-246.38" y="-7.62" size="1.016" layer="95" xref="yes"/>
 </segment>
+<segment>
+<pinref part="JP1" gate="G$1" pin="2"/>
+<wire x1="-116.84" y1="83.82" x2="-121.92" y2="83.82" width="0.1524" layer="91"/>
+<label x="-121.92" y="83.82" size="1.016" layer="95" rot="R180" xref="yes"/>
+</segment>
 </net>
 <net name="X20" class="0">
@@
 <label x="-246.38" y="-12.7" size="1.016" layer="95" xref="yes"/>
 </segment>
-</net>
+<segment>
+<pinref part="JP1" gate="G$1" pin="1"/>
+<wire x1="-116.84" y1="86.36" x2="-121.92" y2="86.36" width="0.1524" layer="91"/>
+<label x="-121.92" y="86.36" size="1.016" layer="95" rot="R180" xref="yes"/>
+</segment>
+</net>

Commit message: add
Parts:
- renumbered BAT1 to BAT, BAT2 to CHG, R12 to HERE
Changed lines of the file:
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@@
 <part name="J3" library="Headers" deviceset="I2C-HEADER" device=""/>
 <part name="JP1" library="pinhead" deviceset="PINHD-1X2" device="M"/>
-<part name="BAT1" library="adafruit" deviceset="JST_2PIN" device="-THM-RA"/>
+<part name="BAT" library="adafruit" deviceset="JST_2PIN" device="-THM-RA"/>
 <part name="S3" library="SparkFun-Switches" deviceset="SWITCH-SPDT" device="-SMD-AYZ0202"/>
 <part name="X4" library="con-JST SH" deviceset="BM06B-SRSS" device="-TB"/>
-<part name="BAT2" library="adafruit" deviceset="JST_2PIN" device="-THM-RA"/>
+<part name="CHG" library="adafruit" deviceset="JST_2PIN" device="-THM-RA"/>
 <part name="LED1" library="adafruit" deviceset="LED" device="CHIPLED_1206"/>
 <part name="Q1" library="2N7002" deviceset="2N7002" device=""/>
 <part name="R15" library="Components" deviceset="RESISTOR" device="-0805" value="100"/>
 <part name="R13" library="Components" deviceset="RESISTOR" device="-0805" value="10k"/>
-<part name="R12" library="Components" deviceset="RESISTOR" device="-0405"/>
+<part name="HERE" library="Components" deviceset="RESISTOR" device="-0405"/>
 <part name="U6" library="WS2812-2020" deviceset="WS2812-2020" device=""/>
 <part name="U7" library="WS2812-2020" deviceset="WS2812-2020" device=""/>
@@
 <attribute name="VALUE" x="-120.65" y="78.74" size="1.778" layer="96"/>
 </instance>
-<instance part="BAT1" gate="G$1" x="-165.1" y="119.38" smashed="yes">
+<instance part="BAT" gate="G$1" x="-165.1" y="119.38" smashed="yes">
 <attribute name="NAME" x="-171.45" y="125.095" size="1.778" layer="95"/>
 <attribute name="VALUE" x="-171.45" y="114.3" size="1.778" layer="96"/>
@@
 <attribute name="NAME" x="-97.79" y="127.762" size="1.778" layer="95"/>
 </instance>
-<instance part="BAT2" gate="G$1" x="-127" y="101.6" smashed="yes" rot="R180">
+<instance part="CHG" gate="G$1" x="-127" y="101.6" smashed="yes" rot="R180">
 <attribute name="NAME" x="-120.65" y="95.885" size="1.778" layer="95" rot="R180"/>
 <attribute name="VALUE" x="-120.65" y="106.68" size="1.778" layer="96" rot="R180"/>
@@
 <attribute name="VALUE" x="-143.51" y="61.722" size="1.778" layer="96" rot="R180"/>
 </instance>
-<instance part="R12" gate="G$1" x="-193.04" y="81.28" smashed="yes">
+<instance part="HERE" gate="G$1" x="-193.04" y="81.28" smashed="yes">
 <attribute name="NAME" x="-196.85" y="82.7786" size="1.778" layer="95"/>
 <attribute name="VALUE" x="-196.85" y="77.978" size="1.778" layer="96"/>
@@
 <wire x1="-152.4" y1="121.92" x2="-152.4" y2="109.22" width="0.1524" layer="91"/>
 <wire x1="-152.4" y1="109.22" x2="-157.48" y2="109.22" width="0.1524" layer="91"/>
-<pinref part="BAT1" gate="G$1" pin="1"/>
+<pinref part="BAT" gate="G$1" pin="1"/>
 </segment>
 <segment>
@@
 <segment>
 <label x="-119.38" y="99.06" size="1.016" layer="95" xref="yes"/>
-<pinref part="BAT2" gate="G$1" pin="1"/>
+<pinref part="CHG" gate="G$1" pin="1"/>
 <wire x1="-124.46" y1="99.06" x2="-119.38" y2="99.06" width="0.1524" layer="91"/>
 </segment>
@@
 </segment>
 <segment>
-<pinref part="R12" gate="G$1" pin="2"/>
+<pinref part="HERE" gate="G$1" pin="2"/>
 <wire x1="-187.96" y1="81.28" x2="-185.42" y2="81.28" width="0.1524" layer="91"/>
 <label x="-185.42" y="81.28" size="1.778" layer="95" xref="yes"/>
@@
 <segment>
 <label x="-119.38" y="101.6" size="1.016" layer="95" xref="yes"/>
-<pinref part="BAT2" gate="G$1" pin="2"/>
+<pinref part="CHG" gate="G$1" pin="2"/>
 <wire x1="-124.46" y1="101.6" x2="-119.38" y2="101.6" width="0.1524" layer="91"/>
 </segment>
@@
 <net name="N$82" class="0">
 <segment>
-<pinref part="BAT1" gate="G$1" pin="2"/>
+<pinref part="BAT" gate="G$1" pin="2"/>
 <pinref part="S3" gate="1" pin="S"/>
 <wire x1="-185.42" y1="119.38" x2="-167.64" y2="119.38" width="0.1524" layer="91"/>
@@
 <wire x1="-208.28" y1="81.28" x2="-198.12" y2="81.28" width="0.1524" layer="91"/>
 <wire x1="-198.12" y1="81.28" x2="-198.12" y2="76.2" width="0.1524" layer="91"/>
-<pinref part="R12" gate="G$1" pin="1"/>
+<pinref part="HERE" gate="G$1" pin="1"/>
 <junction x="-198.12" y="81.28"/>
 </segment>

Commit message: add
Parts:
- removed C15, C16, C17, C18, C19, C20, C21, C22, C23, C24, C25, C26, C27, C28, C29: (no value), Components:CAPACITOR-0603
- removed RALT: KEYSWITCH-PLAIN-MXHSPCB-1U, Keyboard:KEYSWITCH-PLAIN-MXHSPCB-1U
- removed U10, U11, U12, U13, U14, U15, U16, U17, U18, U19, U20, U6, U7, U8, U9: WS2812-2020, WS2812-2020:WS2812-2020
- added =1, =2, =3, =4, =5, RWIN3, TAB1, TAB2, TAB3, TAB4, ~1: KEYSWITCH-PLAIN-MXHSPCB-1U, Keyboard:KEYSWITCH-PLAIN-MXHSPCB-1U
- added D64: (no value), Components:DIODE-SOD-123
- 7U: value KEYSWITCH-PLAIN-MXHSPCB-7U-FLIPPED -> KEYSWITCH-PLAIN-MXHSPCB-7U; device Keyboard:KEYSWITCH-PLAIN-MXHSPCB-7U-FLIPPED -> Keyboard:KEYSWITCH-PLAIN-MXHSPCB-7U
- RSHIFT1: value KEYSWITCH-PLAIN-MXHSPCB-2U -> KEYSWITCH-PLAIN-MXHSPCB-2U-FLIPPED; device Keyboard:KEYSWITCH-PLAIN-MXHSPCB-2U -> Keyboard:KEYSWITCH-PLAIN-MXHSPCB-2U-FLIPPED
Connections:
- net X17 renamed 17
- removed net N$102: U18.DO, U19.DI
- removed net N$105: U19.DO, U20.DI
- removed net N$50: U7.DO, U8.DI
- removed net N$52: U8.DO, U9.DI
- removed net N$61: U10.DI, U9.DO
- removed net N$67: U10.DO, U11.DI
- removed net N$68: D14.A, RSHIFT1.P1, RSHIFT2.P0
- removed net N$74: U11.DO, U12.DI
- removed net N$75: U12.DO, U13.DI
- removed net N$76: U13.DO, U14.DI
- removed net N$79: U14.DO, U15.DI
- removed net N$80: U15.DO, U16.DI
- removed net N$81: U16.DO, U17.DI
- removed net N$84: U17.DO, U18.DI
- new net 01: U1.P0.02
- new net 010: U1.P0.23
- new net 011: U1.P0.28
- new net 012: U1.P0.29
- new net 013: U1.P0.30
- new net 014: U1.P0.31
- new net 02: U1.P0.03
- new net 03: U1.P0.04
- new net 04: U1.P0.05
- new net 05: U1.P0.07
- new net 06: U1.P0.12
- new net 07: U1.P0.19
- new net 08: U1.P0.21
- new net 09: U1.P0.22
- new net 15: U1.P1.00
- new net 16: U1.P1.01
- new net 18: U1.P1.03
- new net 19: U1.P1.04
- new net 20: U1.P1.06
- new net 21: U1.P1.09
- new net 22: U1.P1.10
- new net 23: U1.P1.11
- new net 24: U1.P1.13
- new net 25: U1.P1.15
- new net N$11: D64.A, RWIN2.P1, RWIN3.P0
- net BAT_PIN: no longer U1.P0.04
- net C1: no longer U1.P0.29
- net C10: no longer U1.P0.19
- net C11: now also RALT1.P0; no longer RALT.P0, RALT1.P1, U1.P0.21
- net C12: no longer U1.P0.23
- net C13: now also RSHIFT1.P1, RSHIFT2.P0, RWIN3.P1; no longer RSHIFT1.P0, RSHIFT2.P1, U1.P0.07
- net C14: no longer U1.P0.12
- net C15: now also =1.P0, =2.P0, =3.P0, =4.P0, =5.P0; no longer U1.P1.09
- net C16: now also TAB1.P0, TAB2.P0, TAB3.P0, TAB4.P0, ~1.P0; no longer U1.P0.28
- net C2: no longer U1.P0.30
- net C3: no longer U1.P0.02
- net C4: no longer U1.P0.03
- net C5: no longer U1.P1.10
- net C6: no longer U1.P0.05
- net C7: no longer U1.P1.00
- net C8: no longer U1.P1.03
- net C9: no longer U1.P0.22
- net GND: no longer C15.1, C16.1, C17.1, C18.1, C19.1, C20.1, C21.1, C22.1, C23.1, C24.1, C25.1, C26.1, C27.1, C28.1, C29.1, U10.GND, U11.GND, U12.GND, U13.GND, U14.GND, U15.GND, U16.GND, U17.GND, U18.GND, U19.GND, U20.GND, U6.GND, U7.GND, U8.GND, U9.GND
- net N$22: now also RALT1.P1; no longer RALT.P1, RALT1.P0
- net N$8: now also D14.A, RSHIFT1.P0, RSHIFT2.P1; no longer U6.DO, U7.DI
- net R1: no longer U1.P1.15
- net R2: no longer U1.P1.13
- net R3: no longer U1.P1.11
- net R4: no longer U1.P0.31
- net R5: now also D64.C; no longer U1.P1.01
- net UG: no longer U6.DI
- net UG_PWR: no longer C15.2, C16.2, C17.2, C18.2, C19.2, C20.2, C21.2, C22.2, C23.2, C24.2, C25.2, C26.2, C27.2, C28.2, C29.2, U10.VDD, U11.VDD, U12.VDD, U13.VDD, U14.VDD, U15.VDD, U16.VDD, U17.VDD, U18.VDD, U19.VDD, U20.VDD, U6.VDD, U7.VDD, U8.VDD, U9.VDD
- net X19: no longer U1.P1.04
- net X20: no longer U1.P1.06
Other:
- moved on the sheet: RALT1, RSHIFT1, RSHIFT2
