File: New folder/Rable/Rable.sch (EAGLE design)
At the start: 187 parts, among them J1 TYPE-C-31-M-12, J3 I2C-HEADER, J4 I2C-HEADER, Q1 2N7002, U1 HOLYIOT-18010-NRF52840, U2 AP2112K-3.3TRG1, U3 LTC4054, U4 AO3401, U5 AO3401, X1 SM04B-SRSS-TB, X2 BM06B-SRSS-TB, X3 BM06B-SRSS-TB, X4 BM06B-SRSS-TB

Commit message: add
Connections:
- removed net N$100: D11.A, LWIN.P1, LWIN1.P0
- removed net N$101: D10.A, LALT.P1, LALT1.P0
- removed net N$86: D13.A, FN.P0
- new net N$12: D11.A, LWIN.P0, LWIN1.P1
- new net N$13: D10.A, LALT.P0, LALT1.P1
- new net N$14: D13.A, FN.P1
- net C1: now also LCTRL.P1, LCTRL1.P0; no longer LCTRL.P0, LCTRL1.P1
- net C14: now also FN.P0; no longer FN.P1
- net C2: now also LWIN.P1, LWIN1.P0; no longer LWIN.P0, LWIN1.P1
- net C3: now also LALT.P1, LALT1.P0; no longer LALT.P0, LALT1.P1
- net N$6: now also LCTRL.P0, LCTRL1.P1; no longer LCTRL.P1, LCTRL1.P0
Other:
- moved on the sheet: FN, LALT, LALT1, LCTRL, LCTRL1, LWIN, LWIN1

Commit message: add
Parts:
- added D65, D66, D67, D68, D69, D70, D71, D72, D73, D74: (no value), Components:DIODE-SOD-123
- added X5, X6: BM02B-SRSS-TB, con-JST SH:BM02B-SRSS-TB
Connections:
- new net N$15: D65.A, ~1.P1
- new net N$16: D66.A, TAB1.P1
- new net N$17: D67.A, TAB2.P1
- new net N$19: D68.A, TAB3.P1
- new net N$20: D69.A, TAB4.P1
- new net N$21: =1.P1, D70.A
- new net N$23: =2.P1, D71.A
- new net N$35: =3.P1, D72.A
- new net N$37: =4.P1, D73.A
- new net N$47: =5.P1, D74.A
- net GND: now also X4.1, X5.1, X6.1
- net N$82: now also X6.2
- net R1: now also D65.C
- net R2: now also D66.C
- net R3: now also D67.C
- net R4: now also D68.C
- net R5: now also D69.C
- net VUSB: now also X5.2

Commit message: add
Parts:
- added HERE1: (no value), Components:RESISTOR-0405
- added R17: 22R, Components:RESISTOR-0805
- added U10, U11, U12, U13, U14, U15, U16, U17, U18, U19, U20, U21, U22, U23, U6, U7, U8, U9: WS2812-2020, WS2812-2020:WS2812-2020
- added X7, X8: BM06B-SRSS-TB, con-JST SH:BM06B-SRSS-TB
Connections:
- removed net 01: U1.P0.02
- removed net 010: U1.P0.23
- removed net 011: U1.P0.28
- removed net 012: U1.P0.29
- removed net 013: U1.P0.30
- removed net 014: U1.P0.31
- removed net 02: U1.P0.03
- removed net 03: U1.P0.04
- removed net 04: U1.P0.05
- removed net 05: U1.P0.07
- removed net 06: U1.P0.12
- removed net 07: U1.P0.19
- removed net 08: U1.P0.21
- removed net 09: U1.P0.22
- removed net 15: U1.P1.00
- removed net 16: U1.P1.01
- removed net 18: U1.P1.03
- removed net 21: U1.P1.09
- removed net 22: U1.P1.10
- removed net 23: U1.P1.11
- removed net 24: U1.P1.13
- removed net 25: U1.P1.15
- new net N$102: U10.DI, U9.DO
- new net N$104: U10.DO, U11.DI
- new net N$105: U11.DO, U12.DI
- new net N$106: U12.DO, U13.DI
- new net N$107: U13.DO, U14.DI
- new net N$108: U14.DO, U15.DI
- new net N$109: U15.DO, U16.DI
- new net N$110: U16.DO, U17.DI
- new net N$111: U17.DO, U18.DI
- new net N$112: U18.DO, U19.DI
- new net N$113: U19.DO, U20.DI
- new net N$114: U20.DO, U21.DI
- new net N$115: U21.DO, U22.DI
- new net N$116: U22.DO, U23.DI
- new net N$117: R17.2, U8.DI
- new net N$80: U6.DO, U7.DI
- new net N$81: U23.DO, U6.DI
- new net N$98: U8.DO, U9.DI
- net BAT_PIN: now also U1.P0.05
- net C1: now also U1.P0.30
- net C10: now also U1.P0.19
- net C11: now also U1.P0.21
- net C12: now also U1.P0.23
- net C13: now also U1.P0.12
- net C14: now also U1.P1.09
- net C15: now also U1.P0.07, X8.1
- net C16: now also U1.P0.29, X7.1
- net C2: now also U1.P0.31
- net C3: now also U1.P0.28
- net C4: now also U1.P0.02
- net C5: now also U1.P1.11
- net C6: now also U1.P0.03
- net C7: now also U1.P0.22
- net C8: now also U1.P1.03
- net C9: now also U1.P1.00
- net GND: now also U10.GND, U11.GND, U12.GND, U13.GND, U14.GND, U15.GND, U16.GND, U17.GND, U18.GND, U19.GND, U20.GND, U21.GND, U22.GND, U23.GND, U6.GND, U7.GND, U8.GND, U9.GND
- net R1: now also D70.C, U1.P1.10, X7.6, X8.6
- net R2: now also D71.C, U1.P1.13, X7.5, X8.5
- net R3: now also D72.C, U1.P1.15, X7.4, X8.4
- net R4: now also D73.C, U1.P0.04, X7.3, X8.3
- net R5: now also D74.C, U1.P1.01, X7.2, X8.2
- net UG: now also R17.1
- net UG_PWR: now also U10.VDD, U11.VDD, U12.VDD, U13.VDD, U14.VDD, U15.VDD, U16.VDD, U17.VDD, U18.VDD, U19.VDD, U20.VDD, U21.VDD, U22.VDD, U23.VDD, U6.VDD, U7.VDD, U8.VDD, U9.VDD
- net VBAT: now also HERE1.2
- net VBAT2: now also HERE1.1

Commit message: add
Parts:
- renumbered HERE to USB_INT, HERE1 to USB_EXT, LED1 to LED_CHG
Changed lines of the file:
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@@
 <part name="X4" library="con-JST SH" deviceset="BM06B-SRSS" device="-TB"/>
 <part name="CHG" library="adafruit" deviceset="JST_2PIN" device="-THM-RA"/>
-<part name="LED1" library="adafruit" deviceset="LED" device="CHIPLED_1206"/>
+<part name="LED_CHG" library="adafruit" deviceset="LED" device="CHIPLED_1206"/>
 <part name="Q1" library="2N7002" deviceset="2N7002" device=""/>
 <part name="R15" library="Components" deviceset="RESISTOR" device="-0805" value="100"/>
 <part name="R13" library="Components" deviceset="RESISTOR" device="-0805" value="10k"/>
-<part name="HERE" library="Components" deviceset="RESISTOR" device="-0405"/>
+<part name="USB_INT" library="Components" deviceset="RESISTOR" device="-0405"/>
 <part name="RWIN3" library="Keyboard" deviceset="KEYSWITCH-PLAIN" device="-MXHSPCB-1U" value="KEYSWITCH-PLAIN-MXHSPCB-1U"/>
 <part name="D64" library="Components" deviceset="DIODE" device="-SOD-123"/>
@@
 <part name="X7" library="con-JST SH" deviceset="BM06B-SRSS" device="-TB"/>
 <part name="X8" library="con-JST SH" deviceset="BM06B-SRSS" device="-TB"/>
-<part name="HERE1" library="Components" deviceset="RESISTOR" device="-0405"/>
+<part name="USB_EXT" library="Components" deviceset="RESISTOR" device="-0405"/>
 </parts>
 <sheets>
@@
 <attribute name="VALUE" x="-120.65" y="106.68" size="1.778" layer="96" rot="R180"/>
 </instance>
-<instance part="LED1" gate="G$1" x="-208.28" y="68.58" smashed="yes">
+<instance part="LED_CHG" gate="G$1" x="-208.28" y="68.58" smashed="yes">
 <attribute name="NAME" x="-204.724" y="66.548" size="1.778" layer="95" rot="R90"/>
 <attribute name="VALUE" x="-202.565" y="64.008" size="1.778" layer="96" rot="R90"/>
@@
 <attribute name="VALUE" x="-143.51" y="61.722" size="1.778" layer="96" rot="R180"/>
 </instance>
-<instance part="HERE" gate="G$1" x="-193.04" y="81.28" smashed="yes">
+<instance part="USB_INT" gate="G$1" x="-193.04" y="81.28" smashed="yes">
 <attribute name="NAME" x="-196.85" y="82.7786" size="1.778" layer="95"/>
 <attribute name="VALUE" x="-196.85" y="77.978" size="1.778" layer="96"/>
@@
 <attribute name="NAME" x="-344.17" y="18.542" size="1.778" layer="95"/>
 </instance>
-<instance part="HERE1" gate="G$1" x="-190.5" y="116.84" smashed="yes" rot="R90">
+<instance part="USB_EXT" gate="G$1" x="-190.5" y="116.84" smashed="yes" rot="R90">
 <attribute name="NAME" x="-191.9986" y="113.03" size="1.778" layer="95" rot="R90"/>
 <attribute name="VALUE" x="-187.198" y="113.03" size="1.778" layer="96" rot="R90"/>
@@
 </segment>
 <segment>
-<pinref part="HERE" gate="G$1" pin="2"/>
+<pinref part="USB_INT" gate="G$1" pin="2"/>
 <wire x1="-187.96" y1="81.28" x2="-185.42" y2="81.28" width="0.1524" layer="91"/>
 <label x="-185.42" y="81.28" size="1.778" layer="95" xref="yes"/>
@@
 <wire x1="-177.8" y1="116.84" x2="-177.8" y2="109.22" width="0.1524" layer="91"/>
 <pinref part="S3" gate="1" pin="P"/>
-<pinref part="HERE1" gate="G$1" pin="2"/>
+<pinref part="USB_EXT" gate="G$1" pin="2"/>
 <wire x1="-190.5" y1="121.92" x2="-190.5" y2="116.84" width="0.1524" layer="91"/>
 <wire x1="-190.5" y1="116.84" x2="-177.8" y2="116.84" width="0.1524" layer="91"/>
@@
 <segment>
 <pinref part="U3" gate="G$1" pin="CHRG"/>
-<pinref part="LED1" gate="G$1" pin="C"/>
+<pinref part="LED_CHG" gate="G$1" pin="C"/>
 </segment>
 </net>
@@
 <segment>
 <pinref part="R6" gate="G$1" pin="1"/>
-<pinref part="LED1" gate="G$1" pin="A"/>
+<pinref part="LED_CHG" gate="G$1" pin="A"/>
 </segment>
 </net>
@@
 <wire x1="-185.42" y1="114.3" x2="-175.26" y2="114.3" width="0.1524" layer="91"/>
 <label x="-175.26" y="114.3" size="1.778" layer="95" xref="yes"/>
-<pinref part="HERE1" gate="G$1" pin="1"/>
+<pinref part="USB_EXT" gate="G$1" pin="1"/>
 <wire x1="-190.5" y1="111.76" x2="-190.5" y2="114.3" width="0.1524" layer="91"/>
 <wire x1="-190.5" y1="114.3" x2="-185.42" y2="114.3" width="0.1524" layer="91"/>
@@
 <wire x1="-208.28" y1="81.28" x2="-198.12" y2="81.28" width="0.1524" layer="91"/>
 <wire x1="-198.12" y1="81.28" x2="-198.12" y2="76.2" width="0.1524" layer="91"/>
-<pinref part="HERE" gate="G$1" pin="1"/>
+<pinref part="USB_INT" gate="G$1" pin="1"/>
 <junction x="-198.12" y="81.28"/>
 </segment>

Commit message: add
Connections:
- removed net X19: JP1.2
- removed net X20: JP1.1
- net 19: now also JP1.2
- net 20: now also JP1.1
Changed lines of the file:
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@@
-</segment>
-</net>
-<net name="X19" class="0">
-<segment>
-<pinref part="JP1" gate="G$1" pin="2"/>
-<wire x1="-116.84" y1="83.82" x2="-121.92" y2="83.82" width="0.1524" layer="91"/>
-<label x="-121.92" y="83.82" size="1.016" layer="95" rot="R180" xref="yes"/>
-<wire x1="-119.38" y1="83.82" x2="-116.84" y2="83.82" width="0.1524" layer="91"/>
-</segment>
-</net>
-<net name="X20" class="0">
-<segment>
-<pinref part="JP1" gate="G$1" pin="1"/>
-<wire x1="-116.84" y1="86.36" x2="-121.92" y2="86.36" width="0.1524" layer="91"/>
-<label x="-121.92" y="86.36" size="1.016" layer="95" rot="R180" xref="yes"/>
 </segment>
 </net>
@@
 <label x="-246.38" y="-7.62" size="1.016" layer="95" xref="yes"/>
 </segment>
+<segment>
+<pinref part="JP1" gate="G$1" pin="2"/>
+<wire x1="-116.84" y1="83.82" x2="-121.92" y2="83.82" width="0.1524" layer="91"/>
+<label x="-121.92" y="83.82" size="1.016" layer="95" rot="R180" xref="yes"/>
+<wire x1="-119.38" y1="83.82" x2="-116.84" y2="83.82" width="0.1524" layer="91"/>
+</segment>
 </net>
 <net name="20" class="0">
@@
 <label x="-246.38" y="-12.7" size="1.016" layer="95" xref="yes"/>
 </segment>
+<segment>
+<pinref part="JP1" gate="G$1" pin="1"/>
+<wire x1="-116.84" y1="86.36" x2="-121.92" y2="86.36" width="0.1524" layer="91"/>
+<label x="-121.92" y="86.36" size="1.016" layer="95" rot="R180" xref="yes"/>
+</segment>
 </net>

Commit message: add
Parts:
- removed R17: 22R, Components:RESISTOR-0805
- removed U3: LTC4054, LTC4054:LTC4054
- added Q5: 2N7002, 2N7002:2N7002
- added R11: 10k, Components:RESISTOR-0805
- Q1: value 2N7002 -> LTC4054; device 2N7002:2N7002 -> LTC4054:LTC4054
- R10: value 2M -> 10k
- R13: value 10k -> 330
- R5: value 10k -> 1k
- R6: value 1k -> 10k/2k
- R7: value 10k/2k -> 10k
- R8: value 10k -> 2M
- renumbered R15 to R12, U10 to RGB3, U11 to RGB4, U12 to RGB5, U13 to RGB6, U14 to RGB7, U15 to RGB8, U16 to RGB9, U17 to RGB10, U18 to RGB11, U19 to RGB12, U2 to Q3, U20 to RGB13, U21 to RGB14, U22 to RGB15, U23 to RGB16, U4 to Q4, U5 to Q2, U6 to RGB17, U7 to RGB18, U8 to RGB1, U9 to RGB2
Connections:
- net BAT_PIN: now also R8.1; no longer R10.1
- net GND: now also Q1.GND, Q5.S, R11.1, R6.1, R8.2; no longer Q1.S, R10.2, R5.1, R8.1, U3.GND
- net N$117: now also R13.2; no longer R17.2
- net N$51: now also Q5.G, R11.2; no longer Q1.G, R8.2
- net N$53: now also Q5.D, R10.1; no longer Q1.D, R13.1
- net N$7: now also Q1.CHRG; no longer U3.CHRG
- net N$87: now also Q1.PROG, R6.2; no longer R7.2, U3.PROG
- net N$9: now also R5.1; no longer R6.1
- net UG: now also R13.1; no longer R17.1
- net VBAT: now also Q1.BAT; no longer U3.BAT
- net VCC: now also R7.2; no longer R5.2
- net VCCNRF: now also R10.2; no longer R13.2
- net VSS: now also Q1.VCC, R5.2; no longer R6.2, U3.VCC
Other:
- moved on the sheet: R10, R13, R5, R6, R7, R8
