File: New folder/40/40ish.brd (EAGLE design)
At the start: 247.6 x 95.2 mm, 80 parts

Commit message: add
Parts:
- moved D4 4.76 mm to (38.1, 108.9)
- moved D3 2.38 mm to (31.0, 128.0)
Other:
- outline, holes or cut-outs redrawn
