File: New folder/4x4/4x4.brd (EAGLE design)
At the start: 81 x 97.6 mm, 74 parts, among them J1 TYPE-C-31-M-12, U1 W25Q128JVSIQ, U3 RP2040, U4 PMIC-LDO-XC6206P332MR-G(SOT23), U5 SL2.1A, X4 USB-A-H, X5 USB-A-H, X6 BM04B-SRSS-TB

Commit message: add
Parts:
- moved JP4 25.3 mm to (46.4, -0.60)
- moved BOOT 25.3 mm to (35.7, -0.60)
- moved R5 25.3 mm to (23.8, -19.1)
- moved U1 4.33 mm to (47.6, 91.1), flipped to the top, turned to 180 degrees
- moved C3 2.45 mm to (33.3, 99.4), flipped to the bottom, turned to 90 degrees
- moved C9 2.45 mm to (36.9, 99.4), flipped to the bottom, turned to 90 degrees
- moved C12 2.38 mm to (40.5, 96.4), turned to 180 degrees
- moved C8 1.88 mm to (36.3, 102.4), flipped to the bottom
- moved C2 1.88 mm to (38.1, 102.4), flipped to the bottom
- moved C7 1.33 mm to (39.3, 94.7), flipped to the bottom
- moved U3 1.19 mm to (34.5, 95.2), flipped to the top, turned to 270 degrees
- moved C4 1.19 mm to (40.5, 98.2), flipped to the bottom
- moved C6 1.19 mm to (27.4, 99.4), flipped to the bottom
Routing:
- net 3.3V: track 86.8 -> 0.00 mm, vias 10 -> 0
- net 1V: track 41.2 -> 0.00 mm, vias 3 -> 0
- net N$18: track 37.7 -> 0.00 mm, vias 3 -> 0
- net N$17: track 35.7 -> 0.00 mm, vias 3 -> 0
- net GND2: track 29.4 -> 0.00 mm
- net GND: track 20.3 -> 0.00 mm, vias 1 -> 0
- net N$24: track 19.9 -> 0.00 mm
- net SD1: track 19.7 -> 0.00 mm
- net VCC: track 19.6 -> 0.00 mm, vias 2 -> 0
- net N$7: track 19.5 -> 0.00 mm, vias 2 -> 0
- net N$23: track 18.1 -> 0.00 mm
- net XTAL2: track 17.2 -> 0.00 mm
- net SD2: track 16.4 -> 0.00 mm
- net SS: track 15.1 -> 0.00 mm
- net N$22: track 13.6 -> 0.00 mm
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Other:
- outline, holes or cut-outs redrawn

Commit message: add
Parts:
- removed C22, C23: (no value), Components:C0805
- removed U3: RP2040, RP2040:QFN40P700X700X90-57N
- removed X6: BM04B-SRSS-TB, con-JST SH:BM04B-SRSS-TB
- added D1, D10, D11, D12, D14, D15, D16, D17, D2, D3, D4, D5, D6, D7, D8, D9: (no value), Components:SOD-123
- added J2: 1X5, adafruit:1X05-3.5MM
- added R10: (no value), Components:R0603
- added R8, R9: (no value), Components:R0402
- added U2: W25Q128JVSIQ, W25Q128JVSIQ:SOIC127P790X216-8N
- added X1: BM04B-SRSS-TB, con-JST SH:BM04B-SRSS-TB
- C21: device Components:C0805 -> Components:C0603
- R39: device Fuse:RESC3216X125N -> fuse:RESC3216X125N
- U1: value W25Q128JVSIQ -> RP2040; device W25Q128JVSIQ:SOIC127P790X216-8N -> RP2040:QFN40P700X700X90-57N
- moved R5 110.3 mm to (29.8, 91.1), flipped to the bottom, turned to 180 degrees
- moved JP4 90.9 mm to (8.93, 82.2), turned to 270 degrees
- moved BOOT 89.2 mm to (8.93, 84.5), turned to 270 degrees
- moved C21 70.5 mm to (25.0, 51.2), flipped to the bottom
- moved MT1 57.2 mm to (19.1, 78.6)
- moved MT4 57.2 mm to (76.2, 78.6)
- moved JP3 20.9 mm to (8.93, 102.7), turned to 90 degrees
- moved MT2 19.0 mm to (38.1, 78.6)
- moved MT3 19.0 mm to (57.1, 78.6)
- moved RESET 18.7 mm to (8.93, 100.3), turned to 90 degrees
- moved R1 15.1 mm to (61.9, 95.8), turned to 0 degrees
- moved R2 14.4 mm to (61.9, 97.3), turned to 0 degrees
- moved U1 14.3 mm to (33.9, 95.2), turned to 270 degrees
- moved C2 13.1 mm to (38.7, 89.3), turned to 180 degrees
- moved C8 11.9 mm to (36.3, 90.5)
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Connections:
- removed net 123: U3.41
- removed net 124: U3.40
- removed net 125: U3.39
- removed net C10: U3.7
- removed net C11: U3.6
- removed net C12: U3.5
- removed net C13: U3.3
- removed net C14: U3.2
- removed net C15: U3.29
- removed net C16: U3.34
- removed net C5: U3.14
- removed net C6: U3.13
- removed net C7: U3.12
- removed net C8: U3.11
- removed net C9: U3.8
- removed net CAPS: U3.30
- removed net GND2: C18.2, C19.2, C20.1, C21.1, C22.1, C23.1, D13.2, J1.A1B12, J1.B1A12, J1.S1, J1.S2, J1.S3, J1.S4, R6.2, R7.2, U5.12, X4.GND, X5.GND, X6.4, Y2.2, Y2.4
- removed net N$50: U3.31
- removed net N$51: U3.32
- removed net N$75: U3.38
- removed net R5: U3.28
- removed net VCC2: C21.2, C22.2, C23.2, X4.VBUS, X5.VBUS, X6.1
- removed net VDD: U$13.4, U$14.4, U$15.4, U$16.4, U$20.4, U$21.4, U$22.4, U$23.4, U$24.4
- new net 1: U1.2
- new net 10: U1.13
- new net 11: U1.14
- new net 12: U1.15
- new net 13: U1.11
- new net 4: U1.5
- new net 5: U1.6
- new net 6: U1.7
- new net 7: U1.8
- new net 8: U1.9
- new net 9: U1.12
- new net DN-: D13.4, J1.A7, J1.B7, R9.2, U5.9
- new net DN4: U5.5, X1.2
- new net DP+: D13.3, J1.A6, J1.B6, R8.2, U5.10
- new net DP4: U5.6, X1.3
- new net E11: MT1.A, U1.34
- new net E12: MT1.B, U1.35
- new net E21: MT2.A, U1.38
- new net E22: MT2.B, U1.39
- new net E31: MT3.A, U1.32
- new net E32: MT3.B, U1.31
- new net E41: MT4.A, U1.30
- new net E42: MT4.B, U1.29
- new net L: R10.1, U1.16
- new net N$31: D3.A, U$3.MX2, U$3.P$3, U$3.P$4
- new net N$32: D4.A, U$4.MX2, U$4.P$3, U$4.P$4
- new net N$33: D5.A, MT1.2
- new net N$34: D6.A, MT2.2
- new net N$35: D7.A, MT3.2
- new net N$36: D8.A, MT4.2
- new net N$37: D9.A, U$5.MX2, U$5.P$3, U$5.P$4
- new net N$38: D10.A, U$6.MX2, U$6.P$3, U$6.P$4
- new net N$39: D11.A, U$7.MX2, U$7.P$3, U$7.P$4
- new net N$40: D12.A, U$8.MX2, U$8.P$3, U$8.P$4
- new net N$41: D14.A, U$9.MX2, U$9.P$3, U$9.P$4
- new net N$42: D15.A, U$10.MX2, U$10.P$3, U$10.P$4
- new net N$43: D16.A, U$11.MX2, U$11.P$3, U$11.P$4
- new net N$44: D17.A, U$12.MX2, U$12.P$3, U$12.P$4
- net 1V: now also U1.23, U1.45, U1.50; no longer U3.23, U3.45, U3.50
- net 2: now also U1.3; no longer U3.4
- net 3: now also U1.4; no longer U3.9
- net 3.3V: now also C21.2, J2.1, U$13.4, U$14.4, U$15.4, U$16.4, U$17.4, U$18.4, U$19.4, U$20.4, U$21.4, U$22.4, U$23.4, U$24.4, U1.1, U1.10, U1.22, U1.33, U1.42, U1.43, U1.44, U1.48, U1.49, U2.8; no longer U1.8, U3.1, U3.10, U3.22, U3.33, U3.42, U3.43, U3.44, U3.48, U3.49
- net C1: now also MT1.1, U$1.MX1, U$1.P$1, U$1.P$2, U$5.MX1, U$5.P$1, U$5.P$2, U$9.MX1, U$9.P$1, U$9.P$2, U1.17; no longer U3.36
- net C2: now also MT2.1, U$10.MX1, U$10.P$1, U$10.P$2, U$2.MX1, U$2.P$1, U$2.P$2, U$6.MX1, U$6.P$1, U$6.P$2, U1.36; no longer U3.17
- net C3: now also MT3.1, U$11.MX1, U$11.P$1, U$11.P$2, U$3.MX1, U$3.P$1, U$3.P$2, U$7.MX1, U$7.P$1, U$7.P$2, U1.40; no longer U3.16
- net C4: now also MT4.1, U$12.MX1, U$12.P$1, U$12.P$2, U$4.MX1, U$4.P$1, U$4.P$2, U$8.MX1, U$8.P$1, U$8.P$2, U1.41; no longer U3.15
- net CLK: now also J2.5, U1.24; no longer U3.24
- net DIO: now also J2.4, U1.25; no longer U3.25
- net DN: now also R9.1; no longer X6.3
- net DP: now also R8.1; no longer X6.2
- net GND: now also C18.2, C19.2, C20.1, C21.1, D13.2, J1.A1B12, J1.B1A12, J1.S1, J1.S2, J1.S3, J1.S4, J2.2, MT1.COM, MT1.S1, MT1.S2, MT2.COM, MT2.S1, MT2.S2, MT3.COM, MT3.S1, MT3.S2, MT4.COM, MT4.S1, MT4.S2, R6.2, R7.2, U1.19, U1.57, U2.4, U5.12, X1.4, X4.GND, X5.GND, Y2.2, Y2.4; no longer U1.4, U3.19, U3.57
- net N$13: now also U1.46; no longer U3.46
- net N$14: now also U1.47; no longer U3.47
- net N$153: no longer D13.1
- net N$154: no longer D13.6
- net N$16: now also U2.1; no longer U1.1
- net N$17: now also D1.A, U$1.MX2, U$1.P$3, U$1.P$4; no longer D13.4, J1.A7, J1.B7, U5.9
- net N$18: now also D2.A, U$2.MX2, U$2.P$3, U$2.P$4; no longer D13.3, J1.A6, J1.B6, U5.10
- net N$27: now also U5.3; no longer U5.5
- net N$28: now also U5.4; no longer U5.6
- net R1: now also D5.C, D6.C, D7.C, D8.C, U1.37; no longer U3.35
- net R2: now also D1.C, D2.C, D3.C, D4.C, U1.18; no longer U3.37
- net R3: now also D10.C, D11.C, D12.C, D9.C, U1.27; no longer U3.18
- net R4: now also D14.C, D15.C, D16.C, D17.C, U1.28; no longer U3.27
- net RGB: now also R10.2
- net RST: now also J2.3, U1.26; no longer U3.26
- net SCLK: now also U1.52, U2.6; no longer U1.6, U3.52
- net SD0: now also U1.53, U2.5; no longer U1.5, U3.53
- net SD1: now also U1.55, U2.2; no longer U1.2, U3.55
- net SD2: now also U1.54, U2.3; no longer U1.3, U3.54
- net SD3: now also U1.51, U2.7; no longer U1.7, U3.51
- net SS: now also U1.56; no longer U3.56
- net VCC: now also X1.1, X4.VBUS, X5.VBUS; no longer U$17.4, U$18.4, U$19.4
- net XTAL1: now also U1.20; no longer U3.20
- net XTAL2: now also U1.21; no longer U3.21
Routing:
- net 3.3V: track 0.00 -> 422.1 mm, vias 0 -> 25
- net R4: track 0.00 -> 139.9 mm, vias 0 -> 1
- net GND: track 0.00 -> 126.0 mm, vias 0 -> 12
- net R3: track 0.00 -> 121.8 mm, vias 0 -> 1
- net R2: track 0.00 -> 121.4 mm, vias 0 -> 1
- net C4: track 0.00 -> 114.5 mm
- net VCC: track 0.00 -> 102.7 mm, vias 0 -> 4
- net C1: track 0.00 -> 101.7 mm
- net C3: track 0.00 -> 92.6 mm
- net R1: track 0.00 -> 82.7 mm, vias 0 -> 1
- net E42: track 0.00 -> 81.2 mm, vias 0 -> 1
- net C2: track 0.00 -> 78.6 mm
- net E41: track 0.00 -> 74.9 mm, vias 0 -> 1
- net SS: track 0.00 -> 70.9 mm, vias 0 -> 2
- net L: track 0.00 -> 67.9 mm, vias 0 -> 1
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- added copper zone on layer 1, net GND
- added copper zone on layer 16, net GND

Commit message: add
Parts:
- C21: value (none) -> 100nf
- R10: value (none) -> 330
Changed lines of the file:
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@@
 <drawing>
 <settings>
-<setting alwaysvectorfont="yes"/>
+<setting alwaysvectorfont="no"/>
 <setting verticaltext="up"/>
 </settings>
@@
 <attribute name="VALUE" x="80.3353125" y="19.05" size="1" layer="22" font="vector" ratio="13" rot="MR270" align="top-center"/>
 </element>
-<element name="R10" library="Components" package="R0603" value="" x="13.6921875" y="51.196875" smashed="yes" rot="MR180">
+<element name="R10" library="Components" package="R0603" value="330" x="13.6921875" y="51.196875" smashed="yes" rot="MR180">
 <attribute name="VALUE" x="12.8921875" y="52.846875" size="1" layer="28" ratio="13" rot="MR180"/>
 </element>
-<element name="C21" library="Components" package="C0603" value="" x="25.003125" y="51.196875" smashed="yes" rot="MR0">
+<element name="C21" library="Components" package="C0603" value="100nf" x="25.003125" y="51.196875" smashed="yes" rot="MR0">
 <attribute name="VALUE" x="25.803125" y="49.546875" size="1" layer="28" ratio="13" rot="MR0"/>
 </element>
