File: New folder/4x4/4x4.sch (EAGLE design)
At the start: 74 parts, among them J1 TYPE-C-31-M-12, U1 W25Q128JVSIQ, U3 RP2040, U4 PMIC-LDO-XC6206P332MR-G(SOT23), U5 SL2.1A, X4 USB-A-H, X5 USB-A-H, X6 BM04B-SRSS-TB

Commit message: add
Parts:
- removed C22, C23: (no value), Components:CAPACITOR-C0805
- removed U3: RP2040, RP2040:RP2040
- removed X6: BM04B-SRSS-TB, con-JST SH:BM04B-SRSS-TB
- added D1, D10, D11, D12, D14, D15, D16, D17, D2, D3, D4, D5, D6, D7, D8, D9: (no value), Components:DIODE-SOD-123
- added J2: 1X5, adafruit:1X5
- added R10: (no value), Components:RESISTOR-0603
- added R8, R9: (no value), Components:RESISTOR-0405
- added U2: W25Q128JVSIQ, W25Q128JVSIQ:W25Q128JVSIQ
- added X1: BM04B-SRSS-TB, con-JST SH:BM04B-SRSS-TB
- C21: device Components:CAPACITOR-C0805 -> Components:CAPACITOR-0603
- R39: device Fuse:0ZCJ0075AF2E -> fuse:0ZCJ0075AF2E
- U1: value W25Q128JVSIQ -> RP2040; device W25Q128JVSIQ:W25Q128JVSIQ -> RP2040:RP2040
Connections:
- removed net 123: U3.GPIO29/ADC3
- removed net 124: U3.GPIO28/ADC2
- removed net 125: U3.GPIO27/ADC1
- removed net C10: U3.GPIO5
- removed net C11: U3.GPIO4
- removed net C12: U3.GPIO3
- removed net C13: U3.GPIO1
- removed net C14: U3.GPIO0
- removed net C15: U3.GPIO18
- removed net C16: U3.GPIO22
- removed net C5: U3.GPIO11
- removed net C6: U3.GPIO10
- removed net C7: U3.GPIO9
- removed net C8: U3.GPIO8
- removed net C9: U3.GPIO6
- removed net CAPS: U3.GPIO19
- removed net GND2: C18.2, C19.2, C20.1, C21.1, C22.1, C23.1, D13.2, J1.GND, J1.SHIELD, R6.2, R7.2, U5.GND, X4.GND, X5.GND, X6.4, Y2.GND
- removed net N$50: U3.GPIO20
- removed net N$51: U3.GPIO21
- removed net N$75: U3.GPIO26/ADC0
- removed net R5: U3.GPIO17
- removed net VCC2: C21.2, C22.2, C23.2, X4.VBUS, X5.VBUS, X6.1
- new net 1: U1.GPIO0
- new net 10: U1.GPIO10
- new net 11: U1.GPIO11
- new net 12: U1.GPIO12
- new net 13: U1.GPIO8
- new net 4: U1.GPIO3
- new net 5: U1.GPIO4
- new net 6: U1.GPIO5
- new net 7: U1.GPIO6
- new net 8: U1.GPIO7
- new net 9: U1.GPIO9
- new net DN-: D13.4, J1.DN1, J1.DN2, R9.2, U5.DM
- new net DN4: U5.DM2, X1.2
- new net DP+: D13.3, J1.DP1, J1.DP2, R8.2, U5.DP
- new net DP4: U5.DP2, X1.3
- new net E11: MT1.A, U1.GPIO22
- new net E12: MT1.B, U1.GPIO23
- new net E21: MT2.A, U1.GPIO26/ADC0
- new net E22: MT2.B, U1.GPIO27/ADC1
- new net E31: MT3.A, U1.GPIO21
- new net E32: MT3.B, U1.GPIO20
- new net E41: MT4.A, U1.GPIO19
- new net E42: MT4.B, U1.GPIO18
- new net L: R10.1, U1.GPIO13
- new net N$31: D3.A, U$3.P1
- new net N$32: D4.A, U$4.P1
- new net N$33: D5.A, MT1.2
- new net N$34: D6.A, MT2.2
- new net N$35: D7.A, MT3.2
- new net N$36: D8.A, MT4.2
- new net N$37: D9.A, U$5.P1
- new net N$38: D10.A, U$6.P1
- new net N$39: D11.A, U$7.P1
- new net N$40: D12.A, U$8.P1
- new net N$41: D14.A, U$9.P1
- new net N$42: D15.A, U$10.P1
- new net N$43: D16.A, U$11.P1
- new net N$44: D17.A, U$12.P1
- net 1V: now also U1.DVDD, U1.VREG_VOUT; no longer U3.DVDD, U3.VREG_VOUT
- net 2: now also U1.GPIO1; no longer U3.GPIO2
- net 3: now also U1.GPIO2; no longer U3.GPIO7
- net 3.3V: now also C21.2, J2.1, U$13.VDD, U$14.VDD, U$15.VDD, U$16.VDD, U$17.VDD, U$18.VDD, U$19.VDD, U$20.VDD, U$21.VDD, U$22.VDD, U$23.VDD, U$24.VDD, U1.ADC_AVDD, U1.IOVDD, U1.USB_VDD, U1.VREG_VIN, U2.VCC; no longer U1.VCC, U3.ADC_AVDD, U3.IOVDD, U3.USB_VDD, U3.VREG_VIN
- net C1: now also MT1.1, U$1.P0, U$5.P0, U$9.P0, U1.GPIO14; no longer U3.GPIO24
- net C2: now also MT2.1, U$10.P0, U$2.P0, U$6.P0, U1.GPIO24; no longer U3.GPIO14
- net C3: now also MT3.1, U$11.P0, U$3.P0, U$7.P0, U1.GPIO28/ADC2; no longer U3.GPIO13
- net C4: now also MT4.1, U$12.P0, U$4.P0, U$8.P0, U1.GPIO29/ADC3; no longer U3.GPIO12
- net CLK: now also J2.5, U1.SWCLK; no longer U3.SWCLK
- net DIO: now also J2.4, U1.SWD; no longer U3.SWD
- net DN: now also R9.1; no longer X6.3
- net DP: now also R8.1; no longer X6.2
- net GND: now also C18.2, C19.2, C20.1, C21.1, D13.2, J1.GND, J1.SHIELD, J2.2, MT1.COM, MT1.SHIELD, MT2.COM, MT2.SHIELD, MT3.COM, MT3.SHIELD, MT4.COM, MT4.SHIELD, R6.2, R7.2, U$13.GND, U$14.GND, U$15.GND, U$16.GND, U$20.GND, U$21.GND, U$22.GND, U$23.GND, U$24.GND, U1.TESTEN, U2.GND, U5.GND, X1.4, X4.GND, X5.GND, Y2.GND; no longer U3.GND, U3.TESTEN
- net N$13: now also U1.USB_DM; no longer U3.USB_DM
- net N$14: now also U1.USB_DP; no longer U3.USB_DP
- net N$153: no longer D13.1
- net N$154: no longer D13.6
- net N$16: now also U2./CS; no longer U1./CS
- net N$17: now also D1.A, U$1.P1; no longer D13.4, J1.DN1, J1.DN2, U5.DM
- net N$18: now also D2.A, U$2.P1; no longer D13.3, J1.DP1, J1.DP2, U5.DP
- net N$27: now also U5.DM3; no longer U5.DM2
- net N$28: now also U5.DP3; no longer U5.DP2
- net R1: now also D5.C, D6.C, D7.C, D8.C, U1.GPIO25; no longer U3.GPIO23
- net R2: now also D1.C, D2.C, D3.C, D4.C, U1.GPIO15; no longer U3.GPIO25
- net R3: now also D10.C, D11.C, D12.C, D9.C, U1.GPIO16; no longer U3.GPIO15
- net R4: now also D14.C, D15.C, D16.C, D17.C, U1.GPIO17; no longer U3.GPIO16
- net RGB: now also R10.2
- net RST: now also J2.3, U1.RUN; no longer U3.RUN
- net SCLK: now also U1.QSPI_SCLK, U2.CLK; no longer U1.CLK, U3.QSPI_SCLK
- net SD0: now also U1.QSPI_SD0, U2.DI(IO0); no longer U1.DI(IO0), U3.QSPI_SD0
- net SD1: now also U1.QSPI_SD1, U2.DO(IO1); no longer U1.DO(IO1), U3.QSPI_SD1
- net SD2: now also U1.QSPI_SD2, U2./WP(IO2); no longer U1./WP(IO2), U3.QSPI_SD2
- net SD3: now also U1.QSPI_SD3, U2./HOLD/RESET(IO3); no longer U1./HOLD/RESET(IO3), U3.QSPI_SD3
- net SS: now also U1.QSPI_CSN; no longer U3.QSPI_CSN
- net VCC: now also X1.1, X4.VBUS, X5.VBUS; no longer U$17.VDD, U$18.VDD, U$19.VDD
- net XTAL1: now also U1.XIN; no longer U3.XIN
- net XTAL2: now also U1.XOUT; no longer U3.XOUT
Other:
- moved on the sheet: C21, MT1, MT2, MT3, MT4, U$10, U$11, U$12, U$5, U$6, U$7, U$8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

Commit message: add
Parts:
- C21: value (none) -> 100nf
- R10: value (none) -> 330
Changed lines of the file:
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@@
 <part name="D16" library="Components" deviceset="DIODE" device="-SOD-123"/>
 <part name="D17" library="Components" deviceset="DIODE" device="-SOD-123"/>
-<part name="R10" library="Components" deviceset="RESISTOR" device="-0603"/>
-<part name="C21" library="Components" deviceset="CAPACITOR" device="-0603"/>
+<part name="R10" library="Components" deviceset="RESISTOR" device="-0603" value="330"/>
+<part name="C21" library="Components" deviceset="CAPACITOR" device="-0603" value="100nf"/>
 </parts>
 <sheets>
