File: Planck/rart50.brd (EAGLE design)
At the start: 9.2 x 5.1 mm, 70 parts, among them J1 I2C-HEADER, J2 USB4085-GF-A_REVA, K1 651005136521, U2 ATMEGA32A-PU, Y1 ECS-160-20-4XDN

Commit message: add
Parts:
- removed 10K, 1K5, 75R, 75R.: (no value), adafruit:0204/7
- removed C1, C2, C4, C5: (no value), adafruit:C050-025X075
- removed C3: (no value), adafruit:E2,5-6
- removed F1: (no value), adafruit:0207/5V
- removed J1: I2C-HEADER, Headers:HEADER-4X1-2.54
- removed J2: USB4085-GF-A_REVA, USB4085-GF-A_REVA:GCT_USB4085-GF-A_REVA
- removed JP1: (no value), arduino_jw:CONN-2X03
- removed K1: 651005136521, Wuerth_Elektronik_eiCan_Communication_Connectors_v2.2:651005136521
- removed OLED: 1X4-BIG, adafruit:1X04-BIG
- removed RGB: (no value), adafruit:1X03
- removed S1, S2: DTS-6, switch-tact:DTS-6
- removed U2: ATMEGA32A-PU, ATMEGA32A-PU:DIP254P1524X482-40
- removed Y1: ECS-160-20-4XDN, Crytal:XTAL_ECS-160-20-4XDN
- added D10, D11, D12, D13, D14, D15, D16, D17, D18, D19, D20, D21, D22, D23, D24, D25, D26, D27, D28, D29, D3, D30, D31, D32, D33, D34, D35, D36, D37, D38, D39, D4, D40, D41, D42, D44, D45, D46, D47, D48, D5, D6, D7, D8, D9: (no value), Components:SOD-123
- added U$49, U$50, U$51, U$52, U$53, U$54, U$55, U$56, U$57, U$58, U$59: SK6812MINI, SK6812MINI:LED-3535
- D1, D2: value 1N4148DO35-7 -> (none); device diode1:DO35-7 -> Components:SOD-123
- U$42: value KEYSWITCH-PLAIN-MXHSPCB-1U -> KEYSWITCH-PLAIN-MXHSPCB-2U-FLIPPED; device Keyboard:MXHSPCB-1U -> Keyboard:MXHSPCB-2U-FLIPPED
- U$43: value KEYSWITCH-PLAIN-MXHSPCB-1U -> SK6812MINI; device Keyboard:MXHSPCB-1U -> SK6812MINI:LED-3535
- moved D2 178.0 mm to (29.4, 75.7), flipped to the bottom, turned to 270 degrees
- moved D1 169.0 mm to (22.1, 76.0), flipped to the bottom, turned to 270 degrees
- moved U$43 125.3 mm to (19.0, 71.0), turned to 180 degrees
- moved U$42 9.50 mm to (123.5, 19.0)
- turned U$2 to 270 degrees
- turned U$3 to 90 degrees
Connections:
- removed net BOOT: S1.3, S1.4, U2.18
- removed net C1: U2.5
- removed net C2: U2.33
- removed net C3: U2.35
- removed net C4: U2.34
- removed net C5: U2.25
- removed net D+: 75R.2, U2.16
- removed net D-: 75R..2, U2.17
- removed net E1: U2.19
- removed net E2: U2.24
- removed net LED: U2.40
- removed net MISO: JP1.1, U2.7
- removed net MOSI: JP1.4, U2.6
- removed net N$1: C2.1, U2.12, Y1.1
- removed net N$6: 1K5.2, 75R..1, D1.C, J1.3, K1.2
- removed net N$79: 75R.1, D2.C, J1.2, K1.3
- removed net R1: U2.1
- removed net R10: U2.28
- removed net R11: U2.14
- removed net R12: U2.27
- removed net R13: U2.15
- removed net R14: U2.26
- removed net R2: U2.39
- removed net R3: U2.2
- removed net R4: U2.38
- removed net R5: U2.3
- removed net R6: U2.37
- removed net R7: U2.4
- removed net R8: U2.36
- removed net R9: U2.29
- removed net RGB: RGB.2, U2.21
- removed net RST: 10K.1, JP1.5, S2.3, S2.4, U2.9
- removed net SCK: JP1.3, U2.8
- removed net SCL: OLED.3, U2.22
- removed net SDA: OLED.4, U2.23
- removed net VBUS: J2.A4, J2.A9, J2.B4, J2.B9
- removed net VCC: 10K.2, 1K5.1, C3.+, C4.1, C5.1, F1.1, JP1.2, OLED.2, RGB.3, U2.10, U2.30
- new net N$10: D4.A, U$4.MX2, U$4.P$3, U$4.P$4
- new net N$12: D6.A, U$6.MX2, U$6.P$3, U$6.P$4
- new net N$13: D7.A, U$7.MX2, U$7.P$3, U$7.P$4
- new net N$14: D8.A, U$8.MX2, U$8.P$3, U$8.P$4
- new net N$15: D9.A, U$9.MX2, U$9.P$3, U$9.P$4
- new net N$16: D10.A, U$10.MX2, U$10.P$3, U$10.P$4
- new net N$17: D11.A, U$11.MX2, U$11.P$3, U$11.P$4
- new net N$18: D12.A, U$12.MX2, U$12.P$3, U$12.P$4
- new net N$19: D13.A, U$13.MX2, U$13.P$3, U$13.P$4
- new net N$20: D14.A, U$14.MX2, U$14.P$3, U$14.P$4
- new net N$21: D15.A, U$15.MX2, U$15.P$3, U$15.P$4
- new net N$22: D16.A, U$16.MX2, U$16.P$3, U$16.P$4
- new net N$23: D17.A, U$17.MX2, U$17.P$3, U$17.P$4
- new net N$24: D18.A, U$18.MX2, U$18.P$3, U$18.P$4
- new net N$25: D19.A, U$19.MX2, U$19.P$3, U$19.P$4
- new net N$26: D20.A, U$20.MX2, U$20.P$3, U$20.P$4
- new net N$27: D21.A, U$21.MX2, U$21.P$3, U$21.P$4
- new net N$28: D22.A, U$22.MX2, U$22.P$3, U$22.P$4
- new net N$29: D23.A, U$23.MX2, U$23.P$3, U$23.P$4
- new net N$30: D24.A, U$24.MX2, U$24.P$3, U$24.P$4
- new net N$31: D25.A, U$25.MX2, U$25.P$3, U$25.P$4
- new net N$32: D26.A, U$26.MX2, U$26.P$3, U$26.P$4
- new net N$33: D27.A, U$27.MX2, U$27.P$3, U$27.P$4
- new net N$34: D28.A, U$28.MX2, U$28.P$3, U$28.P$4
- new net N$35: D29.A, U$29.MX2, U$29.P$3, U$29.P$4
- new net N$36: D30.A, U$30.MX2, U$30.P$3, U$30.P$4
- new net N$37: D31.A, U$31.MX2, U$31.P$3, U$31.P$4
- new net N$38: D32.A, U$32.MX2, U$32.P$3, U$32.P$4
- new net N$39: D33.A, U$33.MX2, U$33.P$3, U$33.P$4
- new net N$40: D34.A, U$34.MX2, U$34.P$3, U$34.P$4
- new net N$41: D35.A, U$35.MX2, U$35.P$3, U$35.P$4
- new net N$42: D36.A, U$36.MX2, U$36.P$3, U$36.P$4
- new net N$43: D37.A, U$37.MX2, U$37.P$3, U$37.P$4
- new net N$44: D38.A, U$38.MX2, U$38.P$3, U$38.P$4
- new net N$45: D39.A, U$39.MX2, U$39.P$3, U$39.P$4
- new net N$46: D40.A, U$40.MX2, U$40.P$3, U$40.P$4
- new net N$47: D41.A, U$41.MX2, U$41.P$3, U$41.P$4
- new net N$49: D44.A, U$44.MX2, U$44.P$3, U$44.P$4
- new net N$50: D45.A, U$45.MX2, U$45.P$3, U$45.P$4
- new net N$51: D46.A, U$46.MX2, U$46.P$3, U$46.P$4
- new net N$52: D47.A, U$47.MX2, U$47.P$3, U$47.P$4
- new net N$53: D48.A, U$48.MX2, U$48.P$3, U$48.P$4
- new net N$54: U$43.3, U$49.1
- new net N$55: U$49.3, U$50.1
- new net N$56: U$50.3, U$51.1
- new net N$57: U$51.3, U$52.1
- new net N$58: U$52.3, U$53.1
- new net N$59: U$53.3, U$54.1
- new net N$60: U$54.3, U$55.1
- new net N$61: U$55.3, U$56.1
- new net N$62: U$56.3, U$57.1
- new net N$63: U$57.3, U$58.1
- new net N$64: U$58.3, U$59.1
- new net N$7: D1.A, U$1.MX2, U$1.P$3, U$1.P$4
- new net N$9: D3.A, U$3.MX2, U$3.P$3, U$3.P$4
- new net VDD: U$43.4, U$49.4, U$50.4, U$51.4, U$52.4, U$53.4, U$54.4, U$55.4, U$56.4, U$57.4, U$58.4, U$59.4
- net GND: now also U$43.2, U$49.2, U$50.2, U$51.2, U$52.2, U$53.2, U$54.2, U$55.2, U$56.2, U$57.2, U$58.2, U$59.2; no longer C1.2, C2.2, C3.-, C4.2, C5.2, D1.A, D2.A, J1.1, JP1.6, K1.5, OLED.1, RGB.1, S1.1, S1.2, S2.1, S2.2, U2.11, U2.31
- net N$11: now also D5.A, U$5.MX2, U$5.P$3, U$5.P$4; no longer F1.2, J1.4, K1.1
- net N$48: now also D42.A, U$42.MX2, U$42.P$3, U$42.P$4; no longer U2.20
- net N$8: now also D2.A, U$2.MX2, U$2.P$3, U$2.P$4; no longer C1.1, U2.13, Y1.2
Other:
- board size 9.2 x 5.1 mm -> 228 x 76 mm

Commit message: add
Parts:
- added U$60, U$61, U$62, U$63, U$64, U$65, U$66, U$67, U$68, U$69, U$70, U$71, U$72, U$73, U$74, U$75, U$76, U$77, U$78, U$79, U$80, U$81, U$82, U$83, U$84, U$85, U$86, U$87, U$88, U$89, U$90, U$91, U$92, U$93, U$94: SK6812MINI, SK6812MINI:LED-3535
Connections:
- new net N$65: U$60.3, U$61.1
- new net N$66: U$61.3, U$62.1
- new net N$67: U$62.3, U$63.1
- new net N$68: U$63.3, U$64.1
- new net N$69: U$64.3, U$65.1
- new net N$70: U$65.3, U$66.1
- new net N$71: U$66.3, U$67.1
- new net N$72: U$67.3, U$68.1
- new net N$73: U$68.3, U$69.1
- new net N$74: U$69.3, U$70.1
- new net N$75: U$70.3, U$71.1
- new net N$76: U$72.3, U$73.1
- new net N$77: U$73.3, U$74.1
- new net N$78: U$74.3, U$75.1
- new net N$79: U$75.3, U$76.1
- new net N$80: U$76.3, U$77.1
- new net N$81: U$77.3, U$78.1
- new net N$82: U$78.3, U$79.1
- new net N$83: U$79.3, U$80.1
- new net N$84: U$80.3, U$81.1
- new net N$85: U$81.3, U$82.1
- new net N$86: U$82.3, U$83.1
- new net N$87: U$84.3, U$85.1
- new net N$88: U$85.3, U$86.1
- new net N$89: U$86.3, U$87.1
- new net N$90: U$87.3, U$88.1
- new net N$91: U$88.3, U$89.1
- new net N$92: U$89.3, U$90.1
- new net N$93: U$90.3, U$91.1
- new net N$94: U$91.3, U$92.1
- new net N$95: U$92.3, U$93.1
- new net N$96: U$93.3, U$94.1
- net GND: now also U$60.2, U$61.2, U$62.2, U$63.2, U$64.2, U$65.2, U$66.2, U$67.2, U$68.2, U$69.2, U$70.2, U$71.2, U$72.2, U$73.2, U$74.2, U$75.2, U$76.2, U$77.2, U$78.2, U$79.2, U$80.2, U$81.2, U$82.2, U$83.2, U$84.2, U$85.2, U$86.2, U$87.2, U$88.2, U$89.2, U$90.2, U$91.2, U$92.2, U$93.2, U$94.2
- net VDD: now also U$60.4, U$61.4, U$62.4, U$63.4, U$64.4, U$65.4, U$66.4, U$67.4, U$68.4, U$69.4, U$70.4, U$71.4, U$72.4, U$73.4, U$74.4, U$75.4, U$76.4, U$77.4, U$78.4, U$79.4, U$80.4, U$81.4, U$82.4, U$83.4, U$84.4, U$85.4, U$86.4, U$87.4, U$88.4, U$89.4, U$90.4, U$91.4, U$92.4, U$93.4, U$94.4
Other:
- outline, holes or cut-outs redrawn

Commit message: add
Parts:
- added BOOT, RESET: (no value), adafruit:1X01
- added C1, C2, C3, C4, C5, C6, C7: 100nf, Components:C0603
- added C10, C16, C17, C8: 1uF, Components:C0603
- added C11, C12, C13: 100nF, Components:C0603
- added C14, C15: 22pF, Components:C0603
- added C9: 10uF, Components:C0603
- added D43: SRV05-4.TCT, SRV05-4.TCT:SOT95P280X145-6N
- added J1: TYPE-C-31-M-12, TYPE-C-31-M-12:HRO_TYPE-C-31-M-12
- added J2: 1X5, adafruit:1X05-3.5MM
- added JP3, JP4: (no value), adafruit:1X01-CLEANBIG
- added R1, R2: 27R, Components:R0603
- added R3, R5: 1k, Components:R0603
- added R39: 0ZCJ0075AF2E, fuse:RESC3216X125N
- added R4: 1K, Components:R0603
- added R6, R7: 5.1k, Components:R0603
- added U1: RP2040, RP2040:QFN40P700X700X90-57N
- added U2: W25Q128JVSIQ, W25Q128JVSIQ:SOIC127P790X216-8N
- added U4: PMIC-LDO-XC6206P332MR-G(SOT23), C5446-XC6206P332MR-G_SOT23_:SOT-23
- added Y1: (no value), Components:CRYSTAL-3.2X2.5
- moved D14 14.2 mm to (26.9, 57.0)
- moved D3 11.7 mm to (53.9, 76.0)
- moved U$49 10.4 mm to (38.0, 81.0)
- moved U$50 10.1 mm to (57.0, 81.0)
- moved D2 5.52 mm to (34.9, 76.0)
- turned U$2 to 180 degrees
- turned U$3 to 180 degrees
Connections:
- new net 1: U1.2
- new net 10: U1.13
- new net 11: U1.14
- new net 12: U1.15
- new net 13: U1.11
- new net 14: U1.16
- new net 15: U1.17
- new net 16: U1.18
- new net 17: U1.27
- new net 18: U1.28
- new net 19: U1.29
- new net 1V: C10.2, C11.2, C12.2, U1.23, U1.45, U1.50
- new net 2: U1.3
- new net 20: U1.30
- new net 21: U1.31
- new net 22: U1.32
- new net 23: U1.34
- new net 24: U1.35
- new net 25: U1.36
- new net 26: U1.37
- new net 27: U1.38
- new net 28: U1.39
- new net 29: U1.40
- new net 3: U1.4
- new net 3.3V: C1.2, C13.2, C17.2, C2.2, C3.2, C4.2, C5.2, C6.2, C7.2, C8.2, C9.2, J2.1, R5.2, U1.1, U1.10, U1.22, U1.33, U1.42, U1.43, U1.44, U1.48, U1.49, U2.8, U4.2
- new net 30: U1.41
- new net 4: U1.5
- new net 5: U1.6
- new net 6: U1.7
- new net 7: U1.8
- new net 8: U1.9
- new net 9: U1.12
- new net CLK: J2.5, U1.24
- new net DIO: J2.4, U1.25
- new net DN: R1.2
- new net DN-: D43.4, J1.A7, J1.B7
- new net DP: R2.2
- new net DP+: D43.3, J1.A6, J1.B6
- new net GND1: D43.2, J1.A1B12, J1.B1A12, J1.S1, J1.S2, J1.S3, J1.S4, R6.2, R7.2
- new net N$100: R3.1, U2.1
- new net N$101: D43.5, J1.A4B9, J1.B4A9, R39.2
- new net N$153: J1.B5, R6.1
- new net N$154: J1.A5, R7.1
- new net N$97: R1.1, U1.46
- new net N$98: R2.1, U1.47
- new net N$99: C14.2, R4.1, Y1.1
- new net RST: J2.3, R5.1, RESET.1, U1.26
- new net SCLK: U1.52, U2.6
- new net SD0: U1.53, U2.5
- new net SD1: U1.55, U2.2
- new net SD2: U1.54, U2.3
- new net SD3: U1.51, U2.7
- new net SS: BOOT.1, R3.2, U1.56
- new net VCC: C16.2, U4.3
- new net VCC1: R39.1
- new net XTAL1: R4.2, U1.20
- new net XTAL2: C15.2, U1.21, Y1.3
- net GND: now also C1.1, C10.1, C11.1, C12.1, C13.1, C14.1, C15.1, C16.1, C17.1, C2.1, C3.1, C4.1, C5.1, C6.1, C7.1, C8.1, C9.1, J2.2, JP3.1, JP4.1, U1.19, U1.57, U2.4, U4.1, Y1.2, Y1.4
Other:
- board size 228 x 76 mm -> 228 x 77.2 mm
