File: Planck/rart50.sch (EAGLE design)
At the start: 70 parts, among them J1 I2C-HEADER, J2 USB4085-GF-A_REVA, K1 651005136521, U2 ATMEGA32A-PU, Y1 ECS-160-20-4XDN

Commit message: add
Parts:
- removed 10K, 1K5, 75R, 75R.: (no value), adafruit:R-US_0204/7
- removed C1, C2, C4, C5: (no value), adafruit:C-US050-025X075
- removed C3: (no value), adafruit:CPOL-USE2.5-6
- removed F1: (no value), adafruit:R-US_0207/5V
- removed J1: I2C-HEADER, Headers:I2C-HEADER
- removed J2: USB4085-GF-A_REVA, USB4085-GF-A_REVA:USB4085-GF-A_REVA
- removed JP1: (no value), arduino_jw:ARDUINO_CONN-ICSP
- removed K1: 651005136521, Wuerth_Elektronik_eiCan_Communication_Connectors_v2.2:651005136521
- removed OLED: 1X4-BIG, adafruit:1X4-BIG
- removed RGB: (no value), adafruit:PINHD-1X3
- removed S1, S2: DTS-6, switch-tact:DTS-6
- removed U2: ATMEGA32A-PU, ATMEGA32A-PU:ATMEGA32A-PU
- removed Y1: ECS-160-20-4XDN, Crytal:ECS-160-20-4XDN
- added D10, D11, D12, D13, D14, D15, D16, D17, D18, D19, D20, D21, D22, D23, D24, D25, D26, D27, D28, D29, D3, D30, D31, D32, D33, D34, D35, D36, D37, D38, D39, D4, D40, D41, D42, D44, D45, D46, D47, D48, D5, D6, D7, D8, D9: (no value), Components:DIODE-SOD-123
- added U$49, U$50, U$51, U$52, U$53, U$54, U$55, U$56, U$57, U$58, U$59: SK6812MINI, SK6812MINI:SK6812MINI
- D1, D2: value 1N4148DO35-7 -> (none); device diode1:1N4148DO35-7 -> Components:DIODE-SOD-123
- U$42: value KEYSWITCH-PLAIN-MXHSPCB-1U -> KEYSWITCH-PLAIN-MXHSPCB-2U-FLIPPED; device Keyboard:KEYSWITCH-PLAIN-MXHSPCB-1U -> Keyboard:KEYSWITCH-PLAIN-MXHSPCB-2U-FLIPPED
- U$43: value KEYSWITCH-PLAIN-MXHSPCB-1U -> SK6812MINI; device Keyboard:KEYSWITCH-PLAIN-MXHSPCB-1U -> SK6812MINI:SK6812MINI
Connections:
- removed net BOOT: S1.3, S1.4, U2.PD4
- removed net C1: U2.PB4
- removed net C2: U2.PA7
- removed net C3: U2.PA5
- removed net C4: U2.PA6
- removed net C5: U2.PC3
- removed net D+: 75R.2, U2.PD2
- removed net D-: 75R..2, U2.PD3
- removed net E1: U2.PD5
- removed net E2: U2.PC2
- removed net GND: C1.2, C2.2, C3.-, C4.2, C5.2, D1.A, D2.A, J1.GND, JP1.6, K1.GND, OLED.1, RGB.1, S1.1, S1.2, S2.1, S2.2, U2.GND, U2.GND_2
- removed net LED: U2.PA0
- removed net MISO: JP1.1, U2.PB6
- removed net MOSI: JP1.4, U2.PB5
- removed net N$1: C2.1, U2.XTAL2, Y1.1
- removed net N$6: 1K5.2, 75R..1, D1.C, J1.SDA, K1.D-
- removed net N$79: 75R.1, D2.C, J1.SCL, K1.D+
- removed net R1: U2.PB0
- removed net R10: U2.PC6
- removed net R11: U2.PD0
- removed net R12: U2.PC5
- removed net R13: U2.PD1
- removed net R14: U2.PC4
- removed net R2: U2.PA1
- removed net R3: U2.PB1
- removed net R4: U2.PA2
- removed net R5: U2.PB2
- removed net R6: U2.PA3
- removed net R7: U2.PB3
- removed net R8: U2.PA4
- removed net R9: U2.PC7
- removed net RGB: RGB.2, U2.PD7
- removed net RST: 10K.1, JP1.5, S2.3, S2.4, U2.~RESET
- removed net SCK: JP1.3, U2.PB7
- removed net SCL: OLED.3, U2.PC0
- removed net SDA: OLED.4, U2.PC1
- removed net VCC: 10K.2, 1K5.1, C3.+, C4.1, C5.1, F1.1, JP1.2, OLED.2, RGB.3, U2.AVCC, U2.VCC
- new net N$10: D4.A, U$4.P1
- new net N$12: D6.A, U$6.P1
- new net N$13: D7.A, U$7.P1
- new net N$14: D8.A, U$8.P1
- new net N$15: D9.A, U$9.P1
- new net N$16: D10.A, U$10.P1
- new net N$17: D11.A, U$11.P1
- new net N$18: D12.A, U$12.P1
- new net N$19: D13.A, U$13.P1
- new net N$20: D14.A, U$14.P1
- new net N$21: D15.A, U$15.P1
- new net N$22: D16.A, U$16.P1
- new net N$23: D17.A, U$17.P1
- new net N$24: D18.A, U$18.P1
- new net N$25: D19.A, U$19.P1
- new net N$26: D20.A, U$20.P1
- new net N$27: D21.A, U$21.P1
- new net N$28: D22.A, U$22.P1
- new net N$29: D23.A, U$23.P1
- new net N$30: D24.A, U$24.P1
- new net N$31: D25.A, U$25.P1
- new net N$32: D26.A, U$26.P1
- new net N$33: D27.A, U$27.P1
- new net N$34: D28.A, U$28.P1
- new net N$35: D29.A, U$29.P1
- new net N$36: D30.A, U$30.P1
- new net N$37: D31.A, U$31.P1
- new net N$38: D32.A, U$32.P1
- new net N$39: D33.A, U$33.P1
- new net N$40: D34.A, U$34.P1
- new net N$41: D35.A, U$35.P1
- new net N$42: D36.A, U$36.P1
- new net N$43: D37.A, U$37.P1
- new net N$44: D38.A, U$38.P1
- new net N$45: D39.A, U$39.P1
- new net N$46: D40.A, U$40.P1
- new net N$47: D41.A, U$41.P1
- new net N$49: D44.A, U$44.P1
- new net N$50: D45.A, U$45.P1
- new net N$51: D46.A, U$46.P1
- new net N$52: D47.A, U$47.P1
- new net N$53: D48.A, U$48.P1
- new net N$54: U$43.DO, U$49.DI
- new net N$55: U$49.DO, U$50.DI
- new net N$56: U$50.DO, U$51.DI
- new net N$57: U$51.DO, U$52.DI
- new net N$58: U$52.DO, U$53.DI
- new net N$59: U$53.DO, U$54.DI
- new net N$60: U$54.DO, U$55.DI
- new net N$61: U$55.DO, U$56.DI
- new net N$62: U$56.DO, U$57.DI
- new net N$63: U$57.DO, U$58.DI
- new net N$64: U$58.DO, U$59.DI
- new net N$7: D1.A, U$1.P1
- new net N$9: D3.A, U$3.P1
- net N$11: now also D5.A, U$5.P1; no longer F1.2, J1.VCC, K1.VCC
- net N$48: now also D42.A, U$42.P1; no longer U2.PD6
- net N$8: now also D2.A, U$2.P1; no longer C1.1, U2.XTAL1, Y1.2

Commit message: add
Parts:
- added U$60, U$61, U$62, U$63, U$64, U$65, U$66, U$67, U$68, U$69, U$70, U$71, U$72, U$73, U$74, U$75, U$76, U$77, U$78, U$79, U$80, U$81, U$82, U$83, U$84, U$85, U$86, U$87, U$88, U$89, U$90, U$91, U$92, U$93, U$94: SK6812MINI, SK6812MINI:SK6812MINI
Connections:
- new net N$65: U$60.DO, U$61.DI
- new net N$66: U$61.DO, U$62.DI
- new net N$67: U$62.DO, U$63.DI
- new net N$68: U$63.DO, U$64.DI
- new net N$69: U$64.DO, U$65.DI
- new net N$70: U$65.DO, U$66.DI
- new net N$71: U$66.DO, U$67.DI
- new net N$72: U$67.DO, U$68.DI
- new net N$73: U$68.DO, U$69.DI
- new net N$74: U$69.DO, U$70.DI
- new net N$75: U$70.DO, U$71.DI
- new net N$76: U$72.DO, U$73.DI
- new net N$77: U$73.DO, U$74.DI
- new net N$78: U$74.DO, U$75.DI
- new net N$79: U$75.DO, U$76.DI
- new net N$80: U$76.DO, U$77.DI
- new net N$81: U$77.DO, U$78.DI
- new net N$82: U$78.DO, U$79.DI
- new net N$83: U$79.DO, U$80.DI
- new net N$84: U$80.DO, U$81.DI
- new net N$85: U$81.DO, U$82.DI
- new net N$86: U$82.DO, U$83.DI
- new net N$87: U$84.DO, U$85.DI
- new net N$88: U$85.DO, U$86.DI
- new net N$89: U$86.DO, U$87.DI
- new net N$90: U$87.DO, U$88.DI
- new net N$91: U$88.DO, U$89.DI
- new net N$92: U$89.DO, U$90.DI
- new net N$93: U$90.DO, U$91.DI
- new net N$94: U$91.DO, U$92.DI
- new net N$95: U$92.DO, U$93.DI
- new net N$96: U$93.DO, U$94.DI

Commit message: add
Parts:
- added BOOT, RESET: (no value), adafruit:PINHD-1X1
- added C1, C2, C3, C4, C5, C6, C7: 100nf, Components:CAPACITOR-0603
- added C10, C16, C17, C8: 1uF, Components:CAPACITOR-0603
- added C11, C12, C13: 100nF, Components:CAPACITOR-0603
- added C14, C15: 22pF, Components:CAPACITOR-0603
- added C9: 10uF, Components:CAPACITOR-0603
- added D43: SRV05-4.TCT, SRV05-4.TCT:SRV05-4.TCT
- added J1: TYPE-C-31-M-12, TYPE-C-31-M-12:TYPE-C-31-M-12
- added J2: 1X5, adafruit:1X5
- added JP3, JP4: (no value), adafruit:PINHD-1X1CB
- added R1, R2: 27R, Components:RESISTOR-0603
- added R3, R5: 1k, Components:RESISTOR-0603
- added R39: 0ZCJ0075AF2E, fuse:0ZCJ0075AF2E
- added R4: 1K, Components:RESISTOR-0603
- added R6, R7: 5.1k, Components:RESISTOR-0603
- added U1: RP2040, RP2040:RP2040
- added U2: W25Q128JVSIQ, W25Q128JVSIQ:W25Q128JVSIQ
- added U4: PMIC-LDO-XC6206P332MR-G(SOT23), C5446-XC6206P332MR-G_SOT23_:PMIC-LDO-XC6206P332MR-G(SOT23)
- added Y1: (no value), Components:CRYSTAL-4PIN-3.2X2.5
Connections:
- new net 1: U1.GPIO0
- new net 10: U1.GPIO10
- new net 11: U1.GPIO11
- new net 12: U1.GPIO12
- new net 13: U1.GPIO8
- new net 14: U1.GPIO13
- new net 15: U1.GPIO14
- new net 16: U1.GPIO15
- new net 17: U1.GPIO16
- new net 18: U1.GPIO17
- new net 19: U1.GPIO18
- new net 1V: C10.2, C11.2, C12.2, U1.DVDD, U1.VREG_VOUT
- new net 2: U1.GPIO1
- new net 20: U1.GPIO19
- new net 21: U1.GPIO20
- new net 22: U1.GPIO21
- new net 23: U1.GPIO22
- new net 24: U1.GPIO23
- new net 25: U1.GPIO24
- new net 26: U1.GPIO25
- new net 27: U1.GPIO26/ADC0
- new net 28: U1.GPIO27/ADC1
- new net 29: U1.GPIO28/ADC2
- new net 3: U1.GPIO2
- new net 3.3V: C1.2, C13.2, C17.2, C2.2, C3.2, C4.2, C5.2, C6.2, C7.2, C8.2, C9.2, J2.1, R5.2, U1.ADC_AVDD, U1.IOVDD, U1.USB_VDD, U1.VREG_VIN, U2.VCC, U4.VOUT
- new net 30: U1.GPIO29/ADC3
- new net 4: U1.GPIO3
- new net 5: U1.GPIO4
- new net 6: U1.GPIO5
- new net 7: U1.GPIO6
- new net 8: U1.GPIO7
- new net 9: U1.GPIO9
- new net CLK: J2.5, U1.SWCLK
- new net DIO: J2.4, U1.SWD
- new net DN: R1.2
- new net DN-: D43.4, J1.DN1, J1.DN2
- new net DP: R2.2
- new net DP+: D43.3, J1.DP1, J1.DP2
- new net GND: C1.1, C10.1, C11.1, C12.1, C13.1, C14.1, C15.1, C16.1, C17.1, C2.1, C3.1, C4.1, C5.1, C6.1, C7.1, C8.1, C9.1, J2.2, JP3.1, JP4.1, U1.GND, U1.TESTEN, U2.GND, U4.VSS, Y1.GND
- new net GND1: D43.2, J1.GND, J1.SHIELD, R6.2, R7.2
- new net N$100: R3.1, U2./CS
- new net N$101: D43.5, J1.VBUS, R39.2
- new net N$153: J1.CC2, R6.1
- new net N$154: J1.CC1, R7.1
- new net N$97: R1.1, U1.USB_DM
- new net N$98: R2.1, U1.USB_DP
- new net N$99: C14.2, R4.1, Y1.1
- new net RST: J2.3, R5.1, RESET.1, U1.RUN
- new net SCLK: U1.QSPI_SCLK, U2.CLK
- new net SD0: U1.QSPI_SD0, U2.DI(IO0)
- new net SD1: U1.QSPI_SD1, U2.DO(IO1)
- new net SD2: U1.QSPI_SD2, U2./WP(IO2)
- new net SD3: U1.QSPI_SD3, U2./HOLD/RESET(IO3)
- new net SS: BOOT.1, R3.2, U1.QSPI_CSN
- new net VCC: C16.2, U4.VIN
- new net VCC1: R39.1
- new net XTAL1: R4.2, U1.XIN
- new net XTAL2: C15.2, U1.XOUT, Y1.2
